Commit message: halp max

File: src/senseglove/senseglove_description/urdf/dk1.xacro (robot description, xacro)
@@ -2,8 +2,4 @@
 <!-- Revolute-Revolute Manipulator -->
 <robot name="dk1" xmlns:xacro="http://www.ros.org/wiki/xacro">
-    <!-- Switch between airgaiting or standing on the ground-->
-    <!--Value set to: 'world' fixes the robot to the world-->
-    <!--Value set to: 'base_link' makes the robot stand on the ground-->
-    <!--Important note: when changing value make sure rviz fixed frame is set to the same value (moveit.rviz)-->
     <!-- Constants for robot dimensions -->
     <xacro:property name="PI" value="3.1415926535897931"/>
@@ -31,4 +27,8 @@
         <origin xyz="0 ${-joint_base_width} 0" rpy="0 0 0"/>
         <axis xyz="0 1 0"/>
+        <limit velocity="${10}"
+               effort="${10000}"
+               lower="${-5}"
+               upper="${5}"/>
     </joint>
     <!-- Joint Base-->

Commit message: First stable version, can read out sensegloev data, but requires Sensecomm application to run instead of fixing it ourselves

File: src/senseglove/senseglove_description/urdf/dk1.xacro (robot description, xacro)
@@ -17,53 +17,563 @@
     <!-- Used for fixing robot to Gazebo 'base_link' -->
     <link name="world"/>
+    <!-- glove hub -->
+    <link name="glove_hub">
+        <visual>
+            <origin xyz="0 0 0" rpy="0 0 0"/>
+            <geometry>
+                <mesh filename="package://senseglove_description/urdf/STL/MK29_DK1_HUB.STL" scale="1 1 1"/>
+            </geometry>
+        </visual>
+    </link>
+    <!-- thumb brake -->
+    <link name="thumb_brake">
+        <visual>
+            <origin xyz="0 0 ${-bar_length/2}" rpy="0 0 0"/>
+            <geometry>
+                <mesh filename="package://senseglove_description/urdf/STL/MK29_DK1_Brake_assembly_v2.STL" scale="1 1 1"/>
+            </geometry>
+        </visual>
+    </link>
+    <!-- thumb abduction -->
+    <link name="thumb_abduction">
+        <visual>
+            <origin xyz="0 0 ${-bar_length/2}" rpy="0 0 0"/>
+            <geometry>
+                <mesh filename="package://senseglove_description/urdf/STL/MK29_DK1_Abduction_joint_v2.STL" scale="1 1 1"/>
+            </geometry>
+        </visual>
+    </link>
+    <!-- thumb flexion one -->
+    <link name="thumb_flexion_one">
+        <visual>
+            <origin xyz="0 0 ${-bar_length/2}" rpy="0 0 0"/>
+            <geometry>
+                <mesh filename="package://senseglove_description/urdf/STL/MK29_DK1_Flexion_joint_1_v2.STL" scale="1 1 1"/>
+            </geometry>
+        </visual>
+    </link>
+    <!-- thumb flexion two -->
+    <link name="thumb_flexion_two">
+        <visual>
+            <origin xyz="0 0 ${-bar_length/2}" rpy="0 0 0"/>
+            <geometry>
+                <mesh filename="package://senseglove_description/urdf/STL/MK29_DK1_Flexion_joint_2_v2.STL" scale="1 1 1"/>
+            </geometry>
+        </visual>
+    </link>
+    <!-- thumb flexion three -->
+    <link name="thumb_flexion_three">
+        <visual>
+            <origin xyz="0 0 ${-bar_length/2}" rpy="0 0 0"/>
+            <geometry>
+                <mesh filename="package://senseglove_description/urdf/STL/MK29_DK1_Flexion_joint_3_v2.STL" scale="1 1 1"/>
+            </geometry>
+        </visual>
+    </link>
+    <!-- thumb thimble -->
+    <link name="thumb_thimble">
+        <visual>
+            <origin xyz="0 0 ${-bar_length/2}" rpy="0 0 0"/>
+            <geometry>
+                <mesh filename="package://senseglove_description/urdf/STL/MK29_DK1_Thimble_v2.STL" scale="1 1 1"/>
+            </geometry>
+        </visual>
+    </link>
+    <!-- index brake -->
+    <link name="index_brake">
+        <visual>
+            <origin xyz="0 0 ${-bar_length/2}" rpy="0 0 0"/>
+            <geometry>
+                <mesh filename="package://senseglove_description/urdf/STL/MK29_DK1_Brake_assembly_v2.STL" scale="1 1 1"/>
+            </geometry>
+        </visual>
+    </link>
+    <!-- index abduction -->
+    <link name="index_abduction">
+        <visual>
+            <origin xyz="0 0 ${-bar_length/2}" rpy="0 0 0"/>
+            <geometry>
+                <mesh filename="package://senseglove_description/urdf/STL/MK29_DK1_Abduction_joint_v2.STL" scale="1 1 1"/>
+            </geometry>
+        </visual>
+    </link>
+    <!-- index flexion one -->
+    <link name="index_flexion_one">
+        <visual>
+            <origin xyz="0 0 ${-bar_length/2}" rpy="0 0 0"/>
+            <geometry>
+                <mesh filename="package://senseglove_description/urdf/STL/MK29_DK1_Flexion_joint_1_v2.STL" scale="1 1 1"/>
+            </geometry>
+        </visual>
+    </link>
+    <!-- index flexion two -->
+    <link name="index_flexion_two">
+        <visual>
+            <origin xyz="0 0 ${-bar_length/2}" rpy="0 0 0"/>
+            <geometry>
+                <mesh filename="package://senseglove_description/urdf/STL/MK29_DK1_Flexion_joint_2_v2.STL" scale="1 1 1"/>
+            </geometry>
+        </visual>
+    </link>
+    <!-- index flexion three -->
+    <link name="index_flexion_three">
+        <visual>
+            <origin xyz="0 0 ${-bar_length/2}" rpy="0 0 0"/>
+            <geometry>
+                <mesh filename="package://senseglove_description/urdf/STL/MK29_DK1_Flexion_joint_3_v2.STL" scale="1 1 1"/>
+            </geometry>
+        </visual>
+    </link>
+    <!-- index thimble -->
+    <link name="index_thimble">
+        <visual>
+            <origin xyz="0 0 ${-bar_length/2}" rpy="0 0 0"/>
+            <geometry>
+                <mesh filename="package://senseglove_description/urdf/STL/MK29_DK1_Thimble_v2.STL" scale="1 1 1"/>
+            </geometry>
+        </visual>
+    </link>
+    <!-- middle brake -->
+    <link name="middle_brake">
+        <visual>
+            <origin xyz="0 0 ${-bar_length/2}" rpy="0 0 0"/>
+            <geometry>
+                <mesh filename="package://senseglove_description/urdf/STL/MK29_DK1_Brake_assembly_v2.STL" scale="1 1 1"/>
+            </geometry>
+        </visual>
+    </link>
+    <!-- middle abduction -->
+    <link name="middle_abduction">
+        <visual>
+            <origin xyz="0 0 ${-bar_length/2}" rpy="0 0 0"/>
+            <geometry>
+                <mesh filename="package://senseglove_description/urdf/STL/MK29_DK1_Abduction_joint_v2.STL" scale="1 1 1"/>
+            </geometry>
+        </visual>
+    </link>
+    <!-- middle flexion one -->
+    <link name="middle_flexion_one">
+        <visual>
+            <origin xyz="0 0 ${-bar_length/2}" rpy="0 0 0"/>
+            <geometry>
+                <mesh filename="package://senseglove_description/urdf/STL/MK29_DK1_Flexion_joint_1_v2.STL" scale="1 1 1"/>
+            </geometry>
+        </visual>
+    </link>
+    <!-- middle flexion two -->
+    <link name="middle_flexion_two">
+        <visual>
+            <origin xyz="0 0 ${-bar_length/2}" rpy="0 0 0"/>
+            <geometry>
+                <mesh filename="package://senseglove_description/urdf/STL/MK29_DK1_Flexion_joint_2_v2.STL" scale="1 1 1"/>
+            </geometry>
+        </visual>
+    </link>
+    <!-- middle flexion three -->
+    <link name="middle_flexion_three">
+        <visual>
+            <origin xyz="0 0 ${-bar_length/2}" rpy="0 0 0"/>
+            <geometry>
+                <mesh filename="package://senseglove_description/urdf/STL/MK29_DK1_Flexion_joint_3_v2.STL" scale="1 1 1"/>
+            </geometry>
+        </visual>
+    </link>
+    <!-- middle thimble -->
+    <link name="middle_thimble">
+        <visual>
+            <origin xyz="0 0 ${-bar_length/2}" rpy="0 0 0"/>
+            <geometry>
+                <mesh filename="package://senseglove_description/urdf/STL/MK29_DK1_Thimble_v2.STL" scale="1 1 1"/>
+            </geometry>
+        </visual>
+    </link>
+    <!-- ring brake -->
+    <link name="ring_brake">
+        <visual>
+            <origin xyz="0 0 ${-bar_length/2}" rpy="0 0 0"/>
+            <geometry>
+                <mesh filename="package://senseglove_description/urdf/STL/MK29_DK1_Brake_assembly_v2.STL" scale="1 1 1"/>
+            </geometry>
+        </visual>
+    </link>
+    <!-- ring abduction -->
+    <link name="ring_abduction">
+        <visual>
+            <origin xyz="0 0 ${-bar_length/2}" rpy="0 0 0"/>
+            <geometry>
+                <mesh filename="package://senseglove_description/urdf/STL/MK29_DK1_Abduction_joint_v2.STL" scale="1 1 1"/>
+            </geometry>
+        </visual>
+    </link>
+    <!-- ring flexion one -->
+    <link name="ring_flexion_one">
+        <visual>
+            <origin xyz="0 0 ${-bar_length/2}" rpy="0 0 0"/>
+            <geometry>
+                <mesh filename="package://senseglove_description/urdf/STL/MK29_DK1_Flexion_joint_1_v2.STL" scale="1 1 1"/>
+            </geometry>
+        </visual>
+    </link>
+    <!-- ring flexion two -->
+    <link name="ring_flexion_two">
+        <visual>
+            <origin xyz="0 0 ${-bar_length/2}" rpy="0 0 0"/>
+            <geometry>
+                <mesh filename="package://senseglove_description/urdf/STL/MK29_DK1_Flexion_joint_2_v2.STL" scale="1 1 1"/>
+            </geometry>
+        </visual>
+    </link>
+    <!-- ring flexion three -->
+    <link name="ring_flexion_three">
+        <visual>
+            <origin xyz="0 0 ${-bar_length/2}" rpy="0 0 0"/>
+            <geometry>
+                <mesh filename="package://senseglove_description/urdf/STL/MK29_DK1_Flexion_joint_3_v2.STL" scale="1 1 1"/>
+            </geometry>
+        </visual>
+    </link>
+    <!-- ring thimble -->
+    <link name="ring_thimble">
+        <visual>
+            <origin xyz="0 0 ${-bar_length/2}" rpy="0 0 0"/>
+            <geometry>
+                <mesh filename="package://senseglove_description/urdf/STL/MK29_DK1_Thimble_v2.STL" scale="1 1 1"/>
+            </geometry>
+        </visual>
+    </link>
+    <!-- pinky brake -->
+    <link name="pinky_brake">
+        <visual>
+            <origin xyz="0 0 ${-bar_length/2}" rpy="0 0 0"/>
+            <geometry>
+                <mesh filename="package://senseglove_description/urdf/STL/MK29_DK1_Brake_assembly_v2.STL" scale="1 1 1"/>
+            </geometry>
+        </visual>
+    </link>
+    <!-- pinky abduction -->
+    <link name="pinky_abduction">
+        <visual>
+            <origin xyz="0 0 ${-bar_length/2}" rpy="0 0 0"/>
+            <geometry>
+                <mesh filename="package://senseglove_description/urdf/STL/MK29_DK1_Abduction_joint_v2.STL" scale="1 1 1"/>
+            </geometry>
+        </visual>
+    </link>
+    <!-- pinky flexion one -->
+    <link name="pinky_flexion_one">
+        <visual>
+            <origin xyz="0 0 ${-bar_length/2}" rpy="0 0 0"/>
+            <geometry>
+                <mesh filename="package://senseglove_description/urdf/STL/MK29_DK1_Flexion_joint_1_v2.STL" scale="1 1 1"/>
+            </geometry>
+        </visual>
+    </link>
+    <!-- pinky flexion two -->
+    <link name="pinky_flexion_two">
+        <visual>
+            <origin xyz="0 0 ${-bar_length/2}" rpy="0 0 0"/>
+            <geometry>
+                <mesh filename="package://senseglove_description/urdf/STL/MK29_DK1_Flexion_joint_2_v2.STL" scale="1 1 1"/>
+            </geometry>
+        </visual>
+    </link>
+    <!-- pinky flexion three -->
+    <link name="pinky_flexion_three">
+        <visual>
+            <origin xyz="0 0 ${-bar_length/2}" rpy="0 0 0"/>
+            <geometry>
+                <mesh filename="package://senseglove_description/urdf/STL/MK29_DK1_Flexion_joint_3_v2.STL" scale="1 1 1"/>
+            </geometry>
+        </visual>
+    </link>
+    <!-- pinky thimble -->
+    <link name="pinky_thimble">
+        <visual>
+            <origin xyz="0 0 ${-bar_length/2}" rpy="0 0 0"/>
+            <geometry>
+                <mesh filename="package://senseglove_description/urdf/STL/MK29_DK1_Thimble_v2.STL" scale="1 1 1"/>
+            </geometry>
+        </visual>
+    </link>
+    <!-- Joints -->
     <joint name="joint_base_fixed_parent_joint" type="fixed">
         <parent link="world"/>
-        <child link="joint_base"/>
+        <child link="glove_hub"/>
         <origin xyz="0 0 ${hover_height}" rpy="0 0 0"/>
     </joint>
-    <joint name="linear_joint" type="revolute">
-        <parent link="joint_base"/>
-        <child link="bar"/>
-        <origin xyz="0 ${-joint_base_width} 0" rpy="0 0 0"/>
-        <axis xyz="0 1 0"/>
-        <limit velocity="${10}"
-               effort="${10000}"
-               lower="${-5}"
-               upper="${5}"/>
-    </joint>
-    <!-- Joint Base-->
-    <link name="joint_base">
-        <visual>
-            <origin xyz="0 0 0" rpy="0 0 0"/>
-            <geometry>
-                <box size="${joint_base_width} ${joint_base_width} ${joint_base_width}"/>
-            </geometry>
-        </visual>
-        <inertial>
-            <origin xyz="0 0 0" rpy="0 0 0"/>
-            <mass value="${joint_base_mass}"/>
-            <inertia
-                    ixx="${joint_base_mass / 12.0 * (2*(joint_base_width*joint_base_width))}" ixy="0.0" ixz="0.0"
-                    iyy="${joint_base_mass / 12.0 * (2*(joint_base_width*joint_base_width))}" iyz="0.0"
-                    izz="${joint_base_mass / 12.0 * (2*(joint_base_width*joint_base_width))}"/>
-            <!--(joint_base_width*joint_base_width + joint_base_width*joint_base_width)-->
-        </inertial>
-    </link>
-    <!-- Bar-->
-    <link name="bar">
-        <visual>
-            <origin xyz="0 0 ${-bar_length/2}" rpy="0 0 0"/>
-            <geometry>
-                <box size="${bar_width} ${bar_width} ${bar_length}"/>
-            </geometry>
-        </visual>
-        <inertial>
-            <origin xyz="0 0 ${-bar_length/2}" rpy="0 0 0"/>
-            <mass value="${bar_mass}"/>
-            <inertia
-                    ixx="${joint_base_mass / 12.0 * (bar_width*bar_width + bar_length*bar_length)}" ixy="0.0" ixz="0.0"
-                    iyy="${joint_base_mass / 12.0 * (bar_length*bar_length + bar_width*bar_width)}" iyz="0.0"
-                    izz="${joint_base_mass / 12.0 * (bar_width*bar_width + bar_width*bar_width)}"/>
-        </inertial>
-    </link>
+    <joint name="hub_to_thumb_brake" type="fixed">
+        <parent link="glove_hub"/>
+        <child link="thumb_brake"/>
+        <origin xyz="0 ${-joint_base_width} 0" rpy="0 0 0"/>
+    </joint>
+    <joint name="thumb_brake" type="revolute">
+        <parent link="thumb_brake"/>
+        <child link="thumb_abduction"/>
+        <origin xyz="0 0 0" rpy="0 0 0"/>
+        <axis xyz="0 1 0"/>
+        <limit velocity="${1}"
+               effort="${10000}"
+               lower="${-1}"
+               upper="${1}"/>
+    </joint>
+    <joint name="thumb_abduction" type="revolute">
+        <parent link="thumb_abduction"/>
+        <child link="thumb_flexion_one"/>
+        <origin xyz="0 0 0" rpy="0 0 0"/>
+        <axis xyz="0 1 0"/>
+        <limit velocity="${1}"
+               effort="${10000}"
+               lower="${-1}"
+               upper="${1}"/>
+    </joint>
+    <joint name="thumb_cmc" type="revolute">
+        <parent link="thumb_flexion_one"/>
+        <child link="thumb_flexion_two"/>
+        <origin xyz="0 ${-joint_base_width} 0" rpy="0 0 0"/>
+        <axis xyz="0 1 0"/>
+        <limit velocity="${1}"
+               effort="${10000}"
+               lower="${-1}"
+               upper="${1}"/>
+    </joint>
+    <joint name="thumb_mcp" type="revolute">
+        <parent link="thumb_flexion_two"/>
+        <child link="thumb_flexion_three"/>
+        <origin xyz="0 ${-joint_base_width} 0" rpy="0 0 0"/>
+        <axis xyz="0 1 0"/>
+        <limit velocity="${1}"
+               effort="${10000}"
+               lower="${-1}"
+               upper="${1}"/>
+    </joint>
+    <joint name="thumb_pip" type="revolute">
+        <parent link="thumb_flexion_three"/>
+        <child link="thumb_thimble"/>
+        <origin xyz="0 ${-joint_base_width} 0" rpy="0 0 0"/>
+        <axis xyz="0 1 0"/>
+        <limit velocity="${1}"
+               effort="${10000}"
+               lower="${-1}"
+               upper="${1}"/>
+    </joint>
+    <joint name="hub_to_index_brake" type="fixed">
+        <parent link="glove_hub"/>
+        <child link="index_brake"/>
+        <origin xyz="0 ${-joint_base_width} 0" rpy="0 0 0"/>
+    </joint>
+    <joint name="index_brake" type="revolute">
+        <parent link="index_brake"/>
+        <child link="index_abduction"/>
+        <origin xyz="0 0 0" rpy="0 0 0"/>
+        <axis xyz="0 1 0"/>
+        <limit velocity="${1}"
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