Commit message: correct the hub xyz coordinates for the brakes, correct the origins for the brakes and the origins for the abduction joints.

File: src/senseglove/senseglove_description/urdf/dk1.xacro (robot description, xacro)
@@ -6,4 +6,27 @@
     <xacro:property name="joint_base_mass" value="1"/> <!-- arbitrary value for joint_base_mass -->
     <xacro:property name="joint_base_width" value="0.05"/> <!-- Cube dimensions (width x width x width) of joint base -->
+    <!-- Bar lengths -->
+    <xacro:property name="brake_length" value="0.0418"/>
+    <xacro:property name="brake_thickness" value="0.022"/>
+    <xacro:property name="brake_height" value="0.0308"/>
+    <xacro:property name="first_bar_length" value="0.026"/>
+    <xacro:property name="second_bar_length" value="0.0876"/>
+    <xacro:property name="third_bar_length" value="0.0664"/>
+    <!-- Origins on hub for fingers -->
+    <xacro:property name="thumb_hub_X" value="0.02"/>
+    <xacro:property name="thumb_hub_Y" value="0.03"/>
+    <xacro:property name="thumb_hub_Z" value="0.105"/>
+    <xacro:property name="index_hub_X" value="${0.0125+brake_thickness/2}"/>
+    <xacro:property name="index_hub_Y" value="${0.0+brake_height/2}"/>
+    <xacro:property name="index_hub_Z" value="${-0.0945+first_bar_length+second_bar_length+brake_length}"/>
+    <xacro:property name="middle_hub_X" value="${0.035+brake_thickness/2}"/>
+    <xacro:property name="middle_hub_Y" value="${0.0+brake_height/2}"/>
+    <xacro:property name="middle_hub_Z" value="${-0.112+first_bar_length+second_bar_length+brake_length}"/>
+    <xacro:property name="ring_hub_X" value="${0.057+brake_thickness/2}"/>
+    <xacro:property name="ring_hub_Y" value="${0.0+brake_height/2}"/>
+    <xacro:property name="ring_hub_Z" value="${-0.102+first_bar_length+second_bar_length+brake_length}"/>
+    <xacro:property name="pinky_hub_X" value="${0.079+brake_thickness/2}"/>
+    <xacro:property name="pinky_hub_Y" value="${0.0+brake_height/2}"/>
+    <xacro:property name="pinky_hub_Z" value="${-0.09+first_bar_length+second_bar_length+brake_length}"/>
     <xacro:property name="bar_length" value="${0.39}"/>
     <xacro:property name="bar_mass" value="1.080"/>
@@ -16,5 +39,5 @@
     <xacro:property name="hover_height" value="0.5"/>
     <!-- Used for fixing robot to Gazebo 'base_link' -->
-    <link name="world"/>
+    <link name="base_link"/>
     <!-- glove hub -->
     <link name="glove_hub">
@@ -22,5 +45,5 @@
             <origin xyz="0 0 0" rpy="0 0 0"/>
             <geometry>
-                <mesh filename="package://senseglove_description/urdf/STL/MK29_DK1_HUB.STL" scale="1 1 1"/>
+                <mesh filename="package://senseglove_description/urdf/STL/MK29_DK1_HUB.STL" scale="0.001 0.001 0.001"/>
             </geometry>
         </visual>
@@ -29,7 +52,7 @@
     <link name="thumb_brake">
         <visual>
-            <origin xyz="0 0 ${-bar_length/2}" rpy="0 0 0"/>
-            <geometry>
-                <mesh filename="package://senseglove_description/urdf/STL/MK29_DK1_Brake_assembly_v2.STL" scale="1 1 1"/>
+            <origin xyz="${-brake_thickness/2} ${-brake_height/2} ${-first_bar_length-second_bar_length-brake_length}" rpy="0 0 0"/>
+            <geometry>
+                <mesh filename="package://senseglove_description/urdf/STL/MK29_DK1_Brake_assembly_v2.STL" scale="0.001 0.001 0.001"/>
             </geometry>
         </visual>
@@ -38,7 +61,7 @@
     <link name="thumb_abduction">
         <visual>
-            <origin xyz="0 0 ${-bar_length/2}" rpy="0 0 0"/>
-            <geometry>
-                <mesh filename="package://senseglove_description/urdf/STL/MK29_DK1_Abduction_joint_v2.STL" scale="1 1 1"/>
+            <origin xyz="${-brake_thickness/2} ${-brake_height+0.006} ${-second_bar_length-first_bar_length}" rpy="0 0 0"/>
+            <geometry>
+                <mesh filename="package://senseglove_description/urdf/STL/MK29_DK1_Abduction_joint_v2.STL" scale="0.001 0.001 0.001"/>
             </geometry>
         </visual>
@@ -47,7 +70,7 @@
     <link name="thumb_flexion_one">
         <visual>
-            <origin xyz="0 0 ${-bar_length/2}" rpy="0 0 0"/>
-            <geometry>
-                <mesh filename="package://senseglove_description/urdf/STL/MK29_DK1_Flexion_joint_1_v2.STL" scale="1 1 1"/>
+            <origin xyz="0 0 0" rpy="0 0 0"/>
+            <geometry>
+                <mesh filename="package://senseglove_description/urdf/STL/MK29_DK1_Flexion_joint_1_v2.STL" scale="0.001 0.001 0.001"/>
             </geometry>
         </visual>
@@ -56,7 +79,7 @@
     <link name="thumb_flexion_two">
         <visual>
-            <origin xyz="0 0 ${-bar_length/2}" rpy="0 0 0"/>
-            <geometry>
-                <mesh filename="package://senseglove_description/urdf/STL/MK29_DK1_Flexion_joint_2_v2.STL" scale="1 1 1"/>
+            <origin xyz="0 0 ${-first_bar_length}" rpy="0 0 0"/>
+            <geometry>
+                <mesh filename="package://senseglove_description/urdf/STL/MK29_DK1_Flexion_joint_2_v2.STL" scale="0.001 0.001 0.001"/>
             </geometry>
         </visual>
@@ -65,7 +88,7 @@
     <link name="thumb_flexion_three">
         <visual>
-            <origin xyz="0 0 ${-bar_length/2}" rpy="0 0 0"/>
-            <geometry>
-                <mesh filename="package://senseglove_description/urdf/STL/MK29_DK1_Flexion_joint_3_v2.STL" scale="1 1 1"/>
+            <origin xyz="0 0 0" rpy="0 0 0"/>
+            <geometry>
+                <mesh filename="package://senseglove_description/urdf/STL/MK29_DK1_Flexion_joint_3_v2.STL" scale="0.001 0.001 0.001"/>
             </geometry>
         </visual>
@@ -74,7 +97,7 @@
     <link name="thumb_thimble">
         <visual>
-            <origin xyz="0 0 ${-bar_length/2}" rpy="0 0 0"/>
-            <geometry>
-                <mesh filename="package://senseglove_description/urdf/STL/MK29_DK1_Thimble_v2.STL" scale="1 1 1"/>
+            <origin xyz="0 0 ${-third_bar_length}" rpy="0 0 0"/>
+            <geometry>
+                <mesh filename="package://senseglove_description/urdf/STL/MK29_DK1_Thimble_v2.STL" scale="0.001 0.001 0.001"/>
             </geometry>
         </visual>
@@ -83,7 +106,7 @@
     <link name="index_brake">
         <visual>
-            <origin xyz="0 0 ${-bar_length/2}" rpy="0 0 0"/>
-            <geometry>
-                <mesh filename="package://senseglove_description/urdf/STL/MK29_DK1_Brake_assembly_v2.STL" scale="1 1 1"/>
+            <origin xyz="${-brake_thickness/2} ${-brake_height/2} ${-first_bar_length-second_bar_length-brake_length}" rpy="0 0 0"/>
+            <geometry>
+                <mesh filename="package://senseglove_description/urdf/STL/MK29_DK1_Brake_assembly_v2.STL" scale="0.001 0.001 0.001"/>
             </geometry>
         </visual>
@@ -92,7 +115,7 @@
     <link name="index_abduction">
         <visual>
-            <origin xyz="0 0 ${-bar_length/2}" rpy="0 0 0"/>
-            <geometry>
-                <mesh filename="package://senseglove_description/urdf/STL/MK29_DK1_Abduction_joint_v2.STL" scale="1 1 1"/>
+            <origin xyz="${-brake_thickness/2} ${-brake_height+0.006} ${-second_bar_length-first_bar_length}" rpy="0 0 0"/>
+            <geometry>
+                <mesh filename="package://senseglove_description/urdf/STL/MK29_DK1_Abduction_joint_v2.STL" scale="0.001 0.001 0.001"/>
             </geometry>
         </visual>
@@ -101,7 +124,7 @@
     <link name="index_flexion_one">
         <visual>
-            <origin xyz="0 0 ${-bar_length/2}" rpy="0 0 0"/>
-            <geometry>
-                <mesh filename="package://senseglove_description/urdf/STL/MK29_DK1_Flexion_joint_1_v2.STL" scale="1 1 1"/>
+            <origin xyz="0 0 0" rpy="0 0 0"/>
+            <geometry>
+                <mesh filename="package://senseglove_description/urdf/STL/MK29_DK1_Flexion_joint_1_v2.STL" scale="0.001 0.001 0.001"/>
             </geometry>
         </visual>
@@ -110,7 +133,7 @@
     <link name="index_flexion_two">
         <visual>
-            <origin xyz="0 0 ${-bar_length/2}" rpy="0 0 0"/>
-            <geometry>
-                <mesh filename="package://senseglove_description/urdf/STL/MK29_DK1_Flexion_joint_2_v2.STL" scale="1 1 1"/>
+            <origin xyz="0 0 ${-first_bar_length}" rpy="0 0 0"/>
+            <geometry>
+                <mesh filename="package://senseglove_description/urdf/STL/MK29_DK1_Flexion_joint_2_v2.STL" scale="0.001 0.001 0.001"/>
             </geometry>
         </visual>
@@ -119,7 +142,7 @@
     <link name="index_flexion_three">
         <visual>
-            <origin xyz="0 0 ${-bar_length/2}" rpy="0 0 0"/>
-            <geometry>
-                <mesh filename="package://senseglove_description/urdf/STL/MK29_DK1_Flexion_joint_3_v2.STL" scale="1 1 1"/>
+            <origin xyz="0 0 0" rpy="0 0 0"/>
+            <geometry>
+                <mesh filename="package://senseglove_description/urdf/STL/MK29_DK1_Flexion_joint_3_v2.STL" scale="0.001 0.001 0.001"/>
             </geometry>
         </visual>
@@ -128,7 +151,7 @@
     <link name="index_thimble">
         <visual>
-            <origin xyz="0 0 ${-bar_length/2}" rpy="0 0 0"/>
-            <geometry>
-                <mesh filename="package://senseglove_description/urdf/STL/MK29_DK1_Thimble_v2.STL" scale="1 1 1"/>
+            <origin xyz="0 0 ${-third_bar_length}" rpy="0 0 0"/>
+            <geometry>
+                <mesh filename="package://senseglove_description/urdf/STL/MK29_DK1_Thimble_v2.STL" scale="0.001 0.001 0.001"/>
             </geometry>
         </visual>
@@ -137,7 +160,7 @@
     <link name="middle_brake">
         <visual>
-            <origin xyz="0 0 ${-bar_length/2}" rpy="0 0 0"/>
-            <geometry>
-                <mesh filename="package://senseglove_description/urdf/STL/MK29_DK1_Brake_assembly_v2.STL" scale="1 1 1"/>
+            <origin xyz="${-brake_thickness/2} ${-brake_height/2} ${-first_bar_length-second_bar_length-brake_length}" rpy="0 0 0"/>
+            <geometry>
+                <mesh filename="package://senseglove_description/urdf/STL/MK29_DK1_Brake_assembly_v2.STL" scale="0.001 0.001 0.001"/>
             </geometry>
         </visual>
@@ -146,7 +169,7 @@
     <link name="middle_abduction">
         <visual>
-            <origin xyz="0 0 ${-bar_length/2}" rpy="0 0 0"/>
-            <geometry>
-                <mesh filename="package://senseglove_description/urdf/STL/MK29_DK1_Abduction_joint_v2.STL" scale="1 1 1"/>
+            <origin xyz="${-brake_thickness/2} ${-brake_height+0.006} ${-second_bar_length-first_bar_length}" rpy="0 0 0"/>
+            <geometry>
+                <mesh filename="package://senseglove_description/urdf/STL/MK29_DK1_Abduction_joint_v2.STL" scale="0.001 0.001 0.001"/>
             </geometry>
         </visual>
@@ -155,7 +178,7 @@
     <link name="middle_flexion_one">
         <visual>
-            <origin xyz="0 0 ${-bar_length/2}" rpy="0 0 0"/>
-            <geometry>
-                <mesh filename="package://senseglove_description/urdf/STL/MK29_DK1_Flexion_joint_1_v2.STL" scale="1 1 1"/>
+            <origin xyz="0 0 0" rpy="0 0 0"/>
+            <geometry>
+                <mesh filename="package://senseglove_description/urdf/STL/MK29_DK1_Flexion_joint_1_v2.STL" scale="0.001 0.001 0.001"/>
             </geometry>
         </visual>
@@ -164,7 +187,7 @@
     <link name="middle_flexion_two">
         <visual>
-            <origin xyz="0 0 ${-bar_length/2}" rpy="0 0 0"/>
-            <geometry>
-                <mesh filename="package://senseglove_description/urdf/STL/MK29_DK1_Flexion_joint_2_v2.STL" scale="1 1 1"/>
+            <origin xyz="0 0 ${-first_bar_length}" rpy="0 0 0"/>
+            <geometry>
+                <mesh filename="package://senseglove_description/urdf/STL/MK29_DK1_Flexion_joint_2_v2.STL" scale="0.001 0.001 0.001"/>
             </geometry>
         </visual>
@@ -173,7 +196,7 @@
     <link name="middle_flexion_three">
         <visual>
-            <origin xyz="0 0 ${-bar_length/2}" rpy="0 0 0"/>
-            <geometry>
-                <mesh filename="package://senseglove_description/urdf/STL/MK29_DK1_Flexion_joint_3_v2.STL" scale="1 1 1"/>
+            <origin xyz="0 0 0" rpy="0 0 0"/>
+            <geometry>
+                <mesh filename="package://senseglove_description/urdf/STL/MK29_DK1_Flexion_joint_3_v2.STL" scale="0.001 0.001 0.001"/>
             </geometry>
         </visual>
@@ -182,7 +205,7 @@
     <link name="middle_thimble">
         <visual>
-            <origin xyz="0 0 ${-bar_length/2}" rpy="0 0 0"/>
-            <geometry>
-                <mesh filename="package://senseglove_description/urdf/STL/MK29_DK1_Thimble_v2.STL" scale="1 1 1"/>
+            <origin xyz="0 0 ${-third_bar_length}" rpy="0 0 0"/>
+            <geometry>
+                <mesh filename="package://senseglove_description/urdf/STL/MK29_DK1_Thimble_v2.STL" scale="0.001 0.001 0.001"/>
             </geometry>
         </visual>
@@ -191,7 +214,7 @@
     <link name="ring_brake">
         <visual>
-            <origin xyz="0 0 ${-bar_length/2}" rpy="0 0 0"/>
-            <geometry>
-                <mesh filename="package://senseglove_description/urdf/STL/MK29_DK1_Brake_assembly_v2.STL" scale="1 1 1"/>
+            <origin xyz="${-brake_thickness/2} ${-brake_height/2} ${-first_bar_length-second_bar_length-brake_length}" rpy="0 0 0"/>
+            <geometry>
+                <mesh filename="package://senseglove_description/urdf/STL/MK29_DK1_Brake_assembly_v2.STL" scale="0.001 0.001 0.001"/>
             </geometry>
         </visual>
@@ -200,7 +223,7 @@
     <link name="ring_abduction">
         <visual>
-            <origin xyz="0 0 ${-bar_length/2}" rpy="0 0 0"/>
-            <geometry>
-                <mesh filename="package://senseglove_description/urdf/STL/MK29_DK1_Abduction_joint_v2.STL" scale="1 1 1"/>
+            <origin xyz="${-brake_thickness/2} ${-brake_height+0.006} ${-second_bar_length-first_bar_length}" rpy="0 0 0"/>
+            <geometry>
+                <mesh filename="package://senseglove_description/urdf/STL/MK29_DK1_Abduction_joint_v2.STL" scale="0.001 0.001 0.001"/>
             </geometry>
         </visual>
@@ -209,7 +232,7 @@
     <link name="ring_flexion_one">
         <visual>
-            <origin xyz="0 0 ${-bar_length/2}" rpy="0 0 0"/>
-            <geometry>
-                <mesh filename="package://senseglove_description/urdf/STL/MK29_DK1_Flexion_joint_1_v2.STL" scale="1 1 1"/>
+            <origin xyz="0 0 0" rpy="0 0 0"/>
+            <geometry>
+                <mesh filename="package://senseglove_description/urdf/STL/MK29_DK1_Flexion_joint_1_v2.STL" scale="0.001 0.001 0.001"/>
             </geometry>
         </visual>
@@ -218,7 +241,7 @@
     <link name="ring_flexion_two">
         <visual>
-            <origin xyz="0 0 ${-bar_length/2}" rpy="0 0 0"/>
-            <geometry>
-                <mesh filename="package://senseglove_description/urdf/STL/MK29_DK1_Flexion_joint_2_v2.STL" scale="1 1 1"/>
+            <origin xyz="0 0 ${-first_bar_length}" rpy="0 0 0"/>
+            <geometry>
+                <mesh filename="package://senseglove_description/urdf/STL/MK29_DK1_Flexion_joint_2_v2.STL" scale="0.001 0.001 0.001"/>
             </geometry>
         </visual>
@@ -227,7 +250,7 @@
     <link name="ring_flexion_three">
         <visual>
-            <origin xyz="0 0 ${-bar_length/2}" rpy="0 0 0"/>
-            <geometry>
-                <mesh filename="package://senseglove_description/urdf/STL/MK29_DK1_Flexion_joint_3_v2.STL" scale="1 1 1"/>
+            <origin xyz="0 0 0" rpy="0 0 0"/>
+            <geometry>
+                <mesh filename="package://senseglove_description/urdf/STL/MK29_DK1_Flexion_joint_3_v2.STL" scale="0.001 0.001 0.001"/>
             </geometry>
         </visual>
@@ -236,7 +259,7 @@
     <link name="ring_thimble">
         <visual>
-            <origin xyz="0 0 ${-bar_length/2}" rpy="0 0 0"/>
-            <geometry>
-                <mesh filename="package://senseglove_description/urdf/STL/MK29_DK1_Thimble_v2.STL" scale="1 1 1"/>
+            <origin xyz="0 0 ${-third_bar_length}" rpy="0 0 0"/>
+            <geometry>
+                <mesh filename="package://senseglove_description/urdf/STL/MK29_DK1_Thimble_v2.STL" scale="0.001 0.001 0.001"/>
             </geometry>
         </visual>
@@ -245,7 +268,7 @@
     <link name="pinky_brake">
         <visual>
-            <origin xyz="0 0 ${-bar_length/2}" rpy="0 0 0"/>
-            <geometry>
-                <mesh filename="package://senseglove_description/urdf/STL/MK29_DK1_Brake_assembly_v2.STL" scale="1 1 1"/>
+            <origin xyz="${-brake_thickness/2} ${-brake_height/2} ${-first_bar_length-second_bar_length-brake_length}" rpy="0 0 0"/>
+            <geometry>
+                <mesh filename="package://senseglove_description/urdf/STL/MK29_DK1_Brake_assembly_v2.STL" scale="0.001 0.001 0.001"/>
             </geometry>
         </visual>
@@ -254,7 +277,7 @@
     <link name="pinky_abduction">
         <visual>
-            <origin xyz="0 0 ${-bar_length/2}" rpy="0 0 0"/>
-            <geometry>
-                <mesh filename="package://senseglove_description/urdf/STL/MK29_DK1_Abduction_joint_v2.STL" scale="1 1 1"/>
+            <origin xyz="${-brake_thickness/2} ${-brake_height+0.006} ${-second_bar_length-first_bar_length}" rpy="0 0 0"/>
+            <geometry>
+                <mesh filename="package://senseglove_description/urdf/STL/MK29_DK1_Abduction_joint_v2.STL" scale="0.001 0.001 0.001"/>
             </geometry>
         </visual>
@@ -263,7 +286,7 @@
     <link name="pinky_flexion_one">
         <visual>
-            <origin xyz="0 0 ${-bar_length/2}" rpy="0 0 0"/>
-            <geometry>
-                <mesh filename="package://senseglove_description/urdf/STL/MK29_DK1_Flexion_joint_1_v2.STL" scale="1 1 1"/>
+            <origin xyz="0 0 0" rpy="0 0 0"/>
+            <geometry>
+                <mesh filename="package://senseglove_description/urdf/STL/MK29_DK1_Flexion_joint_1_v2.STL" scale="0.001 0.001 0.001"/>
             </geometry>
         </visual>
@@ -272,7 +295,7 @@
     <link name="pinky_flexion_two">
         <visual>
-            <origin xyz="0 0 ${-bar_length/2}" rpy="0 0 0"/>
-            <geometry>
-                <mesh filename="package://senseglove_description/urdf/STL/MK29_DK1_Flexion_joint_2_v2.STL" scale="1 1 1"/>
+            <origin xyz="0 0 ${-first_bar_length}" rpy="0 0 0"/>
+            <geometry>
+                <mesh filename="package://senseglove_description/urdf/STL/MK29_DK1_Flexion_joint_2_v2.STL" scale="0.001 0.001 0.001"/>
             </geometry>
         </visual>
@@ -281,7 +304,7 @@
     <link name="pinky_flexion_three">
         <visual>
-            <origin xyz="0 0 ${-bar_length/2}" rpy="0 0 0"/>
-            <geometry>
-                <mesh filename="package://senseglove_description/urdf/STL/MK29_DK1_Flexion_joint_3_v2.STL" scale="1 1 1"/>
+            <origin xyz="0 0 0" rpy="0 0 0"/>
+            <geometry>
+                <mesh filename="package://senseglove_description/urdf/STL/MK29_DK1_Flexion_joint_3_v2.STL" scale="0.001 0.001 0.001"/>
             </geometry>
         </visual>
@@ -290,7 +313,7 @@
     <link name="pinky_thimble">
         <visual>
-            <origin xyz="0 0 ${-bar_length/2}" rpy="0 0 0"/>
-            <geometry>
-                <mesh filename="package://senseglove_description/urdf/STL/MK29_DK1_Thimble_v2.STL" scale="1 1 1"/>
+            <origin xyz="0 0 ${-third_bar_length}" rpy="0 0 0"/>
+            <geometry>
+                <mesh filename="package://senseglove_description/urdf/STL/MK29_DK1_Thimble_v2.STL" scale="0.001 0.001 0.001"/>
             </geometry>
         </visual>
@@ -298,5 +321,5 @@
     <!-- Joints -->
     <joint name="joint_base_fixed_parent_joint" type="fixed">
-        <parent link="world"/>
+        <parent link="base_link"/>
         <child link="glove_hub"/>
         <origin xyz="0 0 ${hover_height}" rpy="0 0 0"/>
@@ -305,5 +328,5 @@
         <parent link="glove_hub"/>
         <child link="thumb_brake"/>
-        <origin xyz="0 ${-joint_base_width} 0" rpy="0 0 0"/>
+        <origin xyz="${thumb_hub_X} ${thumb_hub_Y} ${thumb_hub_Z}" rpy="${105*PI/180} ${40*PI/180} ${170.0*PI/180.0}"/>
     </joint>
     <joint name="thumb_brake" type="revolute">
@@ -330,6 +353,6 @@
         <parent link="thumb_flexion_one"/>
         <child link="thumb_flexion_two"/>
-        <origin xyz="0 ${-joint_base_width} 0" rpy="0 0 0"/>
-        <axis xyz="0 1 0"/>
+        <origin xyz="0 0 ${first_bar_length}" rpy="0 0 0"/>
+        <axis xyz="1 0 0"/>
         <limit velocity="${1}"
                effort="${10000}"
@@ -340,6 +363,6 @@
         <parent link="thumb_flexion_two"/>
         <child link="thumb_flexion_three"/>
-        <origin xyz="0 ${-joint_base_width} 0" rpy="0 0 0"/>
-        <axis xyz="0 1 0"/>
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