Commit message: Correct the origins of the stls and joint frames

File: src/senseglove/senseglove_description/urdf/dk1.xacro (robot description, xacro)
@@ -8,25 +8,25 @@
     <!-- Bar lengths -->
     <xacro:property name="brake_length" value="0.0418"/>
-    <xacro:property name="brake_thickness" value="0.022"/>
-    <xacro:property name="brake_height" value="0.0308"/>
+    <xacro:property name="brake_thickness" value="0.022279"/>
+    <xacro:property name="brake_height" value="0.0313"/>
     <xacro:property name="first_bar_length" value="0.026"/>
     <xacro:property name="second_bar_length" value="0.0876"/>
     <xacro:property name="third_bar_length" value="0.0664"/>
     <!-- Origins on hub for fingers -->
-    <xacro:property name="thumb_hub_X" value="0.02"/>
-    <xacro:property name="thumb_hub_Y" value="0.03"/>
-    <xacro:property name="thumb_hub_Z" value="0.105"/>
-    <xacro:property name="index_hub_X" value="${0.0125+brake_thickness/2}"/>
-    <xacro:property name="index_hub_Y" value="${0.0+brake_height/2}"/>
-    <xacro:property name="index_hub_Z" value="${-0.0945+first_bar_length+second_bar_length+brake_length}"/>
-    <xacro:property name="middle_hub_X" value="${0.035+brake_thickness/2}"/>
-    <xacro:property name="middle_hub_Y" value="${0.0+brake_height/2}"/>
-    <xacro:property name="middle_hub_Z" value="${-0.112+first_bar_length+second_bar_length+brake_length}"/>
-    <xacro:property name="ring_hub_X" value="${0.057+brake_thickness/2}"/>
-    <xacro:property name="ring_hub_Y" value="${0.0+brake_height/2}"/>
-    <xacro:property name="ring_hub_Z" value="${-0.102+first_bar_length+second_bar_length+brake_length}"/>
-    <xacro:property name="pinky_hub_X" value="${0.079+brake_thickness/2}"/>
-    <xacro:property name="pinky_hub_Y" value="${0.0+brake_height/2}"/>
-    <xacro:property name="pinky_hub_Z" value="${-0.09+first_bar_length+second_bar_length+brake_length}"/>
+    <xacro:property name="thumb_hub_X" value="-0.052034"/>
+    <xacro:property name="thumb_hub_Y" value="-0.0221293"/>
+    <xacro:property name="thumb_hub_Z" value="0.04656"/>
+    <xacro:property name="index_hub_X" value="-0.03309"/>
+    <xacro:property name="index_hub_Y" value="0.00645"/>
+    <xacro:property name="index_hub_Z" value="-0.04436"/>
+    <xacro:property name="middle_hub_X" value="-0.011"/>
+    <xacro:property name="middle_hub_Y" value="0.008"/>
+    <xacro:property name="middle_hub_Z" value="-0.06222"/>
+    <xacro:property name="ring_hub_X" value="0.011"/>
+    <xacro:property name="ring_hub_Y" value="0.008"/>
+    <xacro:property name="ring_hub_Z" value="-0.05422"/>
+    <xacro:property name="pinky_hub_X" value="0.03307"/>
+    <xacro:property name="pinky_hub_Y" value="0.00695"/>
+    <xacro:property name="pinky_hub_Z" value="-0.04125"/>
     <xacro:property name="bar_length" value="${0.39}"/>
     <xacro:property name="bar_mass" value="1.080"/>
@@ -43,5 +43,5 @@
     <link name="glove_hub">
         <visual>
-            <origin xyz="0 0 0" rpy="0 0 0"/>
+            <origin xyz="-0.056692 -0.01955 -0.06803" rpy="0 0 0"/>
             <geometry>
                 <mesh filename="package://senseglove_description/urdf/STL/MK29_DK1_HUB.STL" scale="0.001 0.001 0.001"/>
@@ -52,5 +52,5 @@
     <link name="thumb_brake">
         <visual>
-            <origin xyz="${-brake_thickness/2} ${-brake_height/2} ${-first_bar_length-second_bar_length-brake_length}" rpy="0 0 0"/>
+            <origin xyz="${-brake_thickness/2} ${-brake_height/2 - 0.0025} ${-first_bar_length-second_bar_length}" rpy="0 0 0"/>
             <geometry>
                 <mesh filename="package://senseglove_description/urdf/STL/MK29_DK1_Brake_assembly_v2.STL" scale="0.001 0.001 0.001"/>
@@ -61,5 +61,5 @@
     <link name="thumb_abduction">
         <visual>
-            <origin xyz="${-brake_thickness/2} ${-brake_height+0.006} ${-second_bar_length-first_bar_length}" rpy="0 0 0"/>
+            <origin xyz="${-brake_thickness/2} ${-brake_height+0.006} ${-second_bar_length-first_bar_length-0.003}" rpy="0 0 0"/>
             <geometry>
                 <mesh filename="package://senseglove_description/urdf/STL/MK29_DK1_Abduction_joint_v2.STL" scale="0.001 0.001 0.001"/>
@@ -70,5 +70,5 @@
     <link name="thumb_flexion_one">
         <visual>
-            <origin xyz="0 0 0" rpy="0 0 0"/>
+            <origin xyz="${-brake_thickness/2} ${-brake_height+0.005} ${-second_bar_length-0.0055}" rpy="0 0 0"/>
             <geometry>
                 <mesh filename="package://senseglove_description/urdf/STL/MK29_DK1_Flexion_joint_1_v2.STL" scale="0.001 0.001 0.001"/>
@@ -79,5 +79,5 @@
     <link name="thumb_flexion_two">
         <visual>
-            <origin xyz="0 0 ${-first_bar_length}" rpy="0 0 0"/>
+            <origin xyz="${-brake_thickness/2} ${-brake_height+0.005} ${-second_bar_length-0.005355}" rpy="0 0 0"/>
             <geometry>
                 <mesh filename="package://senseglove_description/urdf/STL/MK29_DK1_Flexion_joint_2_v2.STL" scale="0.001 0.001 0.001"/>
@@ -88,5 +88,5 @@
     <link name="thumb_flexion_three">
         <visual>
-            <origin xyz="0 0 0" rpy="0 0 0"/>
+            <origin xyz="${-brake_thickness/2} ${-brake_height+0.00533} -0.00533" rpy="0 0 0"/>
             <geometry>
                 <mesh filename="package://senseglove_description/urdf/STL/MK29_DK1_Flexion_joint_3_v2.STL" scale="0.001 0.001 0.001"/>
@@ -97,5 +97,5 @@
     <link name="thumb_thimble">
         <visual>
-            <origin xyz="0 0 ${-third_bar_length}" rpy="0 0 0"/>
+            <origin xyz="${-brake_thickness/2} -0.014951 ${-third_bar_length-0.0028}" rpy="0 0 0"/>
             <geometry>
                 <mesh filename="package://senseglove_description/urdf/STL/MK29_DK1_Thimble_v2.STL" scale="0.001 0.001 0.001"/>
@@ -106,5 +106,5 @@
     <link name="index_brake">
         <visual>
-            <origin xyz="${-brake_thickness/2} ${-brake_height/2} ${-first_bar_length-second_bar_length-brake_length}" rpy="0 0 0"/>
+            <origin xyz="${-brake_thickness/2} ${-brake_height/2 - 0.0025} ${-first_bar_length-second_bar_length}" rpy="0 0 0"/>
             <geometry>
                 <mesh filename="package://senseglove_description/urdf/STL/MK29_DK1_Brake_assembly_v2.STL" scale="0.001 0.001 0.001"/>
@@ -115,5 +115,5 @@
     <link name="index_abduction">
         <visual>
-            <origin xyz="${-brake_thickness/2} ${-brake_height+0.006} ${-second_bar_length-first_bar_length}" rpy="0 0 0"/>
+            <origin xyz="${-brake_thickness/2} ${-brake_height+0.006} ${-second_bar_length-first_bar_length-0.003}" rpy="0 0 0"/>
             <geometry>
                 <mesh filename="package://senseglove_description/urdf/STL/MK29_DK1_Abduction_joint_v2.STL" scale="0.001 0.001 0.001"/>
@@ -124,5 +124,5 @@
     <link name="index_flexion_one">
         <visual>
-            <origin xyz="0 0 0" rpy="0 0 0"/>
+            <origin xyz="${-brake_thickness/2} ${-brake_height+0.005} ${-second_bar_length-0.0055}" rpy="0 0 0"/>
             <geometry>
                 <mesh filename="package://senseglove_description/urdf/STL/MK29_DK1_Flexion_joint_1_v2.STL" scale="0.001 0.001 0.001"/>
@@ -133,5 +133,5 @@
     <link name="index_flexion_two">
         <visual>
-            <origin xyz="0 0 ${-first_bar_length}" rpy="0 0 0"/>
+            <origin xyz="${-brake_thickness/2} ${-brake_height+0.005} ${-second_bar_length-0.005355}" rpy="0 0 0"/>
             <geometry>
                 <mesh filename="package://senseglove_description/urdf/STL/MK29_DK1_Flexion_joint_2_v2.STL" scale="0.001 0.001 0.001"/>
@@ -142,5 +142,5 @@
     <link name="index_flexion_three">
         <visual>
-            <origin xyz="0 0 0" rpy="0 0 0"/>
+            <origin xyz="${-brake_thickness/2} ${-brake_height+0.00533} -0.00533" rpy="0 0 0"/>
             <geometry>
                 <mesh filename="package://senseglove_description/urdf/STL/MK29_DK1_Flexion_joint_3_v2.STL" scale="0.001 0.001 0.001"/>
@@ -151,5 +151,5 @@
     <link name="index_thimble">
         <visual>
-            <origin xyz="0 0 ${-third_bar_length}" rpy="0 0 0"/>
+            <origin xyz="${-brake_thickness/2} -0.014951 ${-third_bar_length-0.0028}" rpy="0 0 0"/>
             <geometry>
                 <mesh filename="package://senseglove_description/urdf/STL/MK29_DK1_Thimble_v2.STL" scale="0.001 0.001 0.001"/>
@@ -160,5 +160,5 @@
     <link name="middle_brake">
         <visual>
-            <origin xyz="${-brake_thickness/2} ${-brake_height/2} ${-first_bar_length-second_bar_length-brake_length}" rpy="0 0 0"/>
+            <origin xyz="${-brake_thickness/2} ${-brake_height/2 - 0.0025} ${-first_bar_length-second_bar_length}" rpy="0 0 0"/>
             <geometry>
                 <mesh filename="package://senseglove_description/urdf/STL/MK29_DK1_Brake_assembly_v2.STL" scale="0.001 0.001 0.001"/>
@@ -169,5 +169,5 @@
     <link name="middle_abduction">
         <visual>
-            <origin xyz="${-brake_thickness/2} ${-brake_height+0.006} ${-second_bar_length-first_bar_length}" rpy="0 0 0"/>
+            <origin xyz="${-brake_thickness/2} ${-brake_height+0.006} ${-second_bar_length-first_bar_length-0.003}" rpy="0 0 0"/>
             <geometry>
                 <mesh filename="package://senseglove_description/urdf/STL/MK29_DK1_Abduction_joint_v2.STL" scale="0.001 0.001 0.001"/>
@@ -178,5 +178,5 @@
     <link name="middle_flexion_one">
         <visual>
-            <origin xyz="0 0 0" rpy="0 0 0"/>
+            <origin xyz="${-brake_thickness/2} ${-brake_height+0.005} ${-second_bar_length-0.0055}" rpy="0 0 0"/>
             <geometry>
                 <mesh filename="package://senseglove_description/urdf/STL/MK29_DK1_Flexion_joint_1_v2.STL" scale="0.001 0.001 0.001"/>
@@ -187,5 +187,5 @@
     <link name="middle_flexion_two">
         <visual>
-            <origin xyz="0 0 ${-first_bar_length}" rpy="0 0 0"/>
+            <origin xyz="${-brake_thickness/2} ${-brake_height+0.005} ${-second_bar_length-0.005355}" rpy="0 0 0"/>
             <geometry>
                 <mesh filename="package://senseglove_description/urdf/STL/MK29_DK1_Flexion_joint_2_v2.STL" scale="0.001 0.001 0.001"/>
@@ -196,5 +196,5 @@
     <link name="middle_flexion_three">
         <visual>
-            <origin xyz="0 0 0" rpy="0 0 0"/>
+            <origin xyz="${-brake_thickness/2} ${-brake_height+0.00533} -0.00533" rpy="0 0 0"/>
             <geometry>
                 <mesh filename="package://senseglove_description/urdf/STL/MK29_DK1_Flexion_joint_3_v2.STL" scale="0.001 0.001 0.001"/>
@@ -205,5 +205,5 @@
     <link name="middle_thimble">
         <visual>
-            <origin xyz="0 0 ${-third_bar_length}" rpy="0 0 0"/>
+            <origin xyz="${-brake_thickness/2} -0.014951 ${-third_bar_length-0.0028}" rpy="0 0 0"/>
             <geometry>
                 <mesh filename="package://senseglove_description/urdf/STL/MK29_DK1_Thimble_v2.STL" scale="0.001 0.001 0.001"/>
@@ -214,5 +214,5 @@
     <link name="ring_brake">
         <visual>
-            <origin xyz="${-brake_thickness/2} ${-brake_height/2} ${-first_bar_length-second_bar_length-brake_length}" rpy="0 0 0"/>
+            <origin xyz="${-brake_thickness/2} ${-brake_height/2 - 0.0025} ${-first_bar_length-second_bar_length}" rpy="0 0 0"/>
             <geometry>
                 <mesh filename="package://senseglove_description/urdf/STL/MK29_DK1_Brake_assembly_v2.STL" scale="0.001 0.001 0.001"/>
@@ -223,5 +223,5 @@
     <link name="ring_abduction">
         <visual>
-            <origin xyz="${-brake_thickness/2} ${-brake_height+0.006} ${-second_bar_length-first_bar_length}" rpy="0 0 0"/>
+            <origin xyz="${-brake_thickness/2} ${-brake_height+0.006} ${-second_bar_length-first_bar_length-0.003}" rpy="0 0 0"/>
             <geometry>
                 <mesh filename="package://senseglove_description/urdf/STL/MK29_DK1_Abduction_joint_v2.STL" scale="0.001 0.001 0.001"/>
@@ -232,5 +232,5 @@
     <link name="ring_flexion_one">
         <visual>
-            <origin xyz="0 0 0" rpy="0 0 0"/>
+            <origin xyz="${-brake_thickness/2} ${-brake_height+0.005} ${-second_bar_length-0.0055}" rpy="0 0 0"/>
             <geometry>
                 <mesh filename="package://senseglove_description/urdf/STL/MK29_DK1_Flexion_joint_1_v2.STL" scale="0.001 0.001 0.001"/>
@@ -241,5 +241,5 @@
     <link name="ring_flexion_two">
         <visual>
-            <origin xyz="0 0 ${-first_bar_length}" rpy="0 0 0"/>
+            <origin xyz="${-brake_thickness/2} ${-brake_height+0.005} ${-second_bar_length-0.005355}" rpy="0 0 0"/>
             <geometry>
                 <mesh filename="package://senseglove_description/urdf/STL/MK29_DK1_Flexion_joint_2_v2.STL" scale="0.001 0.001 0.001"/>
@@ -250,5 +250,5 @@
     <link name="ring_flexion_three">
         <visual>
-            <origin xyz="0 0 0" rpy="0 0 0"/>
+            <origin xyz="${-brake_thickness/2} ${-brake_height+0.00533} -0.00533" rpy="0 0 0"/>
             <geometry>
                 <mesh filename="package://senseglove_description/urdf/STL/MK29_DK1_Flexion_joint_3_v2.STL" scale="0.001 0.001 0.001"/>
@@ -259,5 +259,5 @@
     <link name="ring_thimble">
         <visual>
-            <origin xyz="0 0 ${-third_bar_length}" rpy="0 0 0"/>
+            <origin xyz="${-brake_thickness/2} -0.014951 ${-third_bar_length-0.0028}" rpy="0 0 0"/>
             <geometry>
                 <mesh filename="package://senseglove_description/urdf/STL/MK29_DK1_Thimble_v2.STL" scale="0.001 0.001 0.001"/>
@@ -268,5 +268,5 @@
     <link name="pinky_brake">
         <visual>
-            <origin xyz="${-brake_thickness/2} ${-brake_height/2} ${-first_bar_length-second_bar_length-brake_length}" rpy="0 0 0"/>
+            <origin xyz="${-brake_thickness/2-0.0004} ${-brake_height/2 - 0.0025} ${-first_bar_length-second_bar_length-0.003}" rpy="0 0 0"/>
             <geometry>
                 <mesh filename="package://senseglove_description/urdf/STL/MK29_DK1_Brake_assembly_v2.STL" scale="0.001 0.001 0.001"/>
@@ -277,5 +277,5 @@
     <link name="pinky_abduction">
         <visual>
-            <origin xyz="${-brake_thickness/2} ${-brake_height+0.006} ${-second_bar_length-first_bar_length}" rpy="0 0 0"/>
+            <origin xyz="${-brake_thickness/2} ${-brake_height+0.006} ${-second_bar_length-first_bar_length-0.003}" rpy="0 0 0"/>
             <geometry>
                 <mesh filename="package://senseglove_description/urdf/STL/MK29_DK1_Abduction_joint_v2.STL" scale="0.001 0.001 0.001"/>
@@ -286,5 +286,5 @@
     <link name="pinky_flexion_one">
         <visual>
-            <origin xyz="0 0 0" rpy="0 0 0"/>
+            <origin xyz="${-brake_thickness/2} ${-brake_height+0.005} ${-second_bar_length-0.0055}" rpy="0 0 0"/>
             <geometry>
                 <mesh filename="package://senseglove_description/urdf/STL/MK29_DK1_Flexion_joint_1_v2.STL" scale="0.001 0.001 0.001"/>
@@ -295,5 +295,5 @@
     <link name="pinky_flexion_two">
         <visual>
-            <origin xyz="0 0 ${-first_bar_length}" rpy="0 0 0"/>
+            <origin xyz="${-brake_thickness/2} ${-brake_height+0.005} ${-second_bar_length-0.005355}" rpy="0 0 0"/>
             <geometry>
                 <mesh filename="package://senseglove_description/urdf/STL/MK29_DK1_Flexion_joint_2_v2.STL" scale="0.001 0.001 0.001"/>
@@ -304,5 +304,5 @@
     <link name="pinky_flexion_three">
         <visual>
-            <origin xyz="0 0 0" rpy="0 0 0"/>
+            <origin xyz="${-brake_thickness/2} ${-brake_height+0.00533} -0.00533" rpy="0 0 0"/>
             <geometry>
                 <mesh filename="package://senseglove_description/urdf/STL/MK29_DK1_Flexion_joint_3_v2.STL" scale="0.001 0.001 0.001"/>
@@ -313,5 +313,5 @@
     <link name="pinky_thimble">
         <visual>
-            <origin xyz="0 0 ${-third_bar_length}" rpy="0 0 0"/>
+            <origin xyz="${-brake_thickness/2} -0.014951 ${-third_bar_length-0.0028}" rpy="0 0 0"/>
             <geometry>
                 <mesh filename="package://senseglove_description/urdf/STL/MK29_DK1_Thimble_v2.STL" scale="0.001 0.001 0.001"/>
@@ -328,10 +328,10 @@
         <parent link="glove_hub"/>
         <child link="thumb_brake"/>
-        <origin xyz="${thumb_hub_X} ${thumb_hub_Y} ${thumb_hub_Z}" rpy="${105*PI/180} ${40*PI/180} ${170.0*PI/180.0}"/>
+        <origin xyz="${thumb_hub_X} ${thumb_hub_Y} ${thumb_hub_Z}" rpy="${111.5*PI/180} ${40*PI/180} ${170.0*PI/180.0}"/>
     </joint>
     <joint name="thumb_brake" type="revolute">
         <parent link="thumb_brake"/>
         <child link="thumb_abduction"/>
-        <origin xyz="0 0 0" rpy="0 0 0"/>
+        <origin xyz="0 0.0074 ${-0.0}" rpy="0 0 0"/>
         <axis xyz="0 1 0"/>
         <limit velocity="${1}"
@@ -343,6 +343,6 @@
         <parent link="thumb_abduction"/>
         <child link="thumb_flexion_one"/>
-        <origin xyz="0 0 0" rpy="0 0 0"/>
-        <axis xyz="0 1 0"/>
+        <origin xyz="0 0 ${-0.00911-0.01414}" rpy="0 0 0"/>
+        <axis xyz="0 0 1"/>
         <limit velocity="${1}"
                effort="${10000}"
@@ -363,5 +363,5 @@
         <parent link="thumb_flexion_two"/>
         <child link="thumb_flexion_three"/>
-        <origin xyz="0 0 ${second_bar_length}" rpy="0 0 0"/>
+        <origin xyz="0 0 ${-second_bar_length}" rpy="0 0 0"/>
         <axis xyz="1 0 0"/>
         <limit velocity="${1}"
@@ -373,5 +373,5 @@
         <parent link="thumb_flexion_three"/>
         <child link="thumb_thimble"/>
-        <origin xyz="0 0 ${third_bar_length}" rpy="0 0 0"/>
+        <origin xyz="0 -0.012342 ${third_bar_length-0.0025}" rpy="0 0 0"/>
         <axis xyz="1 0 0"/>
         <limit velocity="${1}"
@@ -388,5 +388,5 @@
         <parent link="index_brake"/>
         <child link="index_abduction"/>
-        <origin xyz="0 0 ${brake_length}" rpy="0 0 0"/>
+        <origin xyz="0 0.0074 ${-0.0}" rpy="0 0 0"/>
         <axis xyz="0 1 0"/>
         <limit velocity="${1}"
@@ -398,6 +398,6 @@
         <parent link="index_abduction"/>
         <child link="index_flexion_one"/>
-        <origin xyz="0 0 0" rpy="0 0 0"/>
-        <axis xyz="0 1 0"/>
+        <origin xyz="0 0 ${-0.00911-0.01414}" rpy="0 0 0"/>
+        <axis xyz="0 0 1"/>
         <limit velocity="${1}"
                effort="${10000}"
@@ -408,5 +408,5 @@
         <parent link="index_flexion_one"/>
         <child link="index_flexion_two"/>
-        <origin xyz="0 0 ${first_bar_length}" rpy="0 0 0"/>
+        <origin xyz="0 0 0" rpy="0 0 0"/>
         <axis xyz="1 0 0"/>
         <limit velocity="${1}"
@@ -418,5 +418,5 @@
         <parent link="index_flexion_two"/>
         <child link="index_flexion_three"/>
-        <origin xyz="0 0 ${second_bar_length}" rpy="0 0 0"/>
+        <origin xyz="0 0 ${-second_bar_length}" rpy="0 0 0"/>
         <axis xyz="1 0 0"/>
         <limit velocity="${1}"
@@ -428,5 +428,5 @@
         <parent link="index_flexion_three"/>
         <child link="index_thimble"/>
-        <origin xyz="0 0 ${third_bar_length}" rpy="0 0 0"/>
+        <origin xyz="0 -0.012342 ${third_bar_length-0.0025}" rpy="0 0 0"/>
         <axis xyz="1 0 0"/>
         <limit velocity="${1}"
@@ -443,5 +443,5 @@
         <parent link="middle_brake"/>
         <child link="middle_abduction"/>
-        <origin xyz="0 0 ${brake_length}" rpy="0 0 0"/>
+        <origin xyz="0 0.0074 ${-0.0}" rpy="0 0 0"/>
         <axis xyz="0 1 0"/>
         <limit velocity="${1}"
@@ -453,6 +453,6 @@
         <parent link="middle_abduction"/>
         <child link="middle_flexion_one"/>
-        <origin xyz="0 0 0" rpy="0 0 0"/>
-        <axis xyz="0 1 0"/>
+        <origin xyz="0 0 ${-0.00911-0.01414}" rpy="0 0 0"/>
+        <axis xyz="0 0 1"/>
         <limit velocity="${1}"
                effort="${10000}"
@@ -463,5 +463,5 @@
         <parent link="middle_flexion_one"/>
         <child link="middle_flexion_two"/>
-        <origin xyz="0 0 ${first_bar_length}" rpy="0 0 0"/>
+        <origin xyz="0 0 0" rpy="0 0 0"/>
         <axis xyz="1 0 0"/>
         <limit velocity="${1}"
@@ -473,5 +473,5 @@
         <parent link="middle_flexion_two"/>
         <child link="middle_flexion_three"/>
-        <origin xyz="0 0 ${second_bar_length}" rpy="0 0 0"/>
+        <origin xyz="0 0 ${-second_bar_length}" rpy="0 0 0"/>
         <axis xyz="1 0 0"/>
         <limit velocity="${1}"
@@ -483,5 +483,5 @@
         <parent link="middle_flexion_three"/>
         <child link="middle_thimble"/>
-        <origin xyz="0 0 ${third_bar_length}" rpy="0 0 0"/>
+        <origin xyz="0 -0.012342 ${third_bar_length-0.0025}" rpy="0 0 0"/>
         <axis xyz="1 0 0"/>
         <limit velocity="${1}"
@@ -498,5 +498,5 @@
         <parent link="ring_brake"/>
         <child link="ring_abduction"/>
-        <origin xyz="0 0 ${brake_length}" rpy="0 0 0"/>
+        <origin xyz="0 0.0074 ${-0.0}" rpy="0 0 0"/>
         <axis xyz="0 1 0"/>
         <limit velocity="${1}"
@@ -508,6 +508,6 @@
         <parent link="ring_abduction"/>
         <child link="ring_flexion_one"/>
-        <origin xyz="0 0 0" rpy="0 0 0"/>
-        <axis xyz="0 1 0"/>
+        <origin xyz="0 0 ${-0.00911-0.01414}" rpy="0 0 0"/>
+        <axis xyz="0 0 1"/>
         <limit velocity="${1}"
                effort="${10000}"
@@ -518,5 +518,5 @@
         <parent link="ring_flexion_one"/>
         <child link="ring_flexion_two"/>
-        <origin xyz="0 0 ${first_bar_length}" rpy="0 0 0"/>
+        <origin xyz="0 0 0" rpy="0 0 0"/>
         <axis xyz="1 0 0"/>
         <limit velocity="${1}"
@@ -528,5 +528,5 @@
         <parent link="ring_flexion_two"/>
         <child link="ring_flexion_three"/>
-        <origin xyz="0 0 ${second_bar_length}" rpy="0 0 0"/>
+        <origin xyz="0 0 ${-second_bar_length}" rpy="0 0 0"/>
         <axis xyz="1 0 0"/>
         <limit velocity="${1}"
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