Commit message: Input semi correct ROM for all joints. It's semi correct as the allowed ROM will always provide enough movement when actually wearing the glove, but to avoid collision errors, the ROM was chosen slightly larger than normal.

File: src/senseglove/senseglove_description/urdf/dk1.xacro (robot description, xacro)
@@ -337,6 +337,6 @@
         <limit velocity="${1}"
                effort="${10000}"
-               lower="${-1}"
-               upper="${1}"/>
+               lower="${-2}"
+               upper="${2}"/>
     </joint>
     <joint name="thumb_abduction" type="revolute">
@@ -347,16 +347,16 @@
         <limit velocity="${1}"
                effort="${10000}"
-               lower="${-1}"
-               upper="${1}"/>
+               lower="${-2}"
+               upper="${2}"/>
     </joint>
     <joint name="thumb_cmc" type="revolute">
         <parent link="thumb_flexion_one"/>
         <child link="thumb_flexion_two"/>
-        <origin xyz="0 0 ${first_bar_length}" rpy="0 0 0"/>
-        <axis xyz="1 0 0"/>
-        <limit velocity="${1}"
-               effort="${10000}"
-               lower="${-1}"
-               upper="${1}"/>
+        <origin xyz="0 0 0" rpy="0 0 0"/>
+        <axis xyz="1 0 0"/>
+        <limit velocity="${1}"
+               effort="${10000}"
+               lower="${-2}"
+               upper="${0.25}"/>
     </joint>
     <joint name="thumb_mcp" type="revolute">
@@ -367,6 +367,6 @@
         <limit velocity="${1}"
                effort="${10000}"
-               lower="${-1}"
-               upper="${1}"/>
+               lower="${0}"
+               upper="${2.5}"/>
     </joint>
     <joint name="thumb_pip" type="revolute">
@@ -377,6 +377,6 @@
         <limit velocity="${1}"
                effort="${10000}"
-               lower="${-1}"
-               upper="${1}"/>
+               lower="${-4.2}"
+               upper="${0}"/>
     </joint>
     <joint name="hub_to_index_brake" type="fixed">
@@ -392,6 +392,6 @@
         <limit velocity="${1}"
                effort="${10000}"
-               lower="${-1}"
-               upper="${1}"/>
+               lower="${-2}"
+               upper="${2}"/>
     </joint>
     <joint name="index_abduction" type="revolute">
@@ -402,6 +402,6 @@
         <limit velocity="${1}"
                effort="${10000}"
-               lower="${-1}"
-               upper="${1}"/>
+               lower="${-2}"
+               upper="${2}"/>
     </joint>
     <joint name="index_mcp" type="revolute">
@@ -412,6 +412,6 @@
         <limit velocity="${1}"
                effort="${10000}"
-               lower="${-1}"
-               upper="${1}"/>
+               lower="${-2}"
+               upper="${0.25}"/>
     </joint>
     <joint name="index_pip" type="revolute">
@@ -422,6 +422,6 @@
         <limit velocity="${1}"
                effort="${10000}"
-               lower="${-1}"
-               upper="${1}"/>
+               lower="${0}"
+               upper="${2.5}"/>
     </joint>
     <joint name="index_dip" type="revolute">
@@ -432,6 +432,6 @@
         <limit velocity="${1}"
                effort="${10000}"
-               lower="${-1}"
-               upper="${1}"/>
+               lower="${-4.2}"
+               upper="${0}"/>
     </joint>
     <joint name="hub_to_middle_brake" type="fixed">
@@ -447,6 +447,6 @@
         <limit velocity="${1}"
                effort="${10000}"
-               lower="${-1}"
-               upper="${1}"/>
+               lower="${-2}"
+               upper="${2}"/>
     </joint>
     <joint name="middle_abduction" type="revolute">
@@ -457,6 +457,6 @@
         <limit velocity="${1}"
                effort="${10000}"
-               lower="${-1}"
-               upper="${1}"/>
+               lower="${-2}"
+               upper="${2}"/>
     </joint>
     <joint name="middle_mcp" type="revolute">
@@ -467,6 +467,6 @@
         <limit velocity="${1}"
                effort="${10000}"
-               lower="${-1}"
-               upper="${1}"/>
+               lower="${-2}"
+               upper="${0.25}"/>
     </joint>
     <joint name="middle_pip" type="revolute">
@@ -477,6 +477,6 @@
         <limit velocity="${1}"
                effort="${10000}"
-               lower="${-1}"
-               upper="${1}"/>
+               lower="${0}"
+               upper="${2.5}"/>
     </joint>
     <joint name="middle_dip" type="revolute">
@@ -487,6 +487,6 @@
         <limit velocity="${1}"
                effort="${10000}"
-               lower="${-1}"
-               upper="${1}"/>
+               lower="${-4.2}"
+               upper="${0}"/>
     </joint>
     <joint name="hub_to_ring_brake" type="fixed">
@@ -502,6 +502,6 @@
         <limit velocity="${1}"
                effort="${10000}"
-               lower="${-1}"
-               upper="${1}"/>
+               lower="${-2}"
+               upper="${2}"/>
     </joint>
     <joint name="ring_abduction" type="revolute">
@@ -512,6 +512,6 @@
         <limit velocity="${1}"
                effort="${10000}"
-               lower="${-1}"
-               upper="${1}"/>
+               lower="${-2}"
+               upper="${2}"/>
     </joint>
     <joint name="ring_mcp" type="revolute">
@@ -522,6 +522,6 @@
         <limit velocity="${1}"
                effort="${10000}"
-               lower="${-1}"
-               upper="${1}"/>
+               lower="${-2}"
+               upper="${0.25}"/>
     </joint>
     <joint name="ring_pip" type="revolute">
@@ -532,6 +532,6 @@
         <limit velocity="${1}"
                effort="${10000}"
-               lower="${-1}"
-               upper="${1}"/>
+               lower="${0}"
+               upper="${2.5}"/>
     </joint>
     <joint name="ring_dip" type="revolute">
@@ -542,6 +542,6 @@
         <limit velocity="${1}"
                effort="${10000}"
-               lower="${-1}"
-               upper="${1}"/>
+               lower="${-4.2}"
+               upper="${0}"/>
     </joint>
     <joint name="hub_to_pinky_brake" type="fixed">
@@ -557,6 +557,6 @@
         <limit velocity="${1}"
                effort="${10000}"
-               lower="${-1}"
-               upper="${1}"/>
+               lower="${-2}"
+               upper="${2}"/>
     </joint>
     <joint name="pinky_abduction" type="revolute">
@@ -567,6 +567,6 @@
         <limit velocity="${1}"
                effort="${10000}"
-               lower="${-1}"
-               upper="${1}"/>
+               lower="${-2}"
+               upper="${2}"/>
     </joint>
     <joint name="pinky_mcp" type="revolute">
@@ -577,6 +577,6 @@
         <limit velocity="${1}"
                effort="${10000}"
-               lower="${-1}"
-               upper="${1}"/>
+               lower="${-2}"
+               upper="${0.25}"/>
     </joint>
     <joint name="pinky_pip" type="revolute">
@@ -587,6 +587,6 @@
         <limit velocity="${1}"
                effort="${10000}"
-               lower="${-1}"
-               upper="${1}"/>
+               lower="${0}"
+               upper="${2.5}"/>
     </joint>
     <joint name="pinky_dip" type="revolute">
@@ -597,6 +597,6 @@
         <limit velocity="${1}"
                effort="${10000}"
-               lower="${-1}"
-               upper="${1}"/>
+               lower="${-4.2}"
+               upper="${0}"/>
     </joint>
 </robot>
