Commit message: fixed the force feedback commands from breaking the controller by using Max's new and shiny Senseglove_API .so files as well as fixing transformation errors in the URDF of the left and right glove so that users can call rviz directly when the hardware interface is running.

File: src/senseglove/senseglove_description/urdf/dk1_left.xacro (robot description, xacro)
@@ -38,6 +38,6 @@
     <xacro:property name="joint_velocity_limit" value="1.0"/> <!-- rad/s -->
     <xacro:property name="hover_height" value="0.5"/>
-    <!-- Used for fixing robot to Gazebo 'base_link' -->
-    <link name="base_link"/>
+    <!-- Used for fixing robot to Gazebo 'world' -->
+    <link name="world"/>
     <!-- glove hub -->
     <link name="glove_hub">
@@ -321,5 +321,5 @@
     <!-- Joints -->
     <joint name="joint_base_fixed_parent_joint" type="fixed">
-        <parent link="base_link"/>
+        <parent link="world"/>
         <child link="glove_hub"/>
         <origin xyz="0 0 ${hover_height}" rpy="0 0 0"/>
@@ -340,13 +340,8 @@
                upper="${2}"/>
     </joint>
-    <joint name="thumb_abduction" type="revolute">
+    <joint name="thumb_abduction" type="fixed">
         <parent link="thumb_abduction"/>
         <child link="thumb_flexion_one"/>
         <origin xyz="0 0 ${-0.00911-0.01414}" rpy="0 0 0"/>
-        <axis xyz="0 0 1"/>
-        <limit velocity="${1}"
-               effort="${10000}"
-               lower="${-2}"
-               upper="${2}"/>
     </joint>
     <joint name="thumb_cmc" type="revolute">
@@ -354,5 +349,5 @@
         <child link="thumb_flexion_two"/>
         <origin xyz="0 0 0" rpy="0 0 0"/>
-        <axis xyz="1 0 0"/>
+        <axis xyz="-1 0 0"/>
         <limit velocity="${1}"
                effort="${10000}"
@@ -364,5 +359,5 @@
         <child link="thumb_flexion_three"/>
         <origin xyz="0 0 ${-second_bar_length}" rpy="0 0 0"/>
-        <axis xyz="1 0 0"/>
+        <axis xyz="-1 0 0"/>
         <limit velocity="${1}"
                effort="${10000}"
@@ -374,5 +369,5 @@
         <child link="thumb_thimble"/>
         <origin xyz="0 -0.012342 ${third_bar_length-0.0025}" rpy="0 0 0"/>
-        <axis xyz="1 0 0"/>
+        <axis xyz="-1 0 0"/>
         <limit velocity="${1}"
                effort="${10000}"
@@ -395,13 +390,8 @@
                upper="${2}"/>
     </joint>
-    <joint name="index_abduction" type="revolute">
+    <joint name="index_abduction" type="fixed">
         <parent link="index_abduction"/>
         <child link="index_flexion_one"/>
         <origin xyz="0 0 ${-0.00911-0.01414}" rpy="0 0 0"/>
-        <axis xyz="0 0 1"/>
-        <limit velocity="${1}"
-               effort="${10000}"
-               lower="${-2}"
-               upper="${2}"/>
     </joint>
     <joint name="index_mcp" type="revolute">
@@ -409,5 +399,5 @@
         <child link="index_flexion_two"/>
         <origin xyz="0 0 0" rpy="0 0 0"/>
-        <axis xyz="1 0 0"/>
+        <axis xyz="-1 0 0"/>
         <limit velocity="${1}"
                effort="${10000}"
@@ -419,5 +409,5 @@
         <child link="index_flexion_three"/>
         <origin xyz="0 0 ${-second_bar_length}" rpy="0 0 0"/>
-        <axis xyz="1 0 0"/>
+        <axis xyz="-1 0 0"/>
         <limit velocity="${1}"
                effort="${10000}"
@@ -429,5 +419,5 @@
         <child link="index_thimble"/>
         <origin xyz="0 -0.012342 ${third_bar_length-0.0025}" rpy="0 0 0"/>
-        <axis xyz="1 0 0"/>
+        <axis xyz="-1 0 0"/>
         <limit velocity="${1}"
                effort="${10000}"
@@ -450,13 +440,9 @@
                upper="${2}"/>
     </joint>
-    <joint name="middle_abduction" type="revolute">
+    <joint name="middle_abduction" type="fixed">
         <parent link="middle_abduction"/>
         <child link="middle_flexion_one"/>
         <origin xyz="0 0 ${-0.00911-0.01414}" rpy="0 0 0"/>
-        <axis xyz="0 0 1"/>
-        <limit velocity="${1}"
-               effort="${10000}"
-               lower="${-2}"
-               upper="${2}"/>
+-
     </joint>
     <joint name="middle_mcp" type="revolute">
@@ -464,5 +450,5 @@
         <child link="middle_flexion_two"/>
         <origin xyz="0 0 0" rpy="0 0 0"/>
-        <axis xyz="1 0 0"/>
+        <axis xyz="-1 0 0"/>
         <limit velocity="${1}"
                effort="${10000}"
@@ -474,5 +460,5 @@
         <child link="middle_flexion_three"/>
         <origin xyz="0 0 ${-second_bar_length}" rpy="0 0 0"/>
-        <axis xyz="1 0 0"/>
+        <axis xyz="-1 0 0"/>
         <limit velocity="${1}"
                effort="${10000}"
@@ -484,5 +470,5 @@
         <child link="middle_thimble"/>
         <origin xyz="0 -0.012342 ${third_bar_length-0.0025}" rpy="0 0 0"/>
-        <axis xyz="1 0 0"/>
+        <axis xyz="-1 0 0"/>
         <limit velocity="${1}"
                effort="${10000}"
@@ -505,13 +491,8 @@
                upper="${2}"/>
     </joint>
-    <joint name="ring_abduction" type="revolute">
+    <joint name="ring_abduction" type="fixed">
         <parent link="ring_abduction"/>
         <child link="ring_flexion_one"/>
         <origin xyz="0 0 ${-0.00911-0.01414}" rpy="0 0 0"/>
-        <axis xyz="0 0 1"/>
-        <limit velocity="${1}"
-               effort="${10000}"
-               lower="${-2}"
-               upper="${2}"/>
     </joint>
     <joint name="ring_mcp" type="revolute">
@@ -519,5 +500,5 @@
         <child link="ring_flexion_two"/>
         <origin xyz="0 0 0" rpy="0 0 0"/>
-        <axis xyz="1 0 0"/>
+        <axis xyz="-1 0 0"/>
         <limit velocity="${1}"
                effort="${10000}"
@@ -529,5 +510,5 @@
         <child link="ring_flexion_three"/>
         <origin xyz="0 0 ${-second_bar_length}" rpy="0 0 0"/>
-        <axis xyz="1 0 0"/>
+        <axis xyz="-1 0 0"/>
         <limit velocity="${1}"
                effort="${10000}"
@@ -539,5 +520,5 @@
         <child link="ring_thimble"/>
         <origin xyz="0 -0.012342 ${third_bar_length-0.0025}" rpy="0 0 0"/>
-        <axis xyz="1 0 0"/>
+        <axis xyz="-1 0 0"/>
         <limit velocity="${1}"
                effort="${10000}"
@@ -560,13 +541,8 @@
                upper="${2}"/>
     </joint>
-    <joint name="pinky_abduction" type="revolute">
+    <joint name="pinky_abduction" type="fixed">
         <parent link="pinky_abduction"/>
         <child link="pinky_flexion_one"/>
         <origin xyz="0 0 ${-0.00911-0.01414}" rpy="0 0 0"/>
-        <axis xyz="0 0 1"/>
-        <limit velocity="${1}"
-               effort="${10000}"
-               lower="${-2}"
-               upper="${2}"/>
     </joint>
     <joint name="pinky_mcp" type="revolute">
@@ -574,5 +550,5 @@
         <child link="pinky_flexion_two"/>
         <origin xyz="0 0 0" rpy="0 0 0"/>
-        <axis xyz="1 0 0"/>
+        <axis xyz="-1 0 0"/>
         <limit velocity="${1}"
                effort="${10000}"
@@ -584,5 +560,5 @@
         <child link="pinky_flexion_three"/>
         <origin xyz="0 0 ${-second_bar_length}" rpy="0 0 0"/>
-        <axis xyz="1 0 0"/>
+        <axis xyz="-1 0 0"/>
         <limit velocity="${1}"
                effort="${10000}"
@@ -594,5 +570,5 @@
         <child link="pinky_thimble"/>
         <origin xyz="0 -0.012342 ${third_bar_length-0.0025}" rpy="0 0 0"/>
-        <axis xyz="1 0 0"/>
+        <axis xyz="-1 0 0"/>
         <limit velocity="${1}"
                effort="${10000}"

File: src/senseglove/senseglove_description/urdf/dk1_right.xacro (robot description, xacro)
@@ -38,6 +38,6 @@
     <xacro:property name="joint_velocity_limit" value="1.0"/> <!-- rad/s -->
     <xacro:property name="hover_height" value="0.5"/>
-    <!-- Used for fixing robot to Gazebo 'base_link' -->
-    <link name="base_link"/>
+    <!-- Used for fixing robot to Gazebo 'world' -->
+    <link name="world"/>
     <!-- glove hub -->
     <link name="glove_hub">
@@ -321,5 +321,5 @@
     <!-- Joints -->
     <joint name="joint_base_fixed_parent_joint" type="fixed">
-        <parent link="base_link"/>
+        <parent link="world"/>
         <child link="glove_hub"/>
         <origin xyz="0 0 ${hover_height}" rpy="0 0 0"/>
@@ -340,13 +340,8 @@
                upper="${2}"/>
     </joint>
-    <joint name="thumb_abduction" type="revolute">
+    <joint name="thumb_abduction" type="fixed">
         <parent link="thumb_abduction"/>
         <child link="thumb_flexion_one"/>
         <origin xyz="0 0 ${-0.00911-0.01414}" rpy="0 0 0"/>
-        <axis xyz="0 0 1"/>
-        <limit velocity="${1}"
-               effort="${10000}"
-               lower="${-2}"
-               upper="${2}"/>
     </joint>
     <joint name="thumb_cmc" type="revolute">
@@ -354,5 +349,5 @@
         <child link="thumb_flexion_two"/>
         <origin xyz="0 0 0" rpy="0 0 0"/>
-        <axis xyz="1 0 0"/>
+        <axis xyz="-1 0 0"/>
         <limit velocity="${1}"
                effort="${10000}"
@@ -364,5 +359,5 @@
         <child link="thumb_flexion_three"/>
         <origin xyz="0 0 ${-second_bar_length}" rpy="0 0 0"/>
-        <axis xyz="1 0 0"/>
+        <axis xyz="-1 0 0"/>
         <limit velocity="${1}"
                effort="${10000}"
@@ -374,5 +369,5 @@
         <child link="thumb_thimble"/>
         <origin xyz="0 -0.012342 ${third_bar_length-0.0025}" rpy="0 0 0"/>
-        <axis xyz="1 0 0"/>
+        <axis xyz="-1 0 0"/>
         <limit velocity="${1}"
                effort="${10000}"
@@ -395,13 +390,8 @@
                upper="${2}"/>
     </joint>
-    <joint name="index_abduction" type="revolute">
+    <joint name="index_abduction" type="fixed">
         <parent link="index_abduction"/>
         <child link="index_flexion_one"/>
         <origin xyz="0 0 ${-0.00911-0.01414}" rpy="0 0 0"/>
-        <axis xyz="0 0 1"/>
-        <limit velocity="${1}"
-               effort="${10000}"
-               lower="${-2}"
-               upper="${2}"/>
     </joint>
     <joint name="index_mcp" type="revolute">
@@ -409,5 +399,5 @@
         <child link="index_flexion_two"/>
         <origin xyz="0 0 0" rpy="0 0 0"/>
-        <axis xyz="1 0 0"/>
+        <axis xyz="-1 0 0"/>
         <limit velocity="${1}"
                effort="${10000}"
@@ -419,5 +409,5 @@
         <child link="index_flexion_three"/>
         <origin xyz="0 0 ${-second_bar_length}" rpy="0 0 0"/>
-        <axis xyz="1 0 0"/>
+        <axis xyz="-1 0 0"/>
         <limit velocity="${1}"
                effort="${10000}"
@@ -429,5 +419,5 @@
         <child link="index_thimble"/>
         <origin xyz="0 -0.012342 ${third_bar_length-0.0025}" rpy="0 0 0"/>
-        <axis xyz="1 0 0"/>
+        <axis xyz="-1 0 0"/>
         <limit velocity="${1}"
                effort="${10000}"
@@ -450,13 +440,8 @@
                upper="${2}"/>
     </joint>
-    <joint name="middle_abduction" type="revolute">
+    <joint name="middle_abduction" type="fixed">
         <parent link="middle_abduction"/>
         <child link="middle_flexion_one"/>
         <origin xyz="0 0 ${-0.00911-0.01414}" rpy="0 0 0"/>
-        <axis xyz="0 0 1"/>
-        <limit velocity="${1}"
-               effort="${10000}"
-               lower="${-2}"
-               upper="${2}"/>
     </joint>
     <joint name="middle_mcp" type="revolute">
@@ -464,5 +449,5 @@
         <child link="middle_flexion_two"/>
         <origin xyz="0 0 0" rpy="0 0 0"/>
-        <axis xyz="1 0 0"/>
+        <axis xyz="-1 0 0"/>
         <limit velocity="${1}"
                effort="${10000}"
@@ -474,5 +459,5 @@
         <child link="middle_flexion_three"/>
         <origin xyz="0 0 ${-second_bar_length}" rpy="0 0 0"/>
-        <axis xyz="1 0 0"/>
+        <axis xyz="-1 0 0"/>
         <limit velocity="${1}"
                effort="${10000}"
@@ -484,5 +469,5 @@
         <child link="middle_thimble"/>
         <origin xyz="0 -0.012342 ${third_bar_length-0.0025}" rpy="0 0 0"/>
-        <axis xyz="1 0 0"/>
+        <axis xyz="-1 0 0"/>
         <limit velocity="${1}"
                effort="${10000}"
@@ -505,13 +490,8 @@
                upper="${2}"/>
     </joint>
-    <joint name="ring_abduction" type="revolute">
+    <joint name="ring_abduction" type="fixed">
         <parent link="ring_abduction"/>
         <child link="ring_flexion_one"/>
         <origin xyz="0 0 ${-0.00911-0.01414}" rpy="0 0 0"/>
-        <axis xyz="0 0 1"/>
-        <limit velocity="${1}"
-               effort="${10000}"
-               lower="${-2}"
-               upper="${2}"/>
     </joint>
     <joint name="ring_mcp" type="revolute">
@@ -519,5 +499,5 @@
         <child link="ring_flexion_two"/>
         <origin xyz="0 0 0" rpy="0 0 0"/>
-        <axis xyz="1 0 0"/>
+        <axis xyz="-1 0 0"/>
         <limit velocity="${1}"
                effort="${10000}"
@@ -529,5 +509,5 @@
         <child link="ring_flexion_three"/>
         <origin xyz="0 0 ${-second_bar_length}" rpy="0 0 0"/>
-        <axis xyz="1 0 0"/>
+        <axis xyz="-1 0 0"/>
         <limit velocity="${1}"
                effort="${10000}"
@@ -539,5 +519,5 @@
         <child link="ring_thimble"/>
         <origin xyz="0 -0.012342 ${third_bar_length-0.0025}" rpy="0 0 0"/>
-        <axis xyz="1 0 0"/>
+        <axis xyz="-1 0 0"/>
         <limit velocity="${1}"
                effort="${10000}"
@@ -560,13 +540,8 @@
                upper="${2}"/>
     </joint>
-    <joint name="pinky_abduction" type="revolute">
+    <joint name="pinky_abduction" type="fixed">
         <parent link="pinky_abduction"/>
         <child link="pinky_flexion_one"/>
         <origin xyz="0 0 ${-0.00911-0.01414}" rpy="0 0 0"/>
-        <axis xyz="0 0 1"/>
-        <limit velocity="${1}"
-               effort="${10000}"
-               lower="${-2}"
-               upper="${2}"/>
     </joint>
     <joint name="pinky_mcp" type="revolute">
@@ -574,5 +549,5 @@
         <child link="pinky_flexion_two"/>
         <origin xyz="0 0 0" rpy="0 0 0"/>
-        <axis xyz="1 0 0"/>
+        <axis xyz="-1 0 0"/>
         <limit velocity="${1}"
                effort="${10000}"
@@ -584,5 +559,5 @@
         <child link="pinky_flexion_three"/>
         <origin xyz="0 0 ${-second_bar_length}" rpy="0 0 0"/>
-        <axis xyz="1 0 0"/>
+        <axis xyz="-1 0 0"/>
         <limit velocity="${1}"
                effort="${10000}"
@@ -594,5 +569,5 @@
         <child link="pinky_thimble"/>
         <origin xyz="0 -0.012342 ${third_bar_length-0.0025}" rpy="0 0 0"/>
-        <axis xyz="1 0 0"/>
+        <axis xyz="-1 0 0"/>
         <limit velocity="${1}"
                effort="${10000}"
