Commit message: remove unnecessary print statements. fix mapping of buzzers and brakes. adjust velocity so that actuation of joints does not take forever also adjust the upper limit so the full 100% of the actuators. Add check if all glove and hand poses are updated before updating them in the publisher.

File: src/senseglove/senseglove_description/urdf/dk1_left.xacro (robot description, xacro)
@@ -335,6 +335,6 @@
         <origin xyz="0 0.0074 ${-0.0}" rpy="0 0 0"/>
         <axis xyz="0 1 0"/>
-        <limit velocity="${1}"
-               effort="${10000}"
+        <limit velocity="${1000}"
+               effort="${100}"
                lower="${-2}"
                upper="${2}"/>
@@ -350,8 +350,8 @@
         <origin xyz="0 0 0" rpy="0 0 0"/>
         <axis xyz="-1 0 0"/>
-        <limit velocity="${1}"
-               effort="${10000}"
-               lower="${-2}"
-               upper="${0.25}"/>
+        <limit velocity="${1000}"
+               effort="${100}"
+               lower="${-2}"
+               upper="${100}"/>
     </joint>
     <joint name="thumb_mcp" type="revolute">
@@ -360,8 +360,8 @@
         <origin xyz="0 0 ${-second_bar_length}" rpy="0 0 0"/>
         <axis xyz="-1 0 0"/>
-        <limit velocity="${1}"
-               effort="${10000}"
+        <limit velocity="${1000}"
+               effort="${100}"
                lower="${0}"
-               upper="${2.5}"/>
+               upper="${100}"/>
     </joint>
     <joint name="thumb_pip" type="revolute">
@@ -370,8 +370,8 @@
         <origin xyz="0 -0.012342 ${third_bar_length-0.0025}" rpy="0 0 0"/>
         <axis xyz="-1 0 0"/>
-        <limit velocity="${1}"
-               effort="${10000}"
+        <limit velocity="${1000}"
+               effort="${100}"
                lower="${-4.2}"
-               upper="${0}"/>
+               upper="${100}"/>
     </joint>
     <joint name="hub_to_index_brake" type="fixed">
@@ -385,8 +385,8 @@
         <origin xyz="0 0.0074 ${-0.0}" rpy="0 0 0"/>
         <axis xyz="0 1 0"/>
-        <limit velocity="${1}"
-               effort="${10000}"
-               lower="${-2}"
-               upper="${2}"/>
+        <limit velocity="${1000}"
+               effort="${100}"
+               lower="${-2}"
+               upper="${100}"/>
     </joint>
     <joint name="index_abduction" type="fixed">
@@ -400,8 +400,8 @@
         <origin xyz="0 0 0" rpy="0 0 0"/>
         <axis xyz="-1 0 0"/>
-        <limit velocity="${1}"
-               effort="${10000}"
-               lower="${-2}"
-               upper="${0.25}"/>
+        <limit velocity="${1000}"
+               effort="${100}"
+               lower="${-2}"
+               upper="${100}"/>
     </joint>
     <joint name="index_pip" type="revolute">
@@ -410,8 +410,8 @@
         <origin xyz="0 0 ${-second_bar_length}" rpy="0 0 0"/>
         <axis xyz="-1 0 0"/>
-        <limit velocity="${1}"
-               effort="${10000}"
+        <limit velocity="${1000}"
+               effort="${100}"
                lower="${0}"
-               upper="${2.5}"/>
+               upper="${100}"/>
     </joint>
     <joint name="index_dip" type="revolute">
@@ -420,8 +420,8 @@
         <origin xyz="0 -0.012342 ${third_bar_length-0.0025}" rpy="0 0 0"/>
         <axis xyz="-1 0 0"/>
-        <limit velocity="${1}"
-               effort="${10000}"
+        <limit velocity="${1000}"
+               effort="${100}"
                lower="${-4.2}"
-               upper="${0}"/>
+               upper="${100}"/>
     </joint>
     <joint name="hub_to_middle_brake" type="fixed">
@@ -435,8 +435,8 @@
         <origin xyz="0 0.0074 ${-0.0}" rpy="0 0 0"/>
         <axis xyz="0 1 0"/>
-        <limit velocity="${1}"
-               effort="${10000}"
-               lower="${-2}"
-               upper="${2}"/>
+        <limit velocity="${1000}"
+               effort="${100}"
+               lower="${-2}"
+               upper="${100}"/>
     </joint>
     <joint name="middle_abduction" type="fixed">
@@ -451,8 +451,8 @@
         <origin xyz="0 0 0" rpy="0 0 0"/>
         <axis xyz="-1 0 0"/>
-        <limit velocity="${1}"
-               effort="${10000}"
-               lower="${-2}"
-               upper="${0.25}"/>
+        <limit velocity="${1000}"
+               effort="${100}"
+               lower="${-2}"
+               upper="${100}"/>
     </joint>
     <joint name="middle_pip" type="revolute">
@@ -461,8 +461,8 @@
         <origin xyz="0 0 ${-second_bar_length}" rpy="0 0 0"/>
         <axis xyz="-1 0 0"/>
-        <limit velocity="${1}"
-               effort="${10000}"
+        <limit velocity="${1000}"
+               effort="${100}"
                lower="${0}"
-               upper="${2.5}"/>
+               upper="${100}"/>
     </joint>
     <joint name="middle_dip" type="revolute">
@@ -471,8 +471,8 @@
         <origin xyz="0 -0.012342 ${third_bar_length-0.0025}" rpy="0 0 0"/>
         <axis xyz="-1 0 0"/>
-        <limit velocity="${1}"
-               effort="${10000}"
+        <limit velocity="${1000}"
+               effort="${100}"
                lower="${-4.2}"
-               upper="${0}"/>
+               upper="${100}"/>
     </joint>
     <joint name="hub_to_ring_brake" type="fixed">
@@ -486,8 +486,8 @@
         <origin xyz="0 0.0074 ${-0.0}" rpy="0 0 0"/>
         <axis xyz="0 1 0"/>
-        <limit velocity="${1}"
-               effort="${10000}"
-               lower="${-2}"
-               upper="${2}"/>
+        <limit velocity="${1000}"
+               effort="${100}"
+               lower="${-2}"
+               upper="${100}"/>
     </joint>
     <joint name="ring_abduction" type="fixed">
@@ -501,8 +501,8 @@
         <origin xyz="0 0 0" rpy="0 0 0"/>
         <axis xyz="-1 0 0"/>
-        <limit velocity="${1}"
-               effort="${10000}"
-               lower="${-2}"
-               upper="${0.25}"/>
+        <limit velocity="${1000}"
+               effort="${100}"
+               lower="${-2}"
+               upper="${100}"/>
     </joint>
     <joint name="ring_pip" type="revolute">
@@ -511,8 +511,8 @@
         <origin xyz="0 0 ${-second_bar_length}" rpy="0 0 0"/>
         <axis xyz="-1 0 0"/>
-        <limit velocity="${1}"
-               effort="${10000}"
+        <limit velocity="${1000}"
+               effort="${100}"
                lower="${0}"
-               upper="${2.5}"/>
+               upper="${100}"/>
     </joint>
     <joint name="ring_dip" type="revolute">
@@ -521,8 +521,8 @@
         <origin xyz="0 -0.012342 ${third_bar_length-0.0025}" rpy="0 0 0"/>
         <axis xyz="-1 0 0"/>
-        <limit velocity="${1}"
-               effort="${10000}"
+        <limit velocity="${1000}"
+               effort="${100}"
                lower="${-4.2}"
-               upper="${0}"/>
+               upper="${100}"/>
     </joint>
     <joint name="hub_to_pinky_brake" type="fixed">
@@ -536,8 +536,8 @@
         <origin xyz="0 0.0074 ${-0.0}" rpy="0 0 0"/>
         <axis xyz="0 1 0"/>
-        <limit velocity="${1}"
-               effort="${10000}"
-               lower="${-2}"
-               upper="${2}"/>
+        <limit velocity="${1000}"
+               effort="${100}"
+               lower="${-2}"
+               upper="${100}"/>
     </joint>
     <joint name="pinky_abduction" type="fixed">
@@ -551,8 +551,8 @@
         <origin xyz="0 0 0" rpy="0 0 0"/>
         <axis xyz="-1 0 0"/>
-        <limit velocity="${1}"
-               effort="${10000}"
-               lower="${-2}"
-               upper="${0.25}"/>
+        <limit velocity="${1000}"
+               effort="${100}"
+               lower="${-2}"
+               upper="${100}"/>
     </joint>
     <joint name="pinky_pip" type="revolute">
@@ -561,8 +561,8 @@
         <origin xyz="0 0 ${-second_bar_length}" rpy="0 0 0"/>
         <axis xyz="-1 0 0"/>
-        <limit velocity="${1}"
-               effort="${10000}"
+        <limit velocity="${1000}"
+               effort="${100}"
                lower="${0}"
-               upper="${2.5}"/>
+               upper="${100}"/>
     </joint>
     <joint name="pinky_dip" type="revolute">
@@ -571,8 +571,8 @@
         <origin xyz="0 -0.012342 ${third_bar_length-0.0025}" rpy="0 0 0"/>
         <axis xyz="-1 0 0"/>
-        <limit velocity="${1}"
-               effort="${10000}"
+        <limit velocity="${1000}"
+               effort="${100}"
                lower="${-4.2}"
-               upper="${0}"/>
+               upper="${100}"/>
     </joint>
 </robot>

File: src/senseglove/senseglove_description/urdf/dk1_right.xacro (robot description, xacro)
@@ -335,8 +335,8 @@
         <origin xyz="0 0.0074 ${-0.0}" rpy="0 0 0"/>
         <axis xyz="0 1 0"/>
-        <limit velocity="${1}"
-               effort="${10000}"
-               lower="${-2}"
-               upper="${2}"/>
+        <limit velocity="${1000}"
+               effort="${100}"
+               lower="${0}"
+               upper="${100}"/>
     </joint>
     <joint name="thumb_abduction" type="fixed">
@@ -350,8 +350,8 @@
         <origin xyz="0 0 0" rpy="0 0 0"/>
         <axis xyz="-1 0 0"/>
-        <limit velocity="${1}"
-               effort="${10000}"
-               lower="${-2}"
-               upper="${0.25}"/>
+        <limit velocity="${1000}"
+               effort="${100}"
+               lower="${0}"
+               upper="${100}"/>
     </joint>
     <joint name="thumb_mcp" type="revolute">
@@ -360,8 +360,8 @@
         <origin xyz="0 0 ${-second_bar_length}" rpy="0 0 0"/>
         <axis xyz="-1 0 0"/>
-        <limit velocity="${1}"
-               effort="${10000}"
-               lower="${0}"
-               upper="${2.5}"/>
+        <limit velocity="${1000}"
+               effort="${100}"
+               lower="${0}"
+               upper="${100}"/>
     </joint>
     <joint name="thumb_pip" type="revolute">
@@ -370,8 +370,8 @@
         <origin xyz="0 -0.012342 ${third_bar_length-0.0025}" rpy="0 0 0"/>
         <axis xyz="-1 0 0"/>
-        <limit velocity="${1}"
-               effort="${10000}"
-               lower="${-4.2}"
-               upper="${0}"/>
+        <limit velocity="${1000}"
+               effort="${100}"
+               lower="${0}"
+               upper="${100}"/>
     </joint>
     <joint name="hub_to_index_brake" type="fixed">
@@ -385,8 +385,8 @@
         <origin xyz="0 0.0074 ${-0.0}" rpy="0 0 0"/>
         <axis xyz="0 1 0"/>
-        <limit velocity="${1}"
-               effort="${10000}"
-               lower="${-2}"
-               upper="${2}"/>
+        <limit velocity="${1000}"
+               effort="${100}"
+               lower="${-2}"
+               upper="${100}"/>
     </joint>
     <joint name="index_abduction" type="fixed">
@@ -400,8 +400,8 @@
         <origin xyz="0 0 0" rpy="0 0 0"/>
         <axis xyz="-1 0 0"/>
-        <limit velocity="${1}"
-               effort="${10000}"
-               lower="${-2}"
-               upper="${0.25}"/>
+        <limit velocity="${1000}"
+               effort="${100}"
+               lower="${-2}"
+               upper="${100}"/>
     </joint>
     <joint name="index_pip" type="revolute">
@@ -410,8 +410,8 @@
         <origin xyz="0 0 ${-second_bar_length}" rpy="0 0 0"/>
         <axis xyz="-1 0 0"/>
-        <limit velocity="${1}"
-               effort="${10000}"
-               lower="${0}"
-               upper="${2.5}"/>
+        <limit velocity="${1000}"
+               effort="${100}"
+               lower="${0}"
+               upper="${100}"/>
     </joint>
     <joint name="index_dip" type="revolute">
@@ -420,8 +420,8 @@
         <origin xyz="0 -0.012342 ${third_bar_length-0.0025}" rpy="0 0 0"/>
         <axis xyz="-1 0 0"/>
-        <limit velocity="${1}"
-               effort="${10000}"
+        <limit velocity="${1000}"
+               effort="${100}"
                lower="${-4.2}"
-               upper="${0}"/>
+               upper="${100}"/>
     </joint>
     <joint name="hub_to_middle_brake" type="fixed">
@@ -435,8 +435,8 @@
         <origin xyz="0 0.0074 ${-0.0}" rpy="0 0 0"/>
         <axis xyz="0 1 0"/>
-        <limit velocity="${1}"
-               effort="${10000}"
-               lower="${-2}"
-               upper="${2}"/>
+        <limit velocity="${1000}"
+               effort="${100}"
+               lower="${-2}"
+               upper="${100}"/>
     </joint>
     <joint name="middle_abduction" type="fixed">
@@ -450,8 +450,8 @@
         <origin xyz="0 0 0" rpy="0 0 0"/>
         <axis xyz="-1 0 0"/>
-        <limit velocity="${1}"
-               effort="${10000}"
-               lower="${-2}"
-               upper="${0.25}"/>
+        <limit velocity="${1000}"
+               effort="${100}"
+               lower="${-2}"
+               upper="${100}"/>
     </joint>
     <joint name="middle_pip" type="revolute">
@@ -460,8 +460,8 @@
         <origin xyz="0 0 ${-second_bar_length}" rpy="0 0 0"/>
         <axis xyz="-1 0 0"/>
-        <limit velocity="${1}"
-               effort="${10000}"
-               lower="${0}"
-               upper="${2.5}"/>
+        <limit velocity="${1000}"
+               effort="${100}"
+               lower="${0}"
+               upper="${100}"/>
     </joint>
     <joint name="middle_dip" type="revolute">
@@ -470,8 +470,8 @@
         <origin xyz="0 -0.012342 ${third_bar_length-0.0025}" rpy="0 0 0"/>
         <axis xyz="-1 0 0"/>
-        <limit velocity="${1}"
-               effort="${10000}"
+        <limit velocity="${1000}"
+               effort="${100}"
                lower="${-4.2}"
-               upper="${0}"/>
+               upper="${100}"/>
     </joint>
     <joint name="hub_to_ring_brake" type="fixed">
@@ -485,8 +485,8 @@
         <origin xyz="0 0.0074 ${-0.0}" rpy="0 0 0"/>
         <axis xyz="0 1 0"/>
-        <limit velocity="${1}"
-               effort="${10000}"
-               lower="${-2}"
-               upper="${2}"/>
+        <limit velocity="${1000}"
+               effort="${100}"
+               lower="${-2}"
+               upper="${100}"/>
     </joint>
     <joint name="ring_abduction" type="fixed">
@@ -500,8 +500,8 @@
         <origin xyz="0 0 0" rpy="0 0 0"/>
         <axis xyz="-1 0 0"/>
-        <limit velocity="${1}"
-               effort="${10000}"
-               lower="${-2}"
-               upper="${0.25}"/>
+        <limit velocity="${1000}"
+               effort="${100}"
+               lower="${-2}"
+               upper="${100}"/>
     </joint>
     <joint name="ring_pip" type="revolute">
@@ -510,8 +510,8 @@
         <origin xyz="0 0 ${-second_bar_length}" rpy="0 0 0"/>
         <axis xyz="-1 0 0"/>
-        <limit velocity="${1}"
-               effort="${10000}"
-               lower="${0}"
-               upper="${2.5}"/>
+        <limit velocity="${1000}"
+               effort="${100}"
+               lower="${0}"
+               upper="${100}"/>
     </joint>
     <joint name="ring_dip" type="revolute">
@@ -520,8 +520,8 @@
         <origin xyz="0 -0.012342 ${third_bar_length-0.0025}" rpy="0 0 0"/>
         <axis xyz="-1 0 0"/>
-        <limit velocity="${1}"
-               effort="${10000}"
+        <limit velocity="${1000}"
+               effort="${100}"
                lower="${-4.2}"
-               upper="${0}"/>
+               upper="${100}"/>
     </joint>
     <joint name="hub_to_pinky_brake" type="fixed">
@@ -535,8 +535,8 @@
         <origin xyz="0 0.0074 ${-0.0}" rpy="0 0 0"/>
         <axis xyz="0 1 0"/>
-        <limit velocity="${1}"
-               effort="${10000}"
-               lower="${-2}"
-               upper="${2}"/>
+        <limit velocity="${1000}"
+               effort="${100}"
+               lower="${-2}"
+               upper="${100}"/>
     </joint>
     <joint name="pinky_abduction" type="fixed">
@@ -550,8 +550,8 @@
         <origin xyz="0 0 0" rpy="0 0 0"/>
         <axis xyz="-1 0 0"/>
-        <limit velocity="${1}"
-               effort="${10000}"
-               lower="${-2}"
-               upper="${0.25}"/>
+        <limit velocity="${1000}"
+               effort="${100}"
+               lower="${-2}"
+               upper="${100}"/>
     </joint>
     <joint name="pinky_pip" type="revolute">
@@ -560,8 +560,8 @@
         <origin xyz="0 0 ${-second_bar_length}" rpy="0 0 0"/>
         <axis xyz="-1 0 0"/>
-        <limit velocity="${1}"
-               effort="${10000}"
-               lower="${0}"
-               upper="${2.5}"/>
+        <limit velocity="${1000}"
+               effort="${100}"
+               lower="${0}"
+               upper="${100}"/>
     </joint>
     <joint name="pinky_dip" type="revolute">
@@ -570,8 +570,8 @@
         <origin xyz="0 -0.012342 ${third_bar_length-0.0025}" rpy="0 0 0"/>
         <axis xyz="-1 0 0"/>
-        <limit velocity="${1}"
-               effort="${10000}"
+        <limit velocity="${1000}"
+               effort="${100}"
                lower="${-4.2}"
-               upper="${0}"/>
+               upper="${100}"/>
     </joint>
 </robot>

Commit message: Fix bug introduced by previous commit. Now the system is truly namespace independent. If the user wants to make use of rqt_joint_trajectory_controller launch rqt with the correct namespace arg i.e. rqt robot_description:=senseglove_x/robot_description

File: src/senseglove/senseglove_description/urdf/dk1_left.xacro (robot description, xacro)
@@ -334,5 +334,5 @@
         <child link="thumb_abduction"/>
         <origin xyz="0 0.0074 ${-0.0}" rpy="0 0 0"/>
-        <axis xyz="0 1 0"/>
+        <axis xyz="0 -1 0"/>
         <limit velocity="${1000}"
                effort="${100}"
@@ -384,5 +384,5 @@
         <child link="index_abduction"/>
         <origin xyz="0 0.0074 ${-0.0}" rpy="0 0 0"/>
-        <axis xyz="0 1 0"/>
+        <axis xyz="0 -1 0"/>
         <limit velocity="${1000}"
                effort="${100}"
@@ -434,5 +434,5 @@
         <child link="middle_abduction"/>
         <origin xyz="0 0.0074 ${-0.0}" rpy="0 0 0"/>
-        <axis xyz="0 1 0"/>
+        <axis xyz="0 -1 0"/>
         <limit velocity="${1000}"
                effort="${100}"
@@ -485,5 +485,5 @@
         <child link="ring_abduction"/>
         <origin xyz="0 0.0074 ${-0.0}" rpy="0 0 0"/>
-        <axis xyz="0 1 0"/>
+        <axis xyz="0 -1 0"/>
         <limit velocity="${1000}"
                effort="${100}"
@@ -535,5 +535,5 @@
         <child link="pinky_abduction"/>
         <origin xyz="0 0.0074 ${-0.0}" rpy="0 0 0"/>
-        <axis xyz="0 1 0"/>
+        <axis xyz="0 -1 0"/>
         <limit velocity="${1000}"
                effort="${100}"
