Commit message: refactor urdf/xacro files into two seperate versions for left and right, do the same for the controllers and configs and adjust the hardware launchers to make use of (use_)left and (use_)right args to determine which gloves to simulate. This commit then enables the user to load both robot models in RVIZ at the sametime

File: src/senseglove/senseglove_description/urdf/dk1_right.xacro (robot description, xacro)
@@ -41,5 +41,5 @@
     <link name="world"/>
     <!-- glove hub -->
-    <link name="glove_hub">
+    <link name="r_glove_hub">
         <visual>
             <origin xyz="-0.056692 -0.01955 -0.06803" rpy="0 0 0"/>
@@ -50,5 +50,5 @@
     </link>
     <!-- thumb brake -->
-    <link name="thumb_brake">
+    <link name="r_thumb_brake">
         <visual>
             <origin xyz="${-brake_thickness/2} ${-brake_height/2 - 0.0025} ${-first_bar_length-second_bar_length}" rpy="0 0 0"/>
@@ -59,5 +59,5 @@
     </link>
     <!-- thumb abduction -->
-    <link name="thumb_abduction">
+    <link name="r_thumb_abduction">
         <visual>
             <origin xyz="${-brake_thickness/2} ${-brake_height+0.006} ${-second_bar_length-first_bar_length-0.003}" rpy="0 0 0"/>
@@ -68,5 +68,5 @@
     </link>
     <!-- thumb flexion one -->
-    <link name="thumb_flexion_one">
+    <link name="r_thumb_flexion_one">
         <visual>
             <origin xyz="${-brake_thickness/2} ${-brake_height+0.005} ${-second_bar_length-0.0055}" rpy="0 0 0"/>
@@ -77,5 +77,5 @@
     </link>
     <!-- thumb flexion two -->
-    <link name="thumb_flexion_two">
+    <link name="r_thumb_flexion_two">
         <visual>
             <origin xyz="${-brake_thickness/2} ${-brake_height+0.005} ${-second_bar_length-0.005355}" rpy="0 0 0"/>
@@ -86,5 +86,5 @@
     </link>
     <!-- thumb flexion three -->
-    <link name="thumb_flexion_three">
+    <link name="r_thumb_flexion_three">
         <visual>
             <origin xyz="${-brake_thickness/2} ${-brake_height+0.00533} -0.00533" rpy="0 0 0"/>
@@ -95,5 +95,5 @@
     </link>
     <!-- thumb thimble -->
-    <link name="thumb_thimble">
+    <link name="r_thumb_thimble">
         <visual>
             <origin xyz="${-brake_thickness/2} -0.014951 ${-third_bar_length-0.0028}" rpy="0 0 0"/>
@@ -104,5 +104,5 @@
     </link>
     <!-- index brake -->
-    <link name="index_brake">
+    <link name="r_index_brake">
         <visual>
             <origin xyz="${-brake_thickness/2} ${-brake_height/2 - 0.0025} ${-first_bar_length-second_bar_length}" rpy="0 0 0"/>
@@ -113,5 +113,5 @@
     </link>
     <!-- index abduction -->
-    <link name="index_abduction">
+    <link name="r_index_abduction">
         <visual>
             <origin xyz="${-brake_thickness/2} ${-brake_height+0.006} ${-second_bar_length-first_bar_length-0.003}" rpy="0 0 0"/>
@@ -122,5 +122,5 @@
     </link>
     <!-- index flexion one -->
-    <link name="index_flexion_one">
+    <link name="r_index_flexion_one">
         <visual>
             <origin xyz="${-brake_thickness/2} ${-brake_height+0.005} ${-second_bar_length-0.0055}" rpy="0 0 0"/>
@@ -131,5 +131,5 @@
     </link>
     <!-- index flexion two -->
-    <link name="index_flexion_two">
+    <link name="r_index_flexion_two">
         <visual>
             <origin xyz="${-brake_thickness/2} ${-brake_height+0.005} ${-second_bar_length-0.005355}" rpy="0 0 0"/>
@@ -140,5 +140,5 @@
     </link>
     <!-- index flexion three -->
-    <link name="index_flexion_three">
+    <link name="r_index_flexion_three">
         <visual>
             <origin xyz="${-brake_thickness/2} ${-brake_height+0.00533} -0.00533" rpy="0 0 0"/>
@@ -149,5 +149,5 @@
     </link>
     <!-- index thimble -->
-    <link name="index_thimble">
+    <link name="r_index_thimble">
         <visual>
             <origin xyz="${-brake_thickness/2} -0.014951 ${-third_bar_length-0.0028}" rpy="0 0 0"/>
@@ -158,5 +158,5 @@
     </link>
     <!-- middle brake -->
-    <link name="middle_brake">
+    <link name="r_middle_brake">
         <visual>
             <origin xyz="${-brake_thickness/2} ${-brake_height/2 - 0.0025} ${-first_bar_length-second_bar_length}" rpy="0 0 0"/>
@@ -167,5 +167,5 @@
     </link>
     <!-- middle abduction -->
-    <link name="middle_abduction">
+    <link name="r_middle_abduction">
         <visual>
             <origin xyz="${-brake_thickness/2} ${-brake_height+0.006} ${-second_bar_length-first_bar_length-0.003}" rpy="0 0 0"/>
@@ -176,5 +176,5 @@
     </link>
     <!-- middle flexion one -->
-    <link name="middle_flexion_one">
+    <link name="r_middle_flexion_one">
         <visual>
             <origin xyz="${-brake_thickness/2} ${-brake_height+0.005} ${-second_bar_length-0.0055}" rpy="0 0 0"/>
@@ -185,5 +185,5 @@
     </link>
     <!-- middle flexion two -->
-    <link name="middle_flexion_two">
+    <link name="r_middle_flexion_two">
         <visual>
             <origin xyz="${-brake_thickness/2} ${-brake_height+0.005} ${-second_bar_length-0.005355}" rpy="0 0 0"/>
@@ -194,5 +194,5 @@
     </link>
     <!-- middle flexion three -->
-    <link name="middle_flexion_three">
+    <link name="r_middle_flexion_three">
         <visual>
             <origin xyz="${-brake_thickness/2} ${-brake_height+0.00533} -0.00533" rpy="0 0 0"/>
@@ -203,5 +203,5 @@
     </link>
     <!-- middle thimble -->
-    <link name="middle_thimble">
+    <link name="r_middle_thimble">
         <visual>
             <origin xyz="${-brake_thickness/2} -0.014951 ${-third_bar_length-0.0028}" rpy="0 0 0"/>
@@ -212,5 +212,5 @@
     </link>
     <!-- ring brake -->
-    <link name="ring_brake">
+    <link name="r_ring_brake">
         <visual>
             <origin xyz="${-brake_thickness/2} ${-brake_height/2 - 0.0025} ${-first_bar_length-second_bar_length}" rpy="0 0 0"/>
@@ -221,5 +221,5 @@
     </link>
     <!-- ring abduction -->
-    <link name="ring_abduction">
+    <link name="r_ring_abduction">
         <visual>
             <origin xyz="${-brake_thickness/2} ${-brake_height+0.006} ${-second_bar_length-first_bar_length-0.003}" rpy="0 0 0"/>
@@ -230,5 +230,5 @@
     </link>
     <!-- ring flexion one -->
-    <link name="ring_flexion_one">
+    <link name="r_ring_flexion_one">
         <visual>
             <origin xyz="${-brake_thickness/2} ${-brake_height+0.005} ${-second_bar_length-0.0055}" rpy="0 0 0"/>
@@ -239,5 +239,5 @@
     </link>
     <!-- ring flexion two -->
-    <link name="ring_flexion_two">
+    <link name="r_ring_flexion_two">
         <visual>
             <origin xyz="${-brake_thickness/2} ${-brake_height+0.005} ${-second_bar_length-0.005355}" rpy="0 0 0"/>
@@ -248,5 +248,5 @@
     </link>
     <!-- ring flexion three -->
-    <link name="ring_flexion_three">
+    <link name="r_ring_flexion_three">
         <visual>
             <origin xyz="${-brake_thickness/2} ${-brake_height+0.00533} -0.00533" rpy="0 0 0"/>
@@ -257,5 +257,5 @@
     </link>
     <!-- ring thimble -->
-    <link name="ring_thimble">
+    <link name="r_ring_thimble">
         <visual>
             <origin xyz="${-brake_thickness/2} -0.014951 ${-third_bar_length-0.0028}" rpy="0 0 0"/>
@@ -266,5 +266,5 @@
     </link>
     <!-- pinky brake -->
-    <link name="pinky_brake">
+    <link name="r_pinky_brake">
         <visual>
             <origin xyz="${-brake_thickness/2-0.0004} ${-brake_height/2 - 0.0025} ${-first_bar_length-second_bar_length-0.003}" rpy="0 0 0"/>
@@ -275,5 +275,5 @@
     </link>
     <!-- pinky abduction -->
-    <link name="pinky_abduction">
+    <link name="r_pinky_abduction">
         <visual>
             <origin xyz="${-brake_thickness/2} ${-brake_height+0.006} ${-second_bar_length-first_bar_length-0.003}" rpy="0 0 0"/>
@@ -284,5 +284,5 @@
     </link>
     <!-- pinky flexion one -->
-    <link name="pinky_flexion_one">
+    <link name="r_pinky_flexion_one">
         <visual>
             <origin xyz="${-brake_thickness/2} ${-brake_height+0.005} ${-second_bar_length-0.0055}" rpy="0 0 0"/>
@@ -293,5 +293,5 @@
     </link>
     <!-- pinky flexion two -->
-    <link name="pinky_flexion_two">
+    <link name="r_pinky_flexion_two">
         <visual>
             <origin xyz="${-brake_thickness/2} ${-brake_height+0.005} ${-second_bar_length-0.005355}" rpy="0 0 0"/>
@@ -302,5 +302,5 @@
     </link>
     <!-- pinky flexion three -->
-    <link name="pinky_flexion_three">
+    <link name="r_pinky_flexion_three">
         <visual>
             <origin xyz="${-brake_thickness/2} ${-brake_height+0.00533} -0.00533" rpy="0 0 0"/>
@@ -311,5 +311,5 @@
     </link>
     <!-- pinky thimble -->
-    <link name="pinky_thimble">
+    <link name="r_pinky_thimble">
         <visual>
             <origin xyz="${-brake_thickness/2} -0.014951 ${-third_bar_length-0.0028}" rpy="0 0 0"/>
@@ -322,15 +322,15 @@
     <joint name="joint_base_fixed_parent_joint" type="fixed">
         <parent link="world"/>
-        <child link="glove_hub"/>
-        <origin xyz="0 0 ${hover_height}" rpy="0 0 0"/>
-    </joint>
-    <joint name="hub_to_thumb_brake" type="fixed">
-        <parent link="glove_hub"/>
-        <child link="thumb_brake"/>
+        <child link="r_glove_hub"/>
+        <origin xyz="0.5 0 ${hover_height}" rpy="0 0 0"/>
+    </joint>
+    <joint name="r_hub_to_thumb_brake" type="fixed">
+        <parent link="r_glove_hub"/>
+        <child link="r_thumb_brake"/>
         <origin xyz="${thumb_hub_X} ${thumb_hub_Y} ${thumb_hub_Z}" rpy="${111.5*PI/180} ${40*PI/180} ${170.0*PI/180.0}"/>
     </joint>
-    <joint name="thumb_brake" type="revolute">
-        <parent link="thumb_brake"/>
-        <child link="thumb_abduction"/>
+    <joint name="r_thumb_brake" type="revolute">
+        <parent link="r_thumb_brake"/>
+        <child link="r_thumb_abduction"/>
         <origin xyz="0 0.0074 ${-0.0}" rpy="0 0 0"/>
         <axis xyz="0 1 0"/>
@@ -340,12 +340,12 @@
                upper="${100}"/>
     </joint>
-    <joint name="thumb_abduction" type="fixed">
-        <parent link="thumb_abduction"/>
-        <child link="thumb_flexion_one"/>
+    <joint name="r_thumb_abduction" type="fixed">
+        <parent link="r_thumb_abduction"/>
+        <child link="r_thumb_flexion_one"/>
         <origin xyz="0 0 ${-0.00911-0.01414}" rpy="0 0 0"/>
     </joint>
-    <joint name="thumb_cmc" type="revolute">
-        <parent link="thumb_flexion_one"/>
-        <child link="thumb_flexion_two"/>
+    <joint name="r_thumb_cmc" type="revolute">
+        <parent link="r_thumb_flexion_one"/>
+        <child link="r_thumb_flexion_two"/>
         <origin xyz="0 0 0" rpy="0 0 0"/>
         <axis xyz="-1 0 0"/>
@@ -355,7 +355,7 @@
                upper="${100}"/>
     </joint>
-    <joint name="thumb_mcp" type="revolute">
-        <parent link="thumb_flexion_two"/>
-        <child link="thumb_flexion_three"/>
+    <joint name="r_thumb_mcp" type="revolute">
+        <parent link="r_thumb_flexion_two"/>
+        <child link="r_thumb_flexion_three"/>
         <origin xyz="0 0 ${-second_bar_length}" rpy="0 0 0"/>
         <axis xyz="-1 0 0"/>
@@ -365,7 +365,7 @@
                upper="${100}"/>
     </joint>
-    <joint name="thumb_pip" type="revolute">
-        <parent link="thumb_flexion_three"/>
-        <child link="thumb_thimble"/>
+    <joint name="r_thumb_pip" type="revolute">
+        <parent link="r_thumb_flexion_three"/>
+        <child link="r_thumb_thimble"/>
         <origin xyz="0 -0.012342 ${third_bar_length-0.0025}" rpy="0 0 0"/>
         <axis xyz="-1 0 0"/>
@@ -375,12 +375,12 @@
                upper="${100}"/>
     </joint>
-    <joint name="hub_to_index_brake" type="fixed">
-        <parent link="glove_hub"/>
-        <child link="index_brake"/>
+    <joint name="r_hub_to_index_brake" type="fixed">
+        <parent link="r_glove_hub"/>
+        <child link="r_index_brake"/>
         <origin xyz="${index_hub_X} ${index_hub_Y} ${index_hub_Z}" rpy="0 0 0"/>
     </joint>
-    <joint name="index_brake" type="revolute">
-        <parent link="index_brake"/>
-        <child link="index_abduction"/>
+    <joint name="r_index_brake" type="revolute">
+        <parent link="r_index_brake"/>
+        <child link="r_index_abduction"/>
         <origin xyz="0 0.0074 ${-0.0}" rpy="0 0 0"/>
         <axis xyz="0 1 0"/>
@@ -390,12 +390,12 @@
                upper="${100}"/>
     </joint>
-    <joint name="index_abduction" type="fixed">
-        <parent link="index_abduction"/>
-        <child link="index_flexion_one"/>
+    <joint name="r_index_abduction" type="fixed">
+        <parent link="r_index_abduction"/>
+        <child link="r_index_flexion_one"/>
         <origin xyz="0 0 ${-0.00911-0.01414}" rpy="0 0 0"/>
     </joint>
-    <joint name="index_mcp" type="revolute">
-        <parent link="index_flexion_one"/>
-        <child link="index_flexion_two"/>
+    <joint name="r_index_mcp" type="revolute">
+        <parent link="r_index_flexion_one"/>
+        <child link="r_index_flexion_two"/>
         <origin xyz="0 0 0" rpy="0 0 0"/>
         <axis xyz="-1 0 0"/>
@@ -405,7 +405,7 @@
                upper="${100}"/>
     </joint>
-    <joint name="index_pip" type="revolute">
-        <parent link="index_flexion_two"/>
-        <child link="index_flexion_three"/>
+    <joint name="r_index_pip" type="revolute">
+        <parent link="r_index_flexion_two"/>
+        <child link="r_index_flexion_three"/>
         <origin xyz="0 0 ${-second_bar_length}" rpy="0 0 0"/>
         <axis xyz="-1 0 0"/>
@@ -415,7 +415,7 @@
                upper="${100}"/>
     </joint>
-    <joint name="index_dip" type="revolute">
-        <parent link="index_flexion_three"/>
-        <child link="index_thimble"/>
+    <joint name="r_index_dip" type="revolute">
+        <parent link="r_index_flexion_three"/>
+        <child link="r_index_thimble"/>
         <origin xyz="0 -0.012342 ${third_bar_length-0.0025}" rpy="0 0 0"/>
         <axis xyz="-1 0 0"/>
@@ -425,12 +425,12 @@
                upper="${100}"/>
     </joint>
-    <joint name="hub_to_middle_brake" type="fixed">
-        <parent link="glove_hub"/>
-        <child link="middle_brake"/>
+    <joint name="r_hub_to_middle_brake" type="fixed">
+        <parent link="r_glove_hub"/>
+        <child link="r_middle_brake"/>
         <origin xyz="${middle_hub_X} ${middle_hub_Y} ${middle_hub_Z}" rpy="0 0 0"/>
     </joint>
-    <joint name="middle_brake" type="revolute">
-        <parent link="middle_brake"/>
-        <child link="middle_abduction"/>
+    <joint name="r_middle_brake" type="revolute">
+        <parent link="r_middle_brake"/>
+        <child link="r_middle_abduction"/>
         <origin xyz="0 0.0074 ${-0.0}" rpy="0 0 0"/>
         <axis xyz="0 1 0"/>
@@ -440,12 +440,12 @@
                upper="${100}"/>
     </joint>
-    <joint name="middle_abduction" type="fixed">
-        <parent link="middle_abduction"/>
-        <child link="middle_flexion_one"/>
+    <joint name="r_middle_abduction" type="fixed">
+        <parent link="r_middle_abduction"/>
+        <child link="r_middle_flexion_one"/>
         <origin xyz="0 0 ${-0.00911-0.01414}" rpy="0 0 0"/>
     </joint>
-    <joint name="middle_mcp" type="revolute">
-        <parent link="middle_flexion_one"/>
-        <child link="middle_flexion_two"/>
+    <joint name="r_middle_mcp" type="revolute">
+        <parent link="r_middle_flexion_one"/>
+        <child link="r_middle_flexion_two"/>
         <origin xyz="0 0 0" rpy="0 0 0"/>
         <axis xyz="-1 0 0"/>
@@ -455,7 +455,7 @@
                upper="${100}"/>
     </joint>
-    <joint name="middle_pip" type="revolute">
-        <parent link="middle_flexion_two"/>
-        <child link="middle_flexion_three"/>
+    <joint name="r_middle_pip" type="revolute">
+        <parent link="r_middle_flexion_two"/>
+        <child link="r_middle_flexion_three"/>
         <origin xyz="0 0 ${-second_bar_length}" rpy="0 0 0"/>
         <axis xyz="-1 0 0"/>
@@ -465,7 +465,7 @@
                upper="${100}"/>
     </joint>
-    <joint name="middle_dip" type="revolute">
-        <parent link="middle_flexion_three"/>
-        <child link="middle_thimble"/>
+    <joint name="r_middle_dip" type="revolute">
+        <parent link="r_middle_flexion_three"/>
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
Commit message: Latest Backend, rough implementation of joint states and haptics

File: src/senseglove/senseglove_description/urdf/dk1_left.xacro (robot description, xacro)
@@ -17,14 +17,14 @@
     <xacro:property name="thumb_hub_Y" value="-0.0221293"/>
     <xacro:property name="thumb_hub_Z" value="0.04656"/>
-    <xacro:property name="pinky_hub_X" value="-0.03309"/>
+    <xacro:property name="index_hub_X" value="0.03307"/>
     <xacro:property name="index_hub_Y" value="0.00645"/>
     <xacro:property name="index_hub_Z" value="-0.04436"/>
-    <xacro:property name="ring_hub_X" value="-0.011"/>
+    <xacro:property name="middle_hub_X" value="0.011"/>
     <xacro:property name="middle_hub_Y" value="0.008"/>
     <xacro:property name="middle_hub_Z" value="-0.06222"/>
-    <xacro:property name="middle_hub_X" value="0.011"/>
+    <xacro:property name="ring_hub_X" value="-0.011"/>
     <xacro:property name="ring_hub_Y" value="0.008"/>
     <xacro:property name="ring_hub_Z" value="-0.05422"/>
-    <xacro:property name="index_hub_X" value="0.03307"/>
+    <xacro:property name="pinky_hub_X" value="-0.03309"/>
     <xacro:property name="pinky_hub_Y" value="0.00695"/>
     <xacro:property name="pinky_hub_Z" value="-0.04125"/>
@@ -345,5 +345,5 @@
         <origin xyz="0 0 ${-0.00911-0.01414}" rpy="0 0 0"/>
     </joint>
-    <joint name="l_thumb_cmc" type="revolute">
+    <joint name="l_thumb_mcp" type="revolute">
         <parent link="l_thumb_flexion_one"/>
         <child link="l_thumb_flexion_two"/>
@@ -355,5 +355,5 @@
                upper="${100}"/>
     </joint>
-    <joint name="l_thumb_mcp" type="revolute">
+    <joint name="l_thumb_pip" type="revolute">
         <parent link="l_thumb_flexion_two"/>
         <child link="l_thumb_flexion_three"/>
@@ -365,5 +365,5 @@
                upper="${100}"/>
     </joint>
-    <joint name="l_thumb_pip" type="revolute">
+    <joint name="l_thumb_dip" type="revolute">
         <parent link="l_thumb_flexion_three"/>
         <child link="l_thumb_thimble"/>

File: src/senseglove/senseglove_description/urdf/dk1_right.xacro (robot description, xacro)
@@ -345,5 +345,5 @@
         <origin xyz="0 0 ${-0.00911-0.01414}" rpy="0 0 0"/>
     </joint>
-    <joint name="r_thumb_cmc" type="revolute">
+    <joint name="r_thumb_mcp" type="revolute">
         <parent link="r_thumb_flexion_one"/>
         <child link="r_thumb_flexion_two"/>
@@ -355,5 +355,5 @@
                upper="${100}"/>
     </joint>
-    <joint name="r_thumb_mcp" type="revolute">
+    <joint name="r_thumb_pip" type="revolute">
         <parent link="r_thumb_flexion_two"/>
         <child link="r_thumb_flexion_three"/>
@@ -365,5 +365,5 @@
                upper="${100}"/>
     </joint>
-    <joint name="r_thumb_pip" type="revolute">
+    <joint name="r_thumb_dip" type="revolute">
         <parent link="r_thumb_flexion_three"/>
         <child link="r_thumb_thimble"/>
