Commit message: Fixed joint states, senseglove states, and finger-tip positions

File: src/senseglove/senseglove_description/urdf/nova_left.xacro (robot description, xacro)
@@ -2,5 +2,5 @@
 <!-- Revolute-Revolute Manipulator -->
 <robot name="nova" xmlns:xacro="http://www.ros.org/wiki/xacro">
-    <!-- Constants for robot dimensions -->
+   <!-- Constants for robot dimensions -->
     <xacro:property name="PI" value="3.1415926535897931"/>
     <xacro:property name="joint_base_mass" value="1"/> <!-- arbitrary value for joint_base_mass -->
@@ -26,4 +26,7 @@
     <xacro:property name="ring_hub_Y" value="0.008"/>
     <xacro:property name="ring_hub_Z" value="-0.05422"/>
+    <xacro:property name="pinky_hub_X" value="-0.03309"/>
+    <xacro:property name="pinky_hub_Y" value="0.00695"/>
+    <xacro:property name="pinky_hub_Z" value="-0.04125"/>
     <xacro:property name="bar_length" value="${0.39}"/>
     <xacro:property name="bar_mass" value="1.080"/>
@@ -82,4 +85,7 @@
         </visual>
     </link>
+    <!-- thumb flexion three -->
+    <link name="l_thumb_flexion_three">
+    </link>
     <!-- index brake -->
     <link name="l_index_brake">
@@ -118,4 +124,7 @@
         </visual>
     </link>
+    <!-- index flexion three -->
+    <link name="l_index_flexion_three">
+    </link>
     <!-- middle brake -->
     <link name="l_middle_brake">
@@ -154,4 +163,7 @@
         </visual>
     </link>
+    <!-- middle flexion three -->
+    <link name="l_middle_flexion_three">
+    </link>
     <!-- ring brake -->
     <link name="l_ring_brake">
@@ -189,4 +201,46 @@
             </geometry>
         </visual>
+    </link>
+    <!-- ring flexion three -->
+    <link name="l_ring_flexion_three">
+    </link>
+    <!-- pinky brake -->
+    <link name="l_pinky_brake">
+        <visual>
+            <origin xyz="${-brake_thickness/2-0.0004} ${-brake_height/2 - 0.0025} ${-first_bar_length-second_bar_length-0.003}" rpy="0 0 0"/>
+            <geometry>
+                <mesh filename="package://senseglove_description/urdf/STL/MK29_DK1_Brake_assembly_v2.STL" scale="0.001 0.001 0.001"/>
+            </geometry>
+        </visual>
+    </link>
+    <!-- pinky abduction -->
+    <link name="l_pinky_abduction">
+        <visual>
+            <origin xyz="${-brake_thickness/2} ${-brake_height+0.006} ${-second_bar_length-first_bar_length-0.003}" rpy="0 0 0"/>
+            <geometry>
+                <mesh filename="package://senseglove_description/urdf/STL/MK29_DK1_Abduction_joint_v2.STL" scale="0.001 0.001 0.001"/>
+            </geometry>
+        </visual>
+    </link>
+    <!-- pinky flexion one -->
+    <link name="l_pinky_flexion_one">
+        <visual>
+            <origin xyz="${-brake_thickness/2} ${-brake_height+0.005} ${-second_bar_length-0.0055}" rpy="0 0 0"/>
+            <geometry>
+                <mesh filename="package://senseglove_description/urdf/STL/MK29_DK1_Flexion_joint_1_v2.STL" scale="0.001 0.001 0.001"/>
+            </geometry>
+        </visual>
+    </link>
+    <!-- pinky flexion two -->
+    <link name="l_pinky_flexion_two">
+        <visual>
+            <origin xyz="${-brake_thickness/2} ${-brake_height+0.005} ${-second_bar_length-0.005355}" rpy="0 0 0"/>
+            <geometry>
+                <mesh filename="package://senseglove_description/urdf/STL/MK29_DK1_Flexion_joint_2_v2.STL" scale="0.001 0.001 0.001"/>
+            </geometry>
+        </visual>
+    </link>
+    <!-- pinky flexion three -->
+    <link name="l_pinky_flexion_three">
     </link>
     <!-- Joints -->
@@ -226,4 +280,14 @@
                upper="${100}"/>
     </joint>
+    <joint name="l_thumb_tip" type="revolute">
+        <parent link="l_thumb_flexion_two"/>
+        <child link="l_thumb_flexion_three"/>
+        <origin xyz="0 0 ${-second_bar_length}" rpy="0 0 0"/>
+        <axis xyz="-1 0 0"/>
+        <limit velocity="${1000}"
+               effort="${100}"
+               lower="${0}"
+               upper="${100}"/>
+    </joint>
     <joint name="l_hub_to_index_brake" type="fixed">
         <parent link="l_glove_hub"/>
@@ -256,4 +320,14 @@
                upper="${100}"/>
     </joint>
+    <joint name="l_index_tip" type="revolute">
+        <parent link="l_index_flexion_two"/>
+        <child link="l_index_flexion_three"/>
+        <origin xyz="0 0 ${-second_bar_length}" rpy="0 0 0"/>
+        <axis xyz="-1 0 0"/>
+        <limit velocity="${1000}"
+               effort="${100}"
+               lower="${0}"
+               upper="${100}"/>
+    </joint>
     <joint name="l_hub_to_middle_brake" type="fixed">
         <parent link="l_glove_hub"/>
@@ -287,8 +361,23 @@
                upper="${100}"/>
     </joint>
-    <joint name="l_hub_to_ring_brake" type="fixed">
-        <parent link="l_glove_hub"/>
-        <child link="l_ring_brake"/>
-        <origin xyz="${ring_hub_X} ${ring_hub_Y} ${ring_hub_Z}" rpy="0 0 0"/>
+    <joint name="l_middle_pip" type="revolute">
+        <parent link="l_middle_flexion_two"/>
+        <child link="l_middle_flexion_three"/>
+        <origin xyz="0 0 ${-second_bar_length}" rpy="0 0 0"/>
+        <axis xyz="-1 0 0"/>
+        <limit velocity="${1000}"
+               effort="${100}"
+               lower="${0}"
+               upper="${100}"/>
+    </joint>
+    <joint name="l_middle_tip" type="revolute">
+        <parent link="l_middle_flexion_three"/>
+        <child link="l_middle_thimble"/>
+        <origin xyz="0 -0.012342 ${third_bar_length-0.0025}" rpy="0 0 0"/>
+        <axis xyz="-1 0 0"/>
+        <limit velocity="${1000}"
+               effort="${100}"
+               lower="${-4.2}"
+               upper="${100}"/>
     </joint>
     <joint name="l_ring_brake" type="revolute">
@@ -317,3 +406,53 @@
                upper="${100}"/>
     </joint>
+    <joint name="l_ring_tip" type="revolute">
+        <parent link="l_ring_flexion_two"/>
+        <child link="l_ring_flexion_three"/>
+        <origin xyz="0 0 ${-second_bar_length}" rpy="0 0 0"/>
+        <axis xyz="-1 0 0"/>
+        <limit velocity="${1000}"
+               effort="${100}"
+               lower="${0}"
+               upper="${100}"/>
+    </joint>
+    <joint name="l_hub_to_pinky_brake" type="fixed">
+        <parent link="l_glove_hub"/>
+        <child link="l_pinky_brake"/>
+        <origin xyz="${pinky_hub_X} ${pinky_hub_Y} ${pinky_hub_Z}" rpy="0 0 0"/>
+    </joint>
+    <joint name="l_pinky_brake" type="revolute">
+        <parent link="l_pinky_brake"/>
+        <child link="l_pinky_abduction"/>
+        <origin xyz="0 0.0074 ${-0.0}" rpy="0 0 0"/>
+        <axis xyz="0 -1 0"/>
+        <limit velocity="${1000}"
+               effort="${100}"
+               lower="${-2}"
+               upper="${100}"/>
+    </joint>
+    <joint name="l_pinky_abduction" type="fixed">
+        <parent link="l_pinky_abduction"/>
+        <child link="l_pinky_flexion_one"/>
+        <origin xyz="0 0 ${-0.00911-0.01414}" rpy="0 0 0"/>
+    </joint>
+    <joint name="l_pinky_mcp" type="revolute">
+        <parent link="l_pinky_flexion_one"/>
+        <child link="l_pinky_flexion_two"/>
+        <origin xyz="0 0 0" rpy="0 0 0"/>
+        <axis xyz="-1 0 0"/>
+        <limit velocity="${1000}"
+               effort="${100}"
+               lower="${-2}"
+               upper="${100}"/>
+    </joint>
+    <joint name="l_pinky_tip" type="revolute">
+        <parent link="l_pinky_flexion_two"/>
+        <child link="l_pinky_flexion_three"/>
+        <origin xyz="0 0 ${-second_bar_length}" rpy="0 0 0"/>
+        <axis xyz="-1 0 0"/>
+        <limit velocity="${1000}"
+               effort="${100}"
+               lower="${0}"
+               upper="${100}"/>
+    </joint>
 </robot>

File: src/senseglove/senseglove_description/urdf/nova_right.xacro (robot description, xacro)
@@ -2,5 +2,5 @@
 <!-- Revolute-Revolute Manipulator -->
 <robot name="nova" xmlns:xacro="http://www.ros.org/wiki/xacro">
-    <!-- Constants for robot dimensions -->
+   <!-- Constants for robot dimensions -->
     <xacro:property name="PI" value="3.1415926535897931"/>
     <xacro:property name="joint_base_mass" value="1"/> <!-- arbitrary value for joint_base_mass -->
@@ -26,4 +26,7 @@
     <xacro:property name="ring_hub_Y" value="0.008"/>
     <xacro:property name="ring_hub_Z" value="-0.05422"/>
+    <xacro:property name="pinky_hub_X" value="0.03307"/>
+    <xacro:property name="pinky_hub_Y" value="0.00695"/>
+    <xacro:property name="pinky_hub_Z" value="-0.04125"/>
     <xacro:property name="bar_length" value="${0.39}"/>
     <xacro:property name="bar_mass" value="1.080"/>
@@ -82,4 +85,7 @@
         </visual>
     </link>
+    <!-- thumb flexion three -->
+    <link name="r_thumb_flexion_three">
+    </link>
     <!-- index brake -->
     <link name="r_index_brake">
@@ -118,4 +124,7 @@
         </visual>
     </link>
+    <!-- index flexion three -->
+    <link name="r_index_flexion_three">
+    </link>
     <!-- middle brake -->
     <link name="r_middle_brake">
@@ -154,4 +163,7 @@
         </visual>
     </link>
+    <!-- middle flexion three -->
+    <link name="r_middle_flexion_three">
+    </link>
     <!-- ring brake -->
     <link name="r_ring_brake">
@@ -189,4 +201,46 @@
             </geometry>
         </visual>
+    </link>
+    <!-- ring flexion three -->
+    <link name="r_ring_flexion_three">
+    </link>
+    <!-- pinky brake -->
+    <link name="r_pinky_brake">
+        <visual>
+            <origin xyz="${-brake_thickness/2-0.0004} ${-brake_height/2 - 0.0025} ${-first_bar_length-second_bar_length-0.003}" rpy="0 0 0"/>
+            <geometry>
+                <mesh filename="package://senseglove_description/urdf/STL/MK29_DK1_Brake_assembly_v2.STL" scale="0.001 0.001 0.001"/>
+            </geometry>
+        </visual>
+    </link>
+    <!-- pinky abduction -->
+    <link name="r_pinky_abduction">
+        <visual>
+            <origin xyz="${-brake_thickness/2} ${-brake_height+0.006} ${-second_bar_length-first_bar_length-0.003}" rpy="0 0 0"/>
+            <geometry>
+                <mesh filename="package://senseglove_description/urdf/STL/MK29_DK1_Abduction_joint_v2.STL" scale="0.001 0.001 0.001"/>
+            </geometry>
+        </visual>
+    </link>
+    <!-- pinky flexion one -->
+    <link name="r_pinky_flexion_one">
+        <visual>
+            <origin xyz="${-brake_thickness/2} ${-brake_height+0.005} ${-second_bar_length-0.0055}" rpy="0 0 0"/>
+            <geometry>
+                <mesh filename="package://senseglove_description/urdf/STL/MK29_DK1_Flexion_joint_1_v2.STL" scale="0.001 0.001 0.001"/>
+            </geometry>
+        </visual>
+    </link>
+    <!-- pinky flexion two -->
+    <link name="r_pinky_flexion_two">
+        <visual>
+            <origin xyz="${-brake_thickness/2} ${-brake_height+0.005} ${-second_bar_length-0.005355}" rpy="0 0 0"/>
+            <geometry>
+                <mesh filename="package://senseglove_description/urdf/STL/MK29_DK1_Flexion_joint_2_v2.STL" scale="0.001 0.001 0.001"/>
+            </geometry>
+        </visual>
+    </link>
+    <!-- pinky flexion three -->
+    <link name="r_pinky_flexion_three">
     </link>
     <!-- Joints -->
@@ -226,4 +280,14 @@
                upper="${100}"/>
     </joint>
+    <joint name="r_thumb_tip" type="revolute">
+        <parent link="r_thumb_flexion_two"/>
+        <child link="r_thumb_flexion_three"/>
+        <origin xyz="0 0 ${-second_bar_length}" rpy="0 0 0"/>
+        <axis xyz="-1 0 0"/>
+        <limit velocity="${1000}"
+               effort="${100}"
+               lower="${0}"
+               upper="${100}"/>
+    </joint>
     <joint name="r_hub_to_index_brake" type="fixed">
         <parent link="r_glove_hub"/>
@@ -256,4 +320,14 @@
                upper="${100}"/>
     </joint>
+    <joint name="r_index_tip" type="revolute">
+        <parent link="r_index_flexion_two"/>
+        <child link="r_index_flexion_three"/>
+        <origin xyz="0 0 ${-second_bar_length}" rpy="0 0 0"/>
+        <axis xyz="-1 0 0"/>
+        <limit velocity="${1000}"
+               effort="${100}"
+               lower="${0}"
+               upper="${100}"/>
+    </joint>
     <joint name="r_hub_to_middle_brake" type="fixed">
         <parent link="r_glove_hub"/>
@@ -286,4 +360,14 @@
                upper="${100}"/>
     </joint>
+    <joint name="r_middle_tip" type="revolute">
+        <parent link="r_middle_flexion_two"/>
+        <child link="r_middle_flexion_three"/>
+        <origin xyz="0 0 ${-second_bar_length}" rpy="0 0 0"/>
+        <axis xyz="-1 0 0"/>
+        <limit velocity="${1000}"
+               effort="${100}"
+               lower="${0}"
+               upper="${100}"/>
+    </joint>
     <joint name="r_hub_to_ring_brake" type="fixed">
         <parent link="r_glove_hub"/>
@@ -316,3 +400,53 @@
                upper="${100}"/>
     </joint>
+    <joint name="r_ring_tip" type="revolute">
+        <parent link="r_ring_flexion_two"/>
+        <child link="r_ring_flexion_three"/>
+        <origin xyz="0 0 ${-second_bar_length}" rpy="0 0 0"/>
+        <axis xyz="-1 0 0"/>
+        <limit velocity="${1000}"
+               effort="${100}"
+               lower="${0}"
+               upper="${100}"/>
+    </joint>
+    <joint name="r_hub_to_pinky_brake" type="fixed">
+        <parent link="r_glove_hub"/>
+        <child link="r_pinky_brake"/>
+        <origin xyz="${pinky_hub_X} ${pinky_hub_Y} ${pinky_hub_Z}" rpy="0 0 0"/>
+    </joint>
+    <joint name="r_pinky_brake" type="revolute">
+        <parent link="r_pinky_brake"/>
+        <child link="r_pinky_abduction"/>
+        <origin xyz="0 0.0074 ${-0.0}" rpy="0 0 0"/>
+        <axis xyz="0 1 0"/>
+        <limit velocity="${1000}"
+               effort="${100}"
+               lower="${-2}"
+               upper="${100}"/>
+    </joint>
+    <joint name="r_pinky_abduction" type="fixed">
+        <parent link="r_pinky_abduction"/>
+        <child link="r_pinky_flexion_one"/>
+        <origin xyz="0 0 ${-0.00911-0.01414}" rpy="0 0 0"/>
+    </joint>
+    <joint name="r_pinky_mcp" type="revolute">
+        <parent link="r_pinky_flexion_one"/>
+        <child link="r_pinky_flexion_two"/>
+        <origin xyz="0 0 0" rpy="0 0 0"/>
+        <axis xyz="-1 0 0"/>
+        <limit velocity="${1000}"
+               effort="${100}"
+               lower="${-2}"
+               upper="${100}"/>
+    </joint>
+    <joint name="r_pinky_tip" type="revolute">
+        <parent link="r_pinky_flexion_two"/>
+        <child link="r_pinky_flexion_three"/>
+        <origin xyz="0 0 ${-second_bar_length}" rpy="0 0 0"/>
+        <axis xyz="-1 0 0"/>
+        <limit velocity="${1000}"
+               effort="${100}"
+               lower="${0}"
+               upper="${100}"/>
+    </joint>
 </robot>

Commit message: Added bash scripts for bluetooth pairing, minor fixes on urdf, improved structure2

File: src/senseglove/senseglove_description/urdf/nova_left.xacro (robot description, xacro)
@@ -361,5 +361,5 @@
                upper="${100}"/>
     </joint>
-    <joint name="l_middle_pip" type="revolute">
+    <joint name="l_middle_tip" type="revolute">
         <parent link="l_middle_flexion_two"/>
         <child link="l_middle_flexion_three"/>
@@ -371,13 +371,8 @@
                upper="${100}"/>
     </joint>
-    <joint name="l_middle_tip" type="revolute">
-        <parent link="l_middle_flexion_three"/>
-        <child link="l_middle_thimble"/>
-        <origin xyz="0 -0.012342 ${third_bar_length-0.0025}" rpy="0 0 0"/>
-        <axis xyz="-1 0 0"/>
-        <limit velocity="${1000}"
-               effort="${100}"
-               lower="${-4.2}"
-               upper="${100}"/>
+    <joint name="l_hub_to_ring_brake" type="fixed">
+        <parent link="l_glove_hub"/>
+        <child link="l_ring_brake"/>
+        <origin xyz="${ring_hub_X} ${ring_hub_Y} ${ring_hub_Z}" rpy="0 0 0"/>
     </joint>
     <joint name="l_ring_brake" type="revolute">
