Commit message: implemented a more universal joint configuration for haptics

File: src/senseglove/senseglove_description/urdf/nova_left.xacro (robot description, xacro)
@@ -2,5 +2,5 @@
 <!-- Revolute-Revolute Manipulator -->
 <robot name="nova" xmlns:xacro="http://www.ros.org/wiki/xacro">
-   <!-- Constants for robot dimensions -->
+<!-- Constants for robot dimensions -->
     <xacro:property name="PI" value="3.1415926535897931"/>
     <xacro:property name="joint_base_mass" value="1"/> <!-- arbitrary value for joint_base_mass -->
@@ -87,4 +87,19 @@
     <!-- thumb flexion three -->
     <link name="l_thumb_flexion_three">
+        <visual>
+            <origin xyz="${-brake_thickness/2} ${-brake_height+0.00533} -0.00533" rpy="0 0 0"/>
+            <geometry>
+                <mesh filename="package://senseglove_description/urdf/STL/MK29_DK1_Flexion_joint_3_v2.STL" scale="0.001 0.001 0.001"/>
+            </geometry>
+        </visual>
+    </link>
+    <!-- thumb thimble -->
+    <link name="l_thumb_thimble">
+        <visual>
+            <origin xyz="${-brake_thickness/2} -0.014951 ${-third_bar_length-0.0028}" rpy="0 0 0"/>
+            <geometry>
+                <mesh filename="package://senseglove_description/urdf/STL/MK29_DK1_Thimble_v2.STL" scale="0.001 0.001 0.001"/>
+            </geometry>
+        </visual>
     </link>
     <!-- index brake -->
@@ -126,4 +141,19 @@
     <!-- index flexion three -->
     <link name="l_index_flexion_three">
+        <visual>
+            <origin xyz="${-brake_thickness/2} ${-brake_height+0.00533} -0.00533" rpy="0 0 0"/>
+            <geometry>
+                <mesh filename="package://senseglove_description/urdf/STL/MK29_DK1_Flexion_joint_3_v2.STL" scale="0.001 0.001 0.001"/>
+            </geometry>
+        </visual>
+    </link>
+    <!-- index thimble -->
+    <link name="l_index_thimble">
+        <visual>
+            <origin xyz="${-brake_thickness/2} -0.014951 ${-third_bar_length-0.0028}" rpy="0 0 0"/>
+            <geometry>
+                <mesh filename="package://senseglove_description/urdf/STL/MK29_DK1_Thimble_v2.STL" scale="0.001 0.001 0.001"/>
+            </geometry>
+        </visual>
     </link>
     <!-- middle brake -->
@@ -165,4 +195,19 @@
     <!-- middle flexion three -->
     <link name="l_middle_flexion_three">
+        <visual>
+            <origin xyz="${-brake_thickness/2} ${-brake_height+0.00533} -0.00533" rpy="0 0 0"/>
+            <geometry>
+                <mesh filename="package://senseglove_description/urdf/STL/MK29_DK1_Flexion_joint_3_v2.STL" scale="0.001 0.001 0.001"/>
+            </geometry>
+        </visual>
+    </link>
+    <!-- middle thimble -->
+    <link name="l_middle_thimble">
+        <visual>
+            <origin xyz="${-brake_thickness/2} -0.014951 ${-third_bar_length-0.0028}" rpy="0 0 0"/>
+            <geometry>
+                <mesh filename="package://senseglove_description/urdf/STL/MK29_DK1_Thimble_v2.STL" scale="0.001 0.001 0.001"/>
+            </geometry>
+        </visual>
     </link>
     <!-- ring brake -->
@@ -204,4 +249,19 @@
     <!-- ring flexion three -->
     <link name="l_ring_flexion_three">
+        <visual>
+            <origin xyz="${-brake_thickness/2} ${-brake_height+0.00533} -0.00533" rpy="0 0 0"/>
+            <geometry>
+                <mesh filename="package://senseglove_description/urdf/STL/MK29_DK1_Flexion_joint_3_v2.STL" scale="0.001 0.001 0.001"/>
+            </geometry>
+        </visual>
+    </link>
+    <!-- ring thimble -->
+    <link name="l_ring_thimble">
+        <visual>
+            <origin xyz="${-brake_thickness/2} -0.014951 ${-third_bar_length-0.0028}" rpy="0 0 0"/>
+            <geometry>
+                <mesh filename="package://senseglove_description/urdf/STL/MK29_DK1_Thimble_v2.STL" scale="0.001 0.001 0.001"/>
+            </geometry>
+        </visual>
     </link>
     <!-- pinky brake -->
@@ -243,4 +303,19 @@
     <!-- pinky flexion three -->
     <link name="l_pinky_flexion_three">
+        <visual>
+            <origin xyz="${-brake_thickness/2} ${-brake_height+0.00533} -0.00533" rpy="0 0 0"/>
+            <geometry>
+                <mesh filename="package://senseglove_description/urdf/STL/MK29_DK1_Flexion_joint_3_v2.STL" scale="0.001 0.001 0.001"/>
+            </geometry>
+        </visual>
+    </link>
+    <!-- pinky thimble -->
+    <link name="l_pinky_thimble">
+        <visual>
+            <origin xyz="${-brake_thickness/2} -0.014951 ${-third_bar_length-0.0028}" rpy="0 0 0"/>
+            <geometry>
+                <mesh filename="package://senseglove_description/urdf/STL/MK29_DK1_Thimble_v2.STL" scale="0.001 0.001 0.001"/>
+            </geometry>
+        </visual>
     </link>
     <!-- Joints -->
@@ -280,5 +355,5 @@
                upper="${100}"/>
     </joint>
-    <joint name="l_thumb_tip" type="revolute">
+    <joint name="l_thumb_pip" type="revolute">
         <parent link="l_thumb_flexion_two"/>
         <child link="l_thumb_flexion_three"/>
@@ -288,4 +363,14 @@
                effort="${100}"
                lower="${0}"
+               upper="${100}"/>
+    </joint>
+    <joint name="l_thumb_dip" type="revolute">
+        <parent link="l_thumb_flexion_three"/>
+        <child link="l_thumb_thimble"/>
+        <origin xyz="0 -0.012342 ${third_bar_length-0.0025}" rpy="0 0 0"/>
+        <axis xyz="-1 0 0"/>
+        <limit velocity="${1000}"
+               effort="${100}"
+               lower="${-4.2}"
                upper="${100}"/>
     </joint>
@@ -320,5 +405,5 @@
                upper="${100}"/>
     </joint>
-    <joint name="l_index_tip" type="revolute">
+    <joint name="l_index_pip" type="revolute">
         <parent link="l_index_flexion_two"/>
         <child link="l_index_flexion_three"/>
@@ -328,4 +413,14 @@
                effort="${100}"
                lower="${0}"
+               upper="${100}"/>
+    </joint>
+    <joint name="l_index_dip" type="revolute">
+        <parent link="l_index_flexion_three"/>
+        <child link="l_index_thimble"/>
+        <origin xyz="0 -0.012342 ${third_bar_length-0.0025}" rpy="0 0 0"/>
+        <axis xyz="-1 0 0"/>
+        <limit velocity="${1000}"
+               effort="${100}"
+               lower="${-4.2}"
                upper="${100}"/>
     </joint>
@@ -361,5 +456,5 @@
                upper="${100}"/>
     </joint>
-    <joint name="l_middle_tip" type="revolute">
+    <joint name="l_middle_pip" type="revolute">
         <parent link="l_middle_flexion_two"/>
         <child link="l_middle_flexion_three"/>
@@ -369,4 +464,14 @@
                effort="${100}"
                lower="${0}"
+               upper="${100}"/>
+    </joint>
+    <joint name="l_middle_dip" type="revolute">
+        <parent link="l_middle_flexion_three"/>
+        <child link="l_middle_thimble"/>
+        <origin xyz="0 -0.012342 ${third_bar_length-0.0025}" rpy="0 0 0"/>
+        <axis xyz="-1 0 0"/>
+        <limit velocity="${1000}"
+               effort="${100}"
+               lower="${-4.2}"
                upper="${100}"/>
     </joint>
@@ -401,5 +506,5 @@
                upper="${100}"/>
     </joint>
-    <joint name="l_ring_tip" type="revolute">
+    <joint name="l_ring_pip" type="revolute">
         <parent link="l_ring_flexion_two"/>
         <child link="l_ring_flexion_three"/>
@@ -409,4 +514,14 @@
                effort="${100}"
                lower="${0}"
+               upper="${100}"/>
+    </joint>
+    <joint name="l_ring_dip" type="revolute">
+        <parent link="l_ring_flexion_three"/>
+        <child link="l_ring_thimble"/>
+        <origin xyz="0 -0.012342 ${third_bar_length-0.0025}" rpy="0 0 0"/>
+        <axis xyz="-1 0 0"/>
+        <limit velocity="${1000}"
+               effort="${100}"
+               lower="${-4.2}"
                upper="${100}"/>
     </joint>
@@ -441,5 +556,5 @@
                upper="${100}"/>
     </joint>
-    <joint name="l_pinky_tip" type="revolute">
+    <joint name="l_pinky_pip" type="revolute">
         <parent link="l_pinky_flexion_two"/>
         <child link="l_pinky_flexion_three"/>
@@ -451,3 +566,13 @@
                upper="${100}"/>
     </joint>
+    <joint name="l_pinky_dip" type="revolute">
+        <parent link="l_pinky_flexion_three"/>
+        <child link="l_pinky_thimble"/>
+        <origin xyz="0 -0.012342 ${third_bar_length-0.0025}" rpy="0 0 0"/>
+        <axis xyz="-1 0 0"/>
+        <limit velocity="${1000}"
+               effort="${100}"
+               lower="${-4.2}"
+               upper="${100}"/>
+    </joint>
 </robot>

File: src/senseglove/senseglove_description/urdf/nova_right.xacro (robot description, xacro)
@@ -2,5 +2,5 @@
 <!-- Revolute-Revolute Manipulator -->
 <robot name="nova" xmlns:xacro="http://www.ros.org/wiki/xacro">
-   <!-- Constants for robot dimensions -->
+    <!-- Constants for robot dimensions -->
     <xacro:property name="PI" value="3.1415926535897931"/>
     <xacro:property name="joint_base_mass" value="1"/> <!-- arbitrary value for joint_base_mass -->
@@ -87,4 +87,19 @@
     <!-- thumb flexion three -->
     <link name="r_thumb_flexion_three">
+        <visual>
+            <origin xyz="${-brake_thickness/2} ${-brake_height+0.00533} -0.00533" rpy="0 0 0"/>
+            <geometry>
+                <mesh filename="package://senseglove_description/urdf/STL/MK29_DK1_Flexion_joint_3_v2.STL" scale="0.001 0.001 0.001"/>
+            </geometry>
+        </visual>
+    </link>
+    <!-- thumb thimble -->
+    <link name="r_thumb_thimble">
+        <visual>
+            <origin xyz="${-brake_thickness/2} -0.014951 ${-third_bar_length-0.0028}" rpy="0 0 0"/>
+            <geometry>
+                <mesh filename="package://senseglove_description/urdf/STL/MK29_DK1_Thimble_v2.STL" scale="0.001 0.001 0.001"/>
+            </geometry>
+        </visual>
     </link>
     <!-- index brake -->
@@ -126,4 +141,19 @@
     <!-- index flexion three -->
     <link name="r_index_flexion_three">
+        <visual>
+            <origin xyz="${-brake_thickness/2} ${-brake_height+0.00533} -0.00533" rpy="0 0 0"/>
+            <geometry>
+                <mesh filename="package://senseglove_description/urdf/STL/MK29_DK1_Flexion_joint_3_v2.STL" scale="0.001 0.001 0.001"/>
+            </geometry>
+        </visual>
+    </link>
+    <!-- index thimble -->
+    <link name="r_index_thimble">
+        <visual>
+            <origin xyz="${-brake_thickness/2} -0.014951 ${-third_bar_length-0.0028}" rpy="0 0 0"/>
+            <geometry>
+                <mesh filename="package://senseglove_description/urdf/STL/MK29_DK1_Thimble_v2.STL" scale="0.001 0.001 0.001"/>
+            </geometry>
+        </visual>
     </link>
     <!-- middle brake -->
@@ -165,4 +195,19 @@
     <!-- middle flexion three -->
     <link name="r_middle_flexion_three">
+        <visual>
+            <origin xyz="${-brake_thickness/2} ${-brake_height+0.00533} -0.00533" rpy="0 0 0"/>
+            <geometry>
+                <mesh filename="package://senseglove_description/urdf/STL/MK29_DK1_Flexion_joint_3_v2.STL" scale="0.001 0.001 0.001"/>
+            </geometry>
+        </visual>
+    </link>
+    <!-- middle thimble -->
+    <link name="r_middle_thimble">
+        <visual>
+            <origin xyz="${-brake_thickness/2} -0.014951 ${-third_bar_length-0.0028}" rpy="0 0 0"/>
+            <geometry>
+                <mesh filename="package://senseglove_description/urdf/STL/MK29_DK1_Thimble_v2.STL" scale="0.001 0.001 0.001"/>
+            </geometry>
+        </visual>
     </link>
     <!-- ring brake -->
@@ -204,4 +249,19 @@
     <!-- ring flexion three -->
     <link name="r_ring_flexion_three">
+        <visual>
+            <origin xyz="${-brake_thickness/2} ${-brake_height+0.00533} -0.00533" rpy="0 0 0"/>
+            <geometry>
+                <mesh filename="package://senseglove_description/urdf/STL/MK29_DK1_Flexion_joint_3_v2.STL" scale="0.001 0.001 0.001"/>
+            </geometry>
+        </visual>
+    </link>
+    <!-- ring thimble -->
+    <link name="r_ring_thimble">
+        <visual>
+            <origin xyz="${-brake_thickness/2} -0.014951 ${-third_bar_length-0.0028}" rpy="0 0 0"/>
+            <geometry>
+                <mesh filename="package://senseglove_description/urdf/STL/MK29_DK1_Thimble_v2.STL" scale="0.001 0.001 0.001"/>
+            </geometry>
+        </visual>
     </link>
     <!-- pinky brake -->
@@ -243,4 +303,19 @@
     <!-- pinky flexion three -->
     <link name="r_pinky_flexion_three">
+        <visual>
+            <origin xyz="${-brake_thickness/2} ${-brake_height+0.00533} -0.00533" rpy="0 0 0"/>
+            <geometry>
+                <mesh filename="package://senseglove_description/urdf/STL/MK29_DK1_Flexion_joint_3_v2.STL" scale="0.001 0.001 0.001"/>
+            </geometry>
+        </visual>
+    </link>
+    <!-- pinky thimble -->
+    <link name="r_pinky_thimble">
+        <visual>
+            <origin xyz="${-brake_thickness/2} -0.014951 ${-third_bar_length-0.0028}" rpy="0 0 0"/>
+            <geometry>
+                <mesh filename="package://senseglove_description/urdf/STL/MK29_DK1_Thimble_v2.STL" scale="0.001 0.001 0.001"/>
+            </geometry>
+        </visual>
     </link>
     <!-- Joints -->
@@ -280,8 +355,18 @@
                upper="${100}"/>
     </joint>
-    <joint name="r_thumb_tip" type="revolute">
+    <joint name="r_thumb_pip" type="revolute">
         <parent link="r_thumb_flexion_two"/>
         <child link="r_thumb_flexion_three"/>
         <origin xyz="0 0 ${-second_bar_length}" rpy="0 0 0"/>
+        <axis xyz="-1 0 0"/>
+        <limit velocity="${1000}"
+               effort="${100}"
+               lower="${0}"
+               upper="${100}"/>
+    </joint>
+    <joint name="r_thumb_dip" type="revolute">
+        <parent link="r_thumb_flexion_three"/>
+        <child link="r_thumb_thimble"/>
+        <origin xyz="0 -0.012342 ${third_bar_length-0.0025}" rpy="0 0 0"/>
         <axis xyz="-1 0 0"/>
         <limit velocity="${1000}"
@@ -320,5 +405,5 @@
                upper="${100}"/>
     </joint>
-    <joint name="r_index_tip" type="revolute">
+    <joint name="r_index_pip" type="revolute">
         <parent link="r_index_flexion_two"/>
         <child link="r_index_flexion_three"/>
@@ -328,4 +413,14 @@
                effort="${100}"
                lower="${0}"
+               upper="${100}"/>
+    </joint>
+    <joint name="r_index_dip" type="revolute">
+        <parent link="r_index_flexion_three"/>
+        <child link="r_index_thimble"/>
+        <origin xyz="0 -0.012342 ${third_bar_length-0.0025}" rpy="0 0 0"/>
+        <axis xyz="-1 0 0"/>
+        <limit velocity="${1000}"
+               effort="${100}"
+               lower="${-4.2}"
                upper="${100}"/>
     </joint>
@@ -360,5 +455,5 @@
                upper="${100}"/>
     </joint>
-    <joint name="r_middle_tip" type="revolute">
+    <joint name="r_middle_pip" type="revolute">
         <parent link="r_middle_flexion_two"/>
         <child link="r_middle_flexion_three"/>
@@ -368,4 +463,14 @@
                effort="${100}"
                lower="${0}"
+               upper="${100}"/>
+    </joint>
+    <joint name="r_middle_dip" type="revolute">
+        <parent link="r_middle_flexion_three"/>
+        <child link="r_middle_thimble"/>
+        <origin xyz="0 -0.012342 ${third_bar_length-0.0025}" rpy="0 0 0"/>
+        <axis xyz="-1 0 0"/>
+        <limit velocity="${1000}"
+               effort="${100}"
+               lower="${-4.2}"
                upper="${100}"/>
     </joint>
@@ -400,5 +505,5 @@
                upper="${100}"/>
     </joint>
-    <joint name="r_ring_tip" type="revolute">
+    <joint name="r_ring_pip" type="revolute">
         <parent link="r_ring_flexion_two"/>
         <child link="r_ring_flexion_three"/>
@@ -408,4 +513,14 @@
                effort="${100}"
                lower="${0}"
+               upper="${100}"/>
+    </joint>
+    <joint name="r_ring_dip" type="revolute">
+        <parent link="r_ring_flexion_three"/>
+        <child link="r_ring_thimble"/>
+        <origin xyz="0 -0.012342 ${third_bar_length-0.0025}" rpy="0 0 0"/>
+        <axis xyz="-1 0 0"/>
+        <limit velocity="${1000}"
+               effort="${100}"
+               lower="${-4.2}"
                upper="${100}"/>
     </joint>
@@ -440,5 +555,5 @@
                upper="${100}"/>
     </joint>
-    <joint name="r_pinky_tip" type="revolute">
+    <joint name="r_pinky_pip" type="revolute">
         <parent link="r_pinky_flexion_two"/>
         <child link="r_pinky_flexion_three"/>
@@ -450,3 +565,23 @@
                upper="${100}"/>
     </joint>
+    <joint name="r_pinky_dip" type="revolute">
+        <parent link="r_pinky_flexion_three"/>
+        <child link="r_pinky_thimble"/>
+        <origin xyz="0 -0.012342 ${third_bar_length-0.0025}" rpy="0 0 0"/>
+        <axis xyz="-1 0 0"/>
+        <limit velocity="${1000}"
+               effort="${100}"
+               lower="${-4.2}"
+               upper="${100}"/>
+    </joint>
+    <joint name="r_thumper" type="revolute">
+        <parent link="r_glove_hub"/>
+        <child link="r_middle_brake"/>
+        <origin xyz="0 0 0" rpy="0 0 0"/>
+        <axis xyz="-1 0 0"/>
+        <limit velocity="${1000}"
+               effort="${100}"
+               lower="${-2}"
+               upper="${100}"/>
+    </joint>
 </robot>

Commit message: Updated to SenseCom v1.6.1, minor fix on nova yaml

File: src/senseglove/senseglove_description/urdf/nova2_left.xacro (robot description, xacro)
@@ -444,5 +444,4 @@
         <child link="l_middle_flexion_one"/>
         <origin xyz="0 0 ${-0.00911-0.01414}" rpy="0 0 0"/>
--
     </joint>
     <joint name="l_middle_mcp" type="revolute">
@@ -566,4 +565,14 @@
                upper="${100}"/>
     </joint>
+    <joint name="l_pinky_dip" type="revolute">
+        <parent link="l_pinky_flexion_three"/>
+        <child link="l_pinky_thimble"/>
+        <origin xyz="0 -0.012342 ${third_bar_length-0.0025}" rpy="0 0 0"/>
+        <axis xyz="-1 0 0"/>
+        <limit velocity="${1000}"
+               effort="${100}"
+               lower="${-4.2}"
+               upper="${100}"/>
+    </joint>
     <joint name="l_palm_strap" type="revolute">
         <parent link="l_glove_hub"/>

File: src/senseglove/senseglove_description/urdf/nova2_right.xacro (robot description, xacro)
@@ -575,5 +575,15 @@
                upper="${100}"/>
     </joint>
-    <joint name="r_palm_index" type="revolute">
+    <joint name="r_palm_strap" type="revolute">
+        <parent link="r_glove_hub"/>
+        <child link="r_middle_brake"/>
+        <origin xyz="0 0 0" rpy="0 0 0"/>
+        <axis xyz="-1 0 0"/>
+        <limit velocity="${1000}"
+               effort="${100}"
+               lower="${-2}"
+               upper="${100}"/>
+    </joint>
+        <joint name="r_palm_index" type="revolute">
         <parent link="r_glove_hub"/>
         <child link="r_index_brake"/>
@@ -585,5 +595,5 @@
                upper="${100}"/>
     </joint>
-    <joint name="r_palm_pinky" type="revolute">
+        <joint name="r_palm_pinky" type="revolute">
         <parent link="r_glove_hub"/>
         <child link="r_pinky_brake"/>
@@ -595,13 +605,3 @@
                upper="${100}"/>
     </joint>
-    <joint name="r_palm_strap" type="revolute">
-        <parent link="r_glove_hub"/>
-        <child link="r_middle_brake"/>
-        <origin xyz="0 0 0" rpy="0 0 0"/>
-        <axis xyz="-1 0 0"/>
-        <limit velocity="${1000}"
-               effort="${100}"
-               lower="${-2}"
-               upper="${100}"/>
-    </joint>
 </robot>

File: src/senseglove/senseglove_description/urdf/nova_left.xacro (robot description, xacro)
@@ -576,3 +576,13 @@
                upper="${100}"/>
     </joint>
+    <joint name="l_thumper" type="revolute">
+        <parent link="l_glove_hub"/>
+        <child link="l_middle_brake"/>
+        <origin xyz="0 0 0" rpy="0 0 0"/>
+        <axis xyz="-1 0 0"/>
+        <limit velocity="${1000}"
+               effort="${100}"
+               lower="${-2}"
+               upper="${100}"/>
+    </joint>
 </robot>
