Commit message: Haptic Fixes for Nova & Nova2

File: src/senseglove/senseglove_description/urdf/nova2_left.xacro (robot description, xacro)
@@ -319,4 +319,31 @@
         </visual>
     </link>
+    <!-- l_palm_strap -->
+    <link name="l_palm_strap">
+        <visual>
+            <origin xyz="${-brake_thickness/2} ${-brake_height+0.006} ${-second_bar_length-first_bar_length-0.003}" rpy="0 0 0"/>
+            <geometry>
+                <mesh filename="package://senseglove_description/urdf/STL/MK29_DK1_Abduction_joint_v2.STL" scale="0.001 0.001 0.001"/>
+            </geometry>
+        </visual>
+    </link>
+    <!-- l_palm_index -->
+    <link name="l_palm_index">
+        <visual>
+            <origin xyz="${-brake_thickness/2} ${-brake_height+0.006} ${-second_bar_length-first_bar_length-0.003}" rpy="0 0 0"/>
+            <geometry>
+                <mesh filename="package://senseglove_description/urdf/STL/MK29_DK1_Abduction_joint_v2.STL" scale="0.001 0.001 0.001"/>
+            </geometry>
+        </visual>
+    </link>
+    <!-- l_palm_pinky -->
+    <link name="l_palm_pinky">
+        <visual>
+            <origin xyz="${-brake_thickness/2} ${-brake_height+0.006} ${-second_bar_length-first_bar_length-0.003}" rpy="0 0 0"/>
+            <geometry>
+                <mesh filename="package://senseglove_description/urdf/STL/MK29_DK1_Abduction_joint_v2.STL" scale="0.001 0.001 0.001"/>
+            </geometry>
+        </visual>
+    </link>
     <!-- Joints -->
     <joint name="l_joint_base_fixed_parent_joint" type="fixed">
@@ -577,5 +604,5 @@
     <joint name="l_palm_strap" type="revolute">
         <parent link="l_glove_hub"/>
-        <child link="l_middle_brake"/>
+        <child link="l_palm_strap"/>
         <origin xyz="0 0 0" rpy="0 0 0"/>
         <axis xyz="-1 0 0"/>
@@ -587,5 +614,5 @@
         <joint name="l_palm_index" type="revolute">
         <parent link="l_glove_hub"/>
-        <child link="l_index_brake"/>
+        <child link="l_palm_index"/>
         <origin xyz="0 0 0" rpy="0 0 0"/>
         <axis xyz="-1 0 0"/>
@@ -597,5 +624,5 @@
         <joint name="l_palm_pinky" type="revolute">
         <parent link="l_glove_hub"/>
-        <child link="l_pinky_brake"/>
+        <child link="l_palm_pinky"/>
         <origin xyz="0 0 0" rpy="0 0 0"/>
         <axis xyz="-1 0 0"/>

File: src/senseglove/senseglove_description/urdf/nova2_right.xacro (robot description, xacro)
@@ -319,4 +319,31 @@
         </visual>
     </link>
+    <!-- r_palm_strap -->
+    <link name="r_palm_strap">
+        <visual>
+            <origin xyz="${-brake_thickness/2} ${-brake_height+0.006} ${-second_bar_length-first_bar_length-0.003}" rpy="0 0 0"/>
+            <geometry>
+                <mesh filename="package://senseglove_description/urdf/STL/MK29_DK1_Abduction_joint_v2.STL" scale="0.001 0.001 0.001"/>
+            </geometry>
+        </visual>
+    </link>
+    <!-- r_palm_index -->
+    <link name="r_palm_index">
+        <visual>
+            <origin xyz="${-brake_thickness/2} ${-brake_height+0.006} ${-second_bar_length-first_bar_length-0.003}" rpy="0 0 0"/>
+            <geometry>
+                <mesh filename="package://senseglove_description/urdf/STL/MK29_DK1_Abduction_joint_v2.STL" scale="0.001 0.001 0.001"/>
+            </geometry>
+        </visual>
+    </link>
+    <!-- r_palm_pinky -->
+    <link name="r_palm_pinky">
+        <visual>
+            <origin xyz="${-brake_thickness/2} ${-brake_height+0.006} ${-second_bar_length-first_bar_length-0.003}" rpy="0 0 0"/>
+            <geometry>
+                <mesh filename="package://senseglove_description/urdf/STL/MK29_DK1_Abduction_joint_v2.STL" scale="0.001 0.001 0.001"/>
+            </geometry>
+        </visual>
+    </link>
     <!-- Joints -->
     <joint name="joint_base_fixed_parent_joint" type="fixed">
@@ -577,5 +604,5 @@
     <joint name="r_palm_strap" type="revolute">
         <parent link="r_glove_hub"/>
-        <child link="r_middle_brake"/>
+        <child link="r_palm_strap"/>
         <origin xyz="0 0 0" rpy="0 0 0"/>
         <axis xyz="-1 0 0"/>
@@ -587,5 +614,5 @@
         <joint name="r_palm_index" type="revolute">
         <parent link="r_glove_hub"/>
-        <child link="r_index_brake"/>
+        <child link="r_palm_index"/>
         <origin xyz="0 0 0" rpy="0 0 0"/>
         <axis xyz="-1 0 0"/>
@@ -597,5 +624,5 @@
         <joint name="r_palm_pinky" type="revolute">
         <parent link="r_glove_hub"/>
-        <child link="r_pinky_brake"/>
+        <child link="r_palm_pinky"/>
         <origin xyz="0 0 0" rpy="0 0 0"/>
         <axis xyz="-1 0 0"/>

File: src/senseglove/senseglove_description/urdf/nova_left.xacro (robot description, xacro)
@@ -319,4 +319,13 @@
         </visual>
     </link>
+    <!-- Thumper -->
+    <link name="thumper">
+        <visual>
+            <origin xyz="${-brake_thickness/2} ${-brake_height+0.006} ${-second_bar_length-first_bar_length-0.003}" rpy="0 0 0"/>
+            <geometry>
+                <mesh filename="package://senseglove_description/urdf/STL/MK29_DK1_Abduction_joint_v2.STL" scale="0.001 0.001 0.001"/>
+            </geometry>
+        </visual>
+    </link>
     <!-- Joints -->
     <joint name="l_joint_base_fixed_parent_joint" type="fixed">
@@ -578,5 +587,5 @@
     <joint name="l_thumper" type="revolute">
         <parent link="l_glove_hub"/>
-        <child link="l_middle_brake"/>
+        <child link="thumper"/>
         <origin xyz="0 0 0" rpy="0 0 0"/>
         <axis xyz="-1 0 0"/>
