Commit message: Added IMU function, Fixed service name convention, Added TF broadcaster, and grouped python scripts into one main 'Interaction' Folder

File: src/senseglove/senseglove_description/urdf/nova1/nova_right.xacro (robot description, xacro)
@@ -191,5 +191,5 @@
         <parent link="world"/>
         <child link="r_glove_hub"/>
-        <origin xyz="0.5 0 ${hover_height}" rpy="${90*pi/180} 0 ${180*pi/180}"/>
+        <origin xyz="0.5 0 ${hover_height}" rpy="0 0 0"/>
     </joint>
     <joint name="r_thumb_brake" type="revolute">
