Commit message: Built senseglove_description

File: senseglove/senseglove_description/urdf/dk1/dk1_left.xacro (robot description, xacro)
@@ -45,5 +45,5 @@
             <origin xyz="0.056692 -0.01955 -0.06803" rpy="0 0 0"/>
             <geometry>
-                <mesh filename="package://senseglove_description/urdf/STL/MK29_DK1_HUB.STL" scale="-0.001 0.001 0.001"/>
+                <mesh filename="package://senseglove_description/urdf/dk1/MK29_DK1_HUB.STL" scale="-0.001 0.001 0.001"/>
             </geometry>
         </visual>
@@ -54,5 +54,5 @@
             <origin xyz="${-brake_thickness/2} ${-brake_height/2 - 0.0025} ${-first_bar_length-second_bar_length}" rpy="0 0 0"/>
             <geometry>
-                <mesh filename="package://senseglove_description/urdf/STL/MK29_DK1_Brake_assembly_v2.STL" scale="0.001 0.001 0.001"/>
+                <mesh filename="package://senseglove_description/urdf/dk1/MK29_DK1_Brake_assembly_v2.STL" scale="0.001 0.001 0.001"/>
             </geometry>
         </visual>
@@ -63,5 +63,5 @@
             <origin xyz="${-brake_thickness/2} ${-brake_height+0.006} ${-second_bar_length-first_bar_length-0.003}" rpy="0 0 0"/>
             <geometry>
-                <mesh filename="package://senseglove_description/urdf/STL/MK29_DK1_Abduction_joint_v2.STL" scale="0.001 0.001 0.001"/>
+                <mesh filename="package://senseglove_description/urdf/dk1/MK29_DK1_Abduction_joint_v2.STL" scale="0.001 0.001 0.001"/>
             </geometry>
         </visual>
@@ -72,5 +72,5 @@
             <origin xyz="${-brake_thickness/2} ${-brake_height+0.005} ${-second_bar_length-0.0055}" rpy="0 0 0"/>
             <geometry>
-                <mesh filename="package://senseglove_description/urdf/STL/MK29_DK1_Flexion_joint_1_v2.STL" scale="0.001 0.001 0.001"/>
+                <mesh filename="package://senseglove_description/urdf/dk1/MK29_DK1_Flexion_joint_1_v2.STL" scale="0.001 0.001 0.001"/>
             </geometry>
         </visual>
@@ -81,5 +81,5 @@
             <origin xyz="${-brake_thickness/2} ${-brake_height+0.005} ${-second_bar_length-0.005355}" rpy="0 0 0"/>
             <geometry>
-                <mesh filename="package://senseglove_description/urdf/STL/MK29_DK1_Flexion_joint_2_v2.STL" scale="0.001 0.001 0.001"/>
+                <mesh filename="package://senseglove_description/urdf/dk1/MK29_DK1_Flexion_joint_2_v2.STL" scale="0.001 0.001 0.001"/>
             </geometry>
         </visual>
@@ -90,5 +90,5 @@
             <origin xyz="${-brake_thickness/2} ${-brake_height+0.00533} -0.00533" rpy="0 0 0"/>
             <geometry>
-                <mesh filename="package://senseglove_description/urdf/STL/MK29_DK1_Flexion_joint_3_v2.STL" scale="0.001 0.001 0.001"/>
+                <mesh filename="package://senseglove_description/urdf/dk1/MK29_DK1_Flexion_joint_3_v2.STL" scale="0.001 0.001 0.001"/>
             </geometry>
         </visual>
@@ -99,5 +99,5 @@
             <origin xyz="${-brake_thickness/2} -0.014951 ${-third_bar_length-0.0028}" rpy="0 0 0"/>
             <geometry>
-                <mesh filename="package://senseglove_description/urdf/STL/MK29_DK1_Thimble_v2.STL" scale="0.001 0.001 0.001"/>
+                <mesh filename="package://senseglove_description/urdf/dk1/MK29_DK1_Thimble_v2.STL" scale="0.001 0.001 0.001"/>
             </geometry>
         </visual>
@@ -108,5 +108,5 @@
             <origin xyz="${-brake_thickness/2} ${-brake_height/2 - 0.0025} ${-first_bar_length-second_bar_length}" rpy="0 0 0"/>
             <geometry>
-                <mesh filename="package://senseglove_description/urdf/STL/MK29_DK1_Brake_assembly_v2.STL" scale="0.001 0.001 0.001"/>
+                <mesh filename="package://senseglove_description/urdf/dk1/MK29_DK1_Brake_assembly_v2.STL" scale="0.001 0.001 0.001"/>
             </geometry>
         </visual>
@@ -117,5 +117,5 @@
             <origin xyz="${-brake_thickness/2} ${-brake_height+0.006} ${-second_bar_length-first_bar_length-0.003}" rpy="0 0 0"/>
             <geometry>
-                <mesh filename="package://senseglove_description/urdf/STL/MK29_DK1_Abduction_joint_v2.STL" scale="0.001 0.001 0.001"/>
+                <mesh filename="package://senseglove_description/urdf/dk1/MK29_DK1_Abduction_joint_v2.STL" scale="0.001 0.001 0.001"/>
             </geometry>
         </visual>
@@ -126,5 +126,5 @@
             <origin xyz="${-brake_thickness/2} ${-brake_height+0.005} ${-second_bar_length-0.0055}" rpy="0 0 0"/>
             <geometry>
-                <mesh filename="package://senseglove_description/urdf/STL/MK29_DK1_Flexion_joint_1_v2.STL" scale="0.001 0.001 0.001"/>
+                <mesh filename="package://senseglove_description/urdf/dk1/MK29_DK1_Flexion_joint_1_v2.STL" scale="0.001 0.001 0.001"/>
             </geometry>
         </visual>
@@ -135,5 +135,5 @@
             <origin xyz="${-brake_thickness/2} ${-brake_height+0.005} ${-second_bar_length-0.005355}" rpy="0 0 0"/>
             <geometry>
-                <mesh filename="package://senseglove_description/urdf/STL/MK29_DK1_Flexion_joint_2_v2.STL" scale="0.001 0.001 0.001"/>
+                <mesh filename="package://senseglove_description/urdf/dk1/MK29_DK1_Flexion_joint_2_v2.STL" scale="0.001 0.001 0.001"/>
             </geometry>
         </visual>
@@ -144,5 +144,5 @@
             <origin xyz="${-brake_thickness/2} ${-brake_height+0.00533} -0.00533" rpy="0 0 0"/>
             <geometry>
-                <mesh filename="package://senseglove_description/urdf/STL/MK29_DK1_Flexion_joint_3_v2.STL" scale="0.001 0.001 0.001"/>
+                <mesh filename="package://senseglove_description/urdf/dk1/MK29_DK1_Flexion_joint_3_v2.STL" scale="0.001 0.001 0.001"/>
             </geometry>
         </visual>
@@ -153,5 +153,5 @@
             <origin xyz="${-brake_thickness/2} -0.014951 ${-third_bar_length-0.0028}" rpy="0 0 0"/>
             <geometry>
-                <mesh filename="package://senseglove_description/urdf/STL/MK29_DK1_Thimble_v2.STL" scale="0.001 0.001 0.001"/>
+                <mesh filename="package://senseglove_description/urdf/dk1/MK29_DK1_Thimble_v2.STL" scale="0.001 0.001 0.001"/>
             </geometry>
         </visual>
@@ -162,5 +162,5 @@
             <origin xyz="${-brake_thickness/2} ${-brake_height/2 - 0.0025} ${-first_bar_length-second_bar_length}" rpy="0 0 0"/>
             <geometry>
-                <mesh filename="package://senseglove_description/urdf/STL/MK29_DK1_Brake_assembly_v2.STL" scale="0.001 0.001 0.001"/>
+                <mesh filename="package://senseglove_description/urdf/dk1/MK29_DK1_Brake_assembly_v2.STL" scale="0.001 0.001 0.001"/>
             </geometry>
         </visual>
@@ -171,5 +171,5 @@
             <origin xyz="${-brake_thickness/2} ${-brake_height+0.006} ${-second_bar_length-first_bar_length-0.003}" rpy="0 0 0"/>
             <geometry>
-                <mesh filename="package://senseglove_description/urdf/STL/MK29_DK1_Abduction_joint_v2.STL" scale="0.001 0.001 0.001"/>
+                <mesh filename="package://senseglove_description/urdf/dk1/MK29_DK1_Abduction_joint_v2.STL" scale="0.001 0.001 0.001"/>
             </geometry>
         </visual>
@@ -180,5 +180,5 @@
             <origin xyz="${-brake_thickness/2} ${-brake_height+0.005} ${-second_bar_length-0.0055}" rpy="0 0 0"/>
             <geometry>
-                <mesh filename="package://senseglove_description/urdf/STL/MK29_DK1_Flexion_joint_1_v2.STL" scale="0.001 0.001 0.001"/>
+                <mesh filename="package://senseglove_description/urdf/dk1/MK29_DK1_Flexion_joint_1_v2.STL" scale="0.001 0.001 0.001"/>
             </geometry>
         </visual>
@@ -189,5 +189,5 @@
             <origin xyz="${-brake_thickness/2} ${-brake_height+0.005} ${-second_bar_length-0.005355}" rpy="0 0 0"/>
             <geometry>
-                <mesh filename="package://senseglove_description/urdf/STL/MK29_DK1_Flexion_joint_2_v2.STL" scale="0.001 0.001 0.001"/>
+                <mesh filename="package://senseglove_description/urdf/dk1/MK29_DK1_Flexion_joint_2_v2.STL" scale="0.001 0.001 0.001"/>
             </geometry>
         </visual>
@@ -198,5 +198,5 @@
             <origin xyz="${-brake_thickness/2} ${-brake_height+0.00533} -0.00533" rpy="0 0 0"/>
             <geometry>
-                <mesh filename="package://senseglove_description/urdf/STL/MK29_DK1_Flexion_joint_3_v2.STL" scale="0.001 0.001 0.001"/>
+                <mesh filename="package://senseglove_description/urdf/dk1/MK29_DK1_Flexion_joint_3_v2.STL" scale="0.001 0.001 0.001"/>
             </geometry>
         </visual>
@@ -207,5 +207,5 @@
             <origin xyz="${-brake_thickness/2} -0.014951 ${-third_bar_length-0.0028}" rpy="0 0 0"/>
             <geometry>
-                <mesh filename="package://senseglove_description/urdf/STL/MK29_DK1_Thimble_v2.STL" scale="0.001 0.001 0.001"/>
+                <mesh filename="package://senseglove_description/urdf/dk1/MK29_DK1_Thimble_v2.STL" scale="0.001 0.001 0.001"/>
             </geometry>
         </visual>
@@ -216,5 +216,5 @@
             <origin xyz="${-brake_thickness/2} ${-brake_height/2 - 0.0025} ${-first_bar_length-second_bar_length}" rpy="0 0 0"/>
             <geometry>
-                <mesh filename="package://senseglove_description/urdf/STL/MK29_DK1_Brake_assembly_v2.STL" scale="0.001 0.001 0.001"/>
+                <mesh filename="package://senseglove_description/urdf/dk1/MK29_DK1_Brake_assembly_v2.STL" scale="0.001 0.001 0.001"/>
             </geometry>
         </visual>
@@ -225,5 +225,5 @@
             <origin xyz="${-brake_thickness/2} ${-brake_height+0.006} ${-second_bar_length-first_bar_length-0.003}" rpy="0 0 0"/>
             <geometry>
-                <mesh filename="package://senseglove_description/urdf/STL/MK29_DK1_Abduction_joint_v2.STL" scale="0.001 0.001 0.001"/>
+                <mesh filename="package://senseglove_description/urdf/dk1/MK29_DK1_Abduction_joint_v2.STL" scale="0.001 0.001 0.001"/>
             </geometry>
         </visual>
@@ -234,5 +234,5 @@
             <origin xyz="${-brake_thickness/2} ${-brake_height+0.005} ${-second_bar_length-0.0055}" rpy="0 0 0"/>
             <geometry>
-                <mesh filename="package://senseglove_description/urdf/STL/MK29_DK1_Flexion_joint_1_v2.STL" scale="0.001 0.001 0.001"/>
+                <mesh filename="package://senseglove_description/urdf/dk1/MK29_DK1_Flexion_joint_1_v2.STL" scale="0.001 0.001 0.001"/>
             </geometry>
         </visual>
@@ -243,5 +243,5 @@
             <origin xyz="${-brake_thickness/2} ${-brake_height+0.005} ${-second_bar_length-0.005355}" rpy="0 0 0"/>
             <geometry>
-                <mesh filename="package://senseglove_description/urdf/STL/MK29_DK1_Flexion_joint_2_v2.STL" scale="0.001 0.001 0.001"/>
+                <mesh filename="package://senseglove_description/urdf/dk1/MK29_DK1_Flexion_joint_2_v2.STL" scale="0.001 0.001 0.001"/>
             </geometry>
         </visual>
@@ -252,5 +252,5 @@
             <origin xyz="${-brake_thickness/2} ${-brake_height+0.00533} -0.00533" rpy="0 0 0"/>
             <geometry>
-                <mesh filename="package://senseglove_description/urdf/STL/MK29_DK1_Flexion_joint_3_v2.STL" scale="0.001 0.001 0.001"/>
+                <mesh filename="package://senseglove_description/urdf/dk1/MK29_DK1_Flexion_joint_3_v2.STL" scale="0.001 0.001 0.001"/>
             </geometry>
         </visual>
@@ -261,5 +261,5 @@
             <origin xyz="${-brake_thickness/2} -0.014951 ${-third_bar_length-0.0028}" rpy="0 0 0"/>
             <geometry>
-                <mesh filename="package://senseglove_description/urdf/STL/MK29_DK1_Thimble_v2.STL" scale="0.001 0.001 0.001"/>
+                <mesh filename="package://senseglove_description/urdf/dk1/MK29_DK1_Thimble_v2.STL" scale="0.001 0.001 0.001"/>
             </geometry>
         </visual>
@@ -270,5 +270,5 @@
             <origin xyz="${-brake_thickness/2-0.0004} ${-brake_height/2 - 0.0025} ${-first_bar_length-second_bar_length-0.003}" rpy="0 0 0"/>
             <geometry>
-                <mesh filename="package://senseglove_description/urdf/STL/MK29_DK1_Brake_assembly_v2.STL" scale="0.001 0.001 0.001"/>
+                <mesh filename="package://senseglove_description/urdf/dk1/MK29_DK1_Brake_assembly_v2.STL" scale="0.001 0.001 0.001"/>
             </geometry>
         </visual>
@@ -279,5 +279,5 @@
             <origin xyz="${-brake_thickness/2} ${-brake_height+0.006} ${-second_bar_length-first_bar_length-0.003}" rpy="0 0 0"/>
             <geometry>
-                <mesh filename="package://senseglove_description/urdf/STL/MK29_DK1_Abduction_joint_v2.STL" scale="0.001 0.001 0.001"/>
+                <mesh filename="package://senseglove_description/urdf/dk1/MK29_DK1_Abduction_joint_v2.STL" scale="0.001 0.001 0.001"/>
             </geometry>
         </visual>
@@ -288,5 +288,5 @@
             <origin xyz="${-brake_thickness/2} ${-brake_height+0.005} ${-second_bar_length-0.0055}" rpy="0 0 0"/>
             <geometry>
-                <mesh filename="package://senseglove_description/urdf/STL/MK29_DK1_Flexion_joint_1_v2.STL" scale="0.001 0.001 0.001"/>
+                <mesh filename="package://senseglove_description/urdf/dk1/MK29_DK1_Flexion_joint_1_v2.STL" scale="0.001 0.001 0.001"/>
             </geometry>
         </visual>
@@ -297,5 +297,5 @@
             <origin xyz="${-brake_thickness/2} ${-brake_height+0.005} ${-second_bar_length-0.005355}" rpy="0 0 0"/>
             <geometry>
-                <mesh filename="package://senseglove_description/urdf/STL/MK29_DK1_Flexion_joint_2_v2.STL" scale="0.001 0.001 0.001"/>
+                <mesh filename="package://senseglove_description/urdf/dk1/MK29_DK1_Flexion_joint_2_v2.STL" scale="0.001 0.001 0.001"/>
             </geometry>
         </visual>
@@ -306,5 +306,5 @@
             <origin xyz="${-brake_thickness/2} ${-brake_height+0.00533} -0.00533" rpy="0 0 0"/>
             <geometry>
-                <mesh filename="package://senseglove_description/urdf/STL/MK29_DK1_Flexion_joint_3_v2.STL" scale="0.001 0.001 0.001"/>
+                <mesh filename="package://senseglove_description/urdf/dk1/MK29_DK1_Flexion_joint_3_v2.STL" scale="0.001 0.001 0.001"/>
             </geometry>
         </visual>
@@ -315,5 +315,5 @@
             <origin xyz="${-brake_thickness/2} -0.014951 ${-third_bar_length-0.0028}" rpy="0 0 0"/>
             <geometry>
-                <mesh filename="package://senseglove_description/urdf/STL/MK29_DK1_Thimble_v2.STL" scale="0.001 0.001 0.001"/>
+                <mesh filename="package://senseglove_description/urdf/dk1/MK29_DK1_Thimble_v2.STL" scale="0.001 0.001 0.001"/>
             </geometry>
         </visual>
