Commit message: tested description package in rviz with a launch file

File: senseglove/senseglove_description/urdf/dk1/dk1_right.description.xacro (robot description, xacro)
@@ -43,5 +43,5 @@
                 <origin xyz="-0.056692 -0.01955 -0.06803" rpy="0 0 0"/>
                 <geometry>
-                    <mesh filename="package://senseglove_description/urdf/dk1/MK29_DK1_HUB.STL" scale="0.001 0.001 0.001"/>
+                    <mesh filename="package://senseglove_description/meshes/dk1/MK29_DK1_HUB.STL" scale="0.001 0.001 0.001"/>
                 </geometry>
             </visual>
@@ -52,5 +52,5 @@
                 <origin xyz="${-brake_thickness/2} ${-brake_height/2 - 0.0025} ${-first_bar_length-second_bar_length}" rpy="0 0 0"/>
                 <geometry>
-                    <mesh filename="package://senseglove_description/urdf/dk1/MK29_DK1_Brake_assembly_v2.STL" scale="0.001 0.001 0.001"/>
+                    <mesh filename="package://senseglove_description/meshes/dk1/MK29_DK1_Brake_assembly_v2.STL" scale="0.001 0.001 0.001"/>
                 </geometry>
             </visual>
@@ -61,5 +61,5 @@
                 <origin xyz="${-brake_thickness/2} ${-brake_height+0.006} ${-second_bar_length-first_bar_length-0.003}" rpy="0 0 0"/>
                 <geometry>
-                    <mesh filename="package://senseglove_description/urdf/dk1/MK29_DK1_Abduction_joint_v2.STL" scale="0.001 0.001 0.001"/>
+                    <mesh filename="package://senseglove_description/meshes/dk1/MK29_DK1_Abduction_joint_v2.STL" scale="0.001 0.001 0.001"/>
                 </geometry>
             </visual>
@@ -70,5 +70,5 @@
                 <origin xyz="${-brake_thickness/2} ${-brake_height+0.005} ${-second_bar_length-0.0055}" rpy="0 0 0"/>
                 <geometry>
-                    <mesh filename="package://senseglove_description/urdf/dk1/MK29_DK1_Flexion_joint_1_v2.STL" scale="0.001 0.001 0.001"/>
+                    <mesh filename="package://senseglove_description/meshes/dk1/MK29_DK1_Flexion_joint_1_v2.STL" scale="0.001 0.001 0.001"/>
                 </geometry>
             </visual>
@@ -79,5 +79,5 @@
                 <origin xyz="${-brake_thickness/2} ${-brake_height+0.005} ${-second_bar_length-0.005355}" rpy="0 0 0"/>
                 <geometry>
-                    <mesh filename="package://senseglove_description/urdf/dk1/MK29_DK1_Flexion_joint_2_v2.STL" scale="0.001 0.001 0.001"/>
+                    <mesh filename="package://senseglove_description/meshes/dk1/MK29_DK1_Flexion_joint_2_v2.STL" scale="0.001 0.001 0.001"/>
                 </geometry>
             </visual>
@@ -88,5 +88,5 @@
                 <origin xyz="${-brake_thickness/2} ${-brake_height+0.00533} -0.00533" rpy="0 0 0"/>
                 <geometry>
-                    <mesh filename="package://senseglove_description/urdf/dk1/MK29_DK1_Flexion_joint_3_v2.STL" scale="0.001 0.001 0.001"/>
+                    <mesh filename="package://senseglove_description/meshes/dk1/MK29_DK1_Flexion_joint_3_v2.STL" scale="0.001 0.001 0.001"/>
                 </geometry>
             </visual>
@@ -97,5 +97,5 @@
                 <origin xyz="${-brake_thickness/2} -0.014951 ${-third_bar_length-0.0028}" rpy="0 0 0"/>
                 <geometry>
-                    <mesh filename="package://senseglove_description/urdf/dk1/MK29_DK1_Thimble_v2.STL" scale="0.001 0.001 0.001"/>
+                    <mesh filename="package://senseglove_description/meshes/dk1/MK29_DK1_Thimble_v2.STL" scale="0.001 0.001 0.001"/>
                 </geometry>
             </visual>
@@ -106,5 +106,5 @@
                 <origin xyz="${-brake_thickness/2} ${-brake_height/2 - 0.0025} ${-first_bar_length-second_bar_length}" rpy="0 0 0"/>
                 <geometry>
-                    <mesh filename="package://senseglove_description/urdf/dk1/MK29_DK1_Brake_assembly_v2.STL" scale="0.001 0.001 0.001"/>
+                    <mesh filename="package://senseglove_description/meshes/dk1/MK29_DK1_Brake_assembly_v2.STL" scale="0.001 0.001 0.001"/>
                 </geometry>
             </visual>
@@ -115,5 +115,5 @@
                 <origin xyz="${-brake_thickness/2} ${-brake_height+0.006} ${-second_bar_length-first_bar_length-0.003}" rpy="0 0 0"/>
                 <geometry>
-                    <mesh filename="package://senseglove_description/urdf/dk1/MK29_DK1_Abduction_joint_v2.STL" scale="0.001 0.001 0.001"/>
+                    <mesh filename="package://senseglove_description/meshes/dk1/MK29_DK1_Abduction_joint_v2.STL" scale="0.001 0.001 0.001"/>
                 </geometry>
             </visual>
@@ -124,5 +124,5 @@
                 <origin xyz="${-brake_thickness/2} ${-brake_height+0.005} ${-second_bar_length-0.0055}" rpy="0 0 0"/>
                 <geometry>
-                    <mesh filename="package://senseglove_description/urdf/dk1/MK29_DK1_Flexion_joint_1_v2.STL" scale="0.001 0.001 0.001"/>
+                    <mesh filename="package://senseglove_description/meshes/dk1/MK29_DK1_Flexion_joint_1_v2.STL" scale="0.001 0.001 0.001"/>
                 </geometry>
             </visual>
@@ -133,5 +133,5 @@
                 <origin xyz="${-brake_thickness/2} ${-brake_height+0.005} ${-second_bar_length-0.005355}" rpy="0 0 0"/>
                 <geometry>
-                    <mesh filename="package://senseglove_description/urdf/dk1/MK29_DK1_Flexion_joint_2_v2.STL" scale="0.001 0.001 0.001"/>
+                    <mesh filename="package://senseglove_description/meshes/dk1/MK29_DK1_Flexion_joint_2_v2.STL" scale="0.001 0.001 0.001"/>
                 </geometry>
             </visual>
@@ -142,5 +142,5 @@
                 <origin xyz="${-brake_thickness/2} ${-brake_height+0.00533} -0.00533" rpy="0 0 0"/>
                 <geometry>
-                    <mesh filename="package://senseglove_description/urdf/dk1/MK29_DK1_Flexion_joint_3_v2.STL" scale="0.001 0.001 0.001"/>
+                    <mesh filename="package://senseglove_description/meshes/dk1/MK29_DK1_Flexion_joint_3_v2.STL" scale="0.001 0.001 0.001"/>
                 </geometry>
             </visual>
@@ -151,5 +151,5 @@
                 <origin xyz="${-brake_thickness/2} -0.014951 ${-third_bar_length-0.0028}" rpy="0 0 0"/>
                 <geometry>
-                    <mesh filename="package://senseglove_description/urdf/dk1/MK29_DK1_Thimble_v2.STL" scale="0.001 0.001 0.001"/>
+                    <mesh filename="package://senseglove_description/meshes/dk1/MK29_DK1_Thimble_v2.STL" scale="0.001 0.001 0.001"/>
                 </geometry>
             </visual>
@@ -160,5 +160,5 @@
                 <origin xyz="${-brake_thickness/2} ${-brake_height/2 - 0.0025} ${-first_bar_length-second_bar_length}" rpy="0 0 0"/>
                 <geometry>
-                    <mesh filename="package://senseglove_description/urdf/dk1/MK29_DK1_Brake_assembly_v2.STL" scale="0.001 0.001 0.001"/>
+                    <mesh filename="package://senseglove_description/meshes/dk1/MK29_DK1_Brake_assembly_v2.STL" scale="0.001 0.001 0.001"/>
                 </geometry>
             </visual>
@@ -169,5 +169,5 @@
                 <origin xyz="${-brake_thickness/2} ${-brake_height+0.006} ${-second_bar_length-first_bar_length-0.003}" rpy="0 0 0"/>
                 <geometry>
-                    <mesh filename="package://senseglove_description/urdf/dk1/MK29_DK1_Abduction_joint_v2.STL" scale="0.001 0.001 0.001"/>
+                    <mesh filename="package://senseglove_description/meshes/dk1/MK29_DK1_Abduction_joint_v2.STL" scale="0.001 0.001 0.001"/>
                 </geometry>
             </visual>
@@ -178,5 +178,5 @@
                 <origin xyz="${-brake_thickness/2} ${-brake_height+0.005} ${-second_bar_length-0.0055}" rpy="0 0 0"/>
                 <geometry>
-                    <mesh filename="package://senseglove_description/urdf/dk1/MK29_DK1_Flexion_joint_1_v2.STL" scale="0.001 0.001 0.001"/>
+                    <mesh filename="package://senseglove_description/meshes/dk1/MK29_DK1_Flexion_joint_1_v2.STL" scale="0.001 0.001 0.001"/>
                 </geometry>
             </visual>
@@ -187,5 +187,5 @@
                 <origin xyz="${-brake_thickness/2} ${-brake_height+0.005} ${-second_bar_length-0.005355}" rpy="0 0 0"/>
                 <geometry>
-                    <mesh filename="package://senseglove_description/urdf/dk1/MK29_DK1_Flexion_joint_2_v2.STL" scale="0.001 0.001 0.001"/>
+                    <mesh filename="package://senseglove_description/meshes/dk1/MK29_DK1_Flexion_joint_2_v2.STL" scale="0.001 0.001 0.001"/>
                 </geometry>
             </visual>
@@ -196,5 +196,5 @@
                 <origin xyz="${-brake_thickness/2} ${-brake_height+0.00533} -0.00533" rpy="0 0 0"/>
                 <geometry>
-                    <mesh filename="package://senseglove_description/urdf/dk1/MK29_DK1_Flexion_joint_3_v2.STL" scale="0.001 0.001 0.001"/>
+                    <mesh filename="package://senseglove_description/meshes/dk1/MK29_DK1_Flexion_joint_3_v2.STL" scale="0.001 0.001 0.001"/>
                 </geometry>
             </visual>
@@ -205,5 +205,5 @@
                 <origin xyz="${-brake_thickness/2} -0.014951 ${-third_bar_length-0.0028}" rpy="0 0 0"/>
                 <geometry>
-                    <mesh filename="package://senseglove_description/urdf/dk1/MK29_DK1_Thimble_v2.STL" scale="0.001 0.001 0.001"/>
+                    <mesh filename="package://senseglove_description/meshes/dk1/MK29_DK1_Thimble_v2.STL" scale="0.001 0.001 0.001"/>
                 </geometry>
             </visual>
@@ -214,5 +214,5 @@
                 <origin xyz="${-brake_thickness/2} ${-brake_height/2 - 0.0025} ${-first_bar_length-second_bar_length}" rpy="0 0 0"/>
                 <geometry>
-                    <mesh filename="package://senseglove_description/urdf/dk1/MK29_DK1_Brake_assembly_v2.STL" scale="0.001 0.001 0.001"/>
+                    <mesh filename="package://senseglove_description/meshes/dk1/MK29_DK1_Brake_assembly_v2.STL" scale="0.001 0.001 0.001"/>
                 </geometry>
             </visual>
@@ -223,5 +223,5 @@
                 <origin xyz="${-brake_thickness/2} ${-brake_height+0.006} ${-second_bar_length-first_bar_length-0.003}" rpy="0 0 0"/>
                 <geometry>
-                    <mesh filename="package://senseglove_description/urdf/dk1/MK29_DK1_Abduction_joint_v2.STL" scale="0.001 0.001 0.001"/>
+                    <mesh filename="package://senseglove_description/meshes/dk1/MK29_DK1_Abduction_joint_v2.STL" scale="0.001 0.001 0.001"/>
                 </geometry>
             </visual>
@@ -232,5 +232,5 @@
                 <origin xyz="${-brake_thickness/2} ${-brake_height+0.005} ${-second_bar_length-0.0055}" rpy="0 0 0"/>
                 <geometry>
-                    <mesh filename="package://senseglove_description/urdf/dk1/MK29_DK1_Flexion_joint_1_v2.STL" scale="0.001 0.001 0.001"/>
+                    <mesh filename="package://senseglove_description/meshes/dk1/MK29_DK1_Flexion_joint_1_v2.STL" scale="0.001 0.001 0.001"/>
                 </geometry>
             </visual>
@@ -241,5 +241,5 @@
                 <origin xyz="${-brake_thickness/2} ${-brake_height+0.005} ${-second_bar_length-0.005355}" rpy="0 0 0"/>
                 <geometry>
-                    <mesh filename="package://senseglove_description/urdf/dk1/MK29_DK1_Flexion_joint_2_v2.STL" scale="0.001 0.001 0.001"/>
+                    <mesh filename="package://senseglove_description/meshes/dk1/MK29_DK1_Flexion_joint_2_v2.STL" scale="0.001 0.001 0.001"/>
                 </geometry>
             </visual>
@@ -250,5 +250,5 @@
                 <origin xyz="${-brake_thickness/2} ${-brake_height+0.00533} -0.00533" rpy="0 0 0"/>
                 <geometry>
-                    <mesh filename="package://senseglove_description/urdf/dk1/MK29_DK1_Flexion_joint_3_v2.STL" scale="0.001 0.001 0.001"/>
+                    <mesh filename="package://senseglove_description/meshes/dk1/MK29_DK1_Flexion_joint_3_v2.STL" scale="0.001 0.001 0.001"/>
                 </geometry>
             </visual>
@@ -259,5 +259,5 @@
                 <origin xyz="${-brake_thickness/2} -0.014951 ${-third_bar_length-0.0028}" rpy="0 0 0"/>
                 <geometry>
-                    <mesh filename="package://senseglove_description/urdf/dk1/MK29_DK1_Thimble_v2.STL" scale="0.001 0.001 0.001"/>
+                    <mesh filename="package://senseglove_description/meshes/dk1/MK29_DK1_Thimble_v2.STL" scale="0.001 0.001 0.001"/>
                 </geometry>
             </visual>
@@ -268,5 +268,5 @@
                 <origin xyz="${-brake_thickness/2-0.0004} ${-brake_height/2 - 0.0025} ${-first_bar_length-second_bar_length-0.003}" rpy="0 0 0"/>
                 <geometry>
-                    <mesh filename="package://senseglove_description/urdf/dk1/MK29_DK1_Brake_assembly_v2.STL" scale="0.001 0.001 0.001"/>
+                    <mesh filename="package://senseglove_description/meshes/dk1/MK29_DK1_Brake_assembly_v2.STL" scale="0.001 0.001 0.001"/>
                 </geometry>
             </visual>
@@ -277,5 +277,5 @@
                 <origin xyz="${-brake_thickness/2} ${-brake_height+0.006} ${-second_bar_length-first_bar_length-0.003}" rpy="0 0 0"/>
                 <geometry>
-                    <mesh filename="package://senseglove_description/urdf/dk1/MK29_DK1_Abduction_joint_v2.STL" scale="0.001 0.001 0.001"/>
+                    <mesh filename="package://senseglove_description/meshes/dk1/MK29_DK1_Abduction_joint_v2.STL" scale="0.001 0.001 0.001"/>
                 </geometry>
             </visual>
@@ -286,5 +286,5 @@
                 <origin xyz="${-brake_thickness/2} ${-brake_height+0.005} ${-second_bar_length-0.0055}" rpy="0 0 0"/>
                 <geometry>
-                    <mesh filename="package://senseglove_description/urdf/dk1/MK29_DK1_Flexion_joint_1_v2.STL" scale="0.001 0.001 0.001"/>
+                    <mesh filename="package://senseglove_description/meshes/dk1/MK29_DK1_Flexion_joint_1_v2.STL" scale="0.001 0.001 0.001"/>
                 </geometry>
             </visual>
@@ -295,5 +295,5 @@
                 <origin xyz="${-brake_thickness/2} ${-brake_height+0.005} ${-second_bar_length-0.005355}" rpy="0 0 0"/>
                 <geometry>
-                    <mesh filename="package://senseglove_description/urdf/dk1/MK29_DK1_Flexion_joint_2_v2.STL" scale="0.001 0.001 0.001"/>
+                    <mesh filename="package://senseglove_description/meshes/dk1/MK29_DK1_Flexion_joint_2_v2.STL" scale="0.001 0.001 0.001"/>
                 </geometry>
             </visual>
@@ -304,5 +304,5 @@
                 <origin xyz="${-brake_thickness/2} ${-brake_height+0.00533} -0.00533" rpy="0 0 0"/>
                 <geometry>
-                    <mesh filename="package://senseglove_description/urdf/dk1/MK29_DK1_Flexion_joint_3_v2.STL" scale="0.001 0.001 0.001"/>
+                    <mesh filename="package://senseglove_description/meshes/dk1/MK29_DK1_Flexion_joint_3_v2.STL" scale="0.001 0.001 0.001"/>
                 </geometry>
             </visual>
@@ -313,5 +313,5 @@
                 <origin xyz="${-brake_thickness/2} -0.014951 ${-third_bar_length-0.0028}" rpy="0 0 0"/>
                 <geometry>
-                    <mesh filename="package://senseglove_description/urdf/dk1/MK29_DK1_Thimble_v2.STL" scale="0.001 0.001 0.001"/>
+                    <mesh filename="package://senseglove_description/meshes/dk1/MK29_DK1_Thimble_v2.STL" scale="0.001 0.001 0.001"/>
                 </geometry>
             </visual>
