Commit message: updated ros2_control xacros for all gloves

File: senseglove/senseglove_description/ros2_control/dk1/dk1_right.ros2_control.xacro (robot description, xacro)
@@ -1,5 +1,5 @@
 <?xml version='1.0'?>
 <robot xmlns:xacro="http://www.ros.org/wiki/xacro">
-    <xacro:macro name="nova2_right_ros2_control" params="name prefix">
+    <xacro:macro name="dk1_right_ros2_control" params="name prefix">
         <!-- Include joint interfaces macro -->
         <xacro:include filename="$(find senseglove_description)/urdf/urdf_helper_macros/joint_interfaces_macro.xacro"/>
@@ -8,5 +8,5 @@
             <hardware>
                 <plugin>senseglove_hardware_interface/SGHardwareInterface</plugin>
-                <param name="glove_name">nova2_right</param>
+                <param name="glove_name">dk1_right</param>
             </hardware>
             <!-- State Interfaces -->
@@ -17,19 +17,8 @@
             <xacro:add_state_interfaces joint_name="r_middle_mcp"/>
             <xacro:add_state_interfaces joint_name="r_middle_pip"/>
-            <xacro:add_state_interfaces joint_name="r_middle_dip"/>
             <xacro:add_state_interfaces joint_name="r_ring_mcp"/>
             <xacro:add_state_interfaces joint_name="r_ring_pip"/>
-            <xacro:add_state_interfaces joint_name="r_ring_dip"/>
-            <xacro:add_state_interfaces joint_name="r_pinky_brake"/>
             <xacro:add_state_interfaces joint_name="r_pinky_mcp"/>
             <xacro:add_state_interfaces joint_name="r_pinky_pip"/>
-            <xacro:add_state_interfaces joint_name="r_pinky_dip"/>
-            <xacro:add_state_interfaces joint_name="r_palm_index"/>
-            <xacro:add_state_interfaces joint_name="r_palm_pinky"/>
-            <xacro:add_state_interfaces joint_name="r_palm_strap"/>
-            <!-- Command Interfaces -->
-            <xacro:add_command_interfaces joint_name="r_palm_index"/>
-            <xacro:add_command_interfaces joint_name="r_palm_pinky"/>
-            <xacro:add_command_interfaces joint_name="r_palm_strap"/>
             <!-- State and Command Interfaces -->
             <xacro:add_state_and_command_interfaces joint_name="r_thumb_brake"/>
@@ -37,6 +26,10 @@
             <xacro:add_state_and_command_interfaces joint_name="r_middle_brake"/>
             <xacro:add_state_and_command_interfaces joint_name="r_ring_brake"/>
+            <xacro:add_state_and_command_interfaces joint_name="r_pinky_brake"/>
             <xacro:add_state_and_command_interfaces joint_name="r_thumb_dip"/>
             <xacro:add_state_and_command_interfaces joint_name="r_index_dip"/>
+            <xacro:add_state_and_command_interfaces joint_name="r_middle_dip"/>
+            <xacro:add_state_and_command_interfaces joint_name="r_ring_dip"/>
+            <xacro:add_state_and_command_interfaces joint_name="r_pinky_dip"/>
         </ros2_control>
     </xacro:macro>

File: senseglove/senseglove_description/ros2_control/nova1/nova_right.ros2_control.xacro (robot description, xacro)
@@ -1,5 +1,5 @@
 <?xml version='1.0'?>
 <robot xmlns:xacro="http://www.ros.org/wiki/xacro">
-    <xacro:macro name="nova2_right_ros2_control" params="name prefix">
+    <xacro:macro name="nova_right_ros2_control" params="name prefix">
         <!-- Include joint interfaces macro -->
         <xacro:include filename="$(find senseglove_description)/urdf/urdf_helper_macros/joint_interfaces_macro.xacro"/>
@@ -8,5 +8,5 @@
             <hardware>
                 <plugin>senseglove_hardware_interface/SGHardwareInterface</plugin>
-                <param name="glove_name">nova2_right</param>
+                <param name="glove_name">nova_right</param>
             </hardware>
             <!-- State Interfaces -->
@@ -25,11 +25,6 @@
             <xacro:add_state_interfaces joint_name="r_pinky_pip"/>
             <xacro:add_state_interfaces joint_name="r_pinky_dip"/>
-            <xacro:add_state_interfaces joint_name="r_palm_index"/>
-            <xacro:add_state_interfaces joint_name="r_palm_pinky"/>
-            <xacro:add_state_interfaces joint_name="r_palm_strap"/>
             <!-- Command Interfaces -->
-            <xacro:add_command_interfaces joint_name="r_palm_index"/>
-            <xacro:add_command_interfaces joint_name="r_palm_pinky"/>
-            <xacro:add_command_interfaces joint_name="r_palm_strap"/>
+            <xacro:add_command_interfaces joint_name="r_thumper"/>
             <!-- State and Command Interfaces -->
             <xacro:add_state_and_command_interfaces joint_name="r_thumb_brake"/>
