Commit message: default xacro args into ros2_control params for SenseGlove HW init

File: senseglove/senseglove_description/ros2_control/dk1/dk1_left.ros2_control.xacro (robot description, xacro)
@@ -1,5 +1,5 @@
 <?xml version='1.0'?>
 <robot xmlns:xacro="http://www.ros.org/wiki/xacro">
-    <xacro:macro name="dk1_left_ros2_control" params="name prefix">
+    <xacro:macro name="dk1_left_ros2_control" params="name prefix selected_robot glove_index is_right publish_rate">
         <!-- Include joint interfaces macro -->
         <xacro:include filename="$(find senseglove_description)/urdf/urdf_helper_macros/joint_interfaces_macro.xacro"/>
@@ -8,5 +8,8 @@
             <hardware>
                 <plugin>senseglove_hardware_interface/SenseGloveHardwareInterface</plugin>
-                <param name="glove_name">dk1_left</param>
+                <param name="selected_robot">${selected_robot}</param>
+                <param name="glove_index">${glove_index}</param>
+                <param name="is_right">${is_right}</param>
+                <param name="publish_rate">${publish_rate}</param>
             </hardware>
             <!-- State Interfaces -->

File: senseglove/senseglove_description/ros2_control/dk1/dk1_right.ros2_control.xacro (robot description, xacro)
@@ -1,5 +1,5 @@
 <?xml version='1.0'?>
 <robot xmlns:xacro="http://www.ros.org/wiki/xacro">
-    <xacro:macro name="dk1_right_ros2_control" params="name prefix">
+    <xacro:macro name="dk1_right_ros2_control" params="name prefix selected_robot glove_index is_right publish_rate">
         <!-- Include joint interfaces macro -->
         <xacro:include filename="$(find senseglove_description)/urdf/urdf_helper_macros/joint_interfaces_macro.xacro"/>
@@ -8,5 +8,8 @@
             <hardware>
                 <plugin>senseglove_hardware_interface/SenseGloveHardwareInterface</plugin>
-                <param name="glove_name">dk1_right</param>
+                <param name="selected_robot">${selected_robot}</param>
+                <param name="glove_index">${glove_index}</param>
+                <param name="is_right">${is_right}</param>
+                <param name="publish_rate">${publish_rate}</param>
             </hardware>
             <!-- State Interfaces -->

File: senseglove/senseglove_description/ros2_control/nova/nova_left.ros2_control.xacro (robot description, xacro)
@@ -1,5 +1,5 @@
 <?xml version='1.0'?>
 <robot xmlns:xacro="http://www.ros.org/wiki/xacro">
-    <xacro:macro name="nova_left_ros2_control" params="name prefix">
+    <xacro:macro name="nova_left_ros2_control" params="name prefix selected_robot glove_index is_right publish_rate">
         <!-- Include joint interfaces macro -->
         <xacro:include filename="$(find senseglove_description)/urdf/urdf_helper_macros/joint_interfaces_macro.xacro"/>
@@ -8,5 +8,8 @@
             <hardware>
                 <plugin>senseglove_hardware_interface/SenseGloveHardwareInterface</plugin>
-                <param name="glove_name">nova_left</param>
+                <param name="selected_robot">${selected_robot}</param>
+                <param name="glove_index">${glove_index}</param>
+                <param name="is_right">${is_right}</param>
+                <param name="publish_rate">${publish_rate}</param>
             </hardware>
             <!-- State Interfaces -->

File: senseglove/senseglove_description/ros2_control/nova/nova_right.ros2_control.xacro (robot description, xacro)
@@ -1,5 +1,5 @@
 <?xml version='1.0'?>
 <robot xmlns:xacro="http://www.ros.org/wiki/xacro">
-    <xacro:macro name="nova_right_ros2_control" params="name prefix">
+    <xacro:macro name="nova_right_ros2_control" params="name prefix selected_robot glove_index is_right publish_rate">
         <!-- Include joint interfaces macro -->
         <xacro:include filename="$(find senseglove_description)/urdf/urdf_helper_macros/joint_interfaces_macro.xacro"/>
@@ -8,5 +8,8 @@
             <hardware>
                 <plugin>senseglove_hardware_interface/SenseGloveHardwareInterface</plugin>
-                <param name="glove_name">nova_right</param>
+                <param name="selected_robot">${selected_robot}</param>
+                <param name="glove_index">${glove_index}</param>
+                <param name="is_right">${is_right}</param>
+                <param name="publish_rate">${publish_rate}</param>
             </hardware>
             <!-- State Interfaces -->

File: senseglove/senseglove_description/ros2_control/nova2/nova2_left.ros2_control.xacro (robot description, xacro)
@@ -1,5 +1,5 @@
 <?xml version='1.0'?>
 <robot xmlns:xacro="http://www.ros.org/wiki/xacro">
-    <xacro:macro name="nova2_left_ros2_control" params="name prefix">
+    <xacro:macro name="nova2_left_ros2_control" params="name prefix selected_robot glove_index is_right publish_rate">
         <!-- Include joint interfaces macro -->
         <xacro:include filename="$(find senseglove_description)/urdf/urdf_helper_macros/joint_interfaces_macro.xacro"/>
@@ -8,5 +8,8 @@
             <hardware>
                 <plugin>senseglove_hardware_interface/SenseGloveHardwareInterface</plugin>
-                <param name="glove_name">nova2_left</param>
+                <param name="selected_robot">${selected_robot}</param>
+                <param name="glove_index">${glove_index}</param>
+                <param name="is_right">${is_right}</param>
+                <param name="publish_rate">${publish_rate}</param>
             </hardware>
             <!-- State Interfaces -->

File: senseglove/senseglove_description/ros2_control/nova2/nova2_right.ros2_control.xacro (robot description, xacro)
@@ -1,5 +1,5 @@
 <?xml version='1.0'?>
 <robot xmlns:xacro="http://www.ros.org/wiki/xacro">
-    <xacro:macro name="nova2_right_ros2_control" params="name prefix">
+    <xacro:macro name="nova2_right_ros2_control" params="name prefix selected_robot glove_index is_right publish_rate">
         <!-- Include joint interfaces macro -->
         <xacro:include filename="$(find senseglove_description)/urdf/urdf_helper_macros/joint_interfaces_macro.xacro"/>
@@ -8,5 +8,8 @@
             <hardware>
                 <plugin>senseglove_hardware_interface/SenseGloveHardwareInterface</plugin>
-                <param name="glove_name">nova2_right</param>
+                <param name="selected_robot">${selected_robot}</param>
+                <param name="glove_index">${glove_index}</param>
+                <param name="is_right">${is_right}</param>
+                <param name="publish_rate">${publish_rate}</param>
             </hardware>
             <!-- State Interfaces -->

File: senseglove/senseglove_description/urdf/dk1/dk1_left.urdf.xacro (robot description, xacro)
@@ -1,4 +1,8 @@
 <?xml version="1.0"?>
 <robot xmlns:xacro="http://www.ros.org/wiki/xacro" name="dk1">
+  <xacro:arg name="selected_robot"  default="dk1_left" />
+  <xacro:arg name="glove_index"     default="0" />
+  <xacro:arg name="is_right"        default="false" />
+  <xacro:arg name="publish_rate"    default="120" />
   <xacro:arg name="prefix" default="" />
   <!-- Import Dk1 Description Macro -->
@@ -9,4 +13,10 @@
   <link name="world"/>
   <xacro:dk1_left parent="world" prefix="$(arg prefix)" />
-  <xacro:dk1_left_ros2_control name="Dk1LeftControl" prefix="$(arg prefix)" />
+  <xacro:dk1_left_ros2_control
+    name="Dk1LeftControl"
+    prefix="$(arg prefix)"
+    selected_robot="$(arg selected_robot)"
+    glove_index="$(arg glove_index)"
+    is_right="$(arg is_right)"
+    publish_rate="$(arg publish_rate)" />
 </robot>

File: senseglove/senseglove_description/urdf/dk1/dk1_right.urdf.xacro (robot description, xacro)
@@ -1,4 +1,8 @@
 <?xml version="1.0"?>
 <robot xmlns:xacro="http://www.ros.org/wiki/xacro" name="dk1">
+  <xacro:arg name="selected_robot"  default="dk1_right" />
+  <xacro:arg name="glove_index"     default="0" />
+  <xacro:arg name="is_right"        default="true" />
+  <xacro:arg name="publish_rate"    default="120" />
   <xacro:arg name="prefix" default="" />
   <!-- Import Dk1 Description Macro -->
@@ -9,4 +13,10 @@
   <link name="world"/>
   <xacro:dk1_right parent="world" prefix="$(arg prefix)" />
-  <xacro:dk1_right_ros2_control name="Dk1RightControl" prefix="$(arg prefix)" />
+  <xacro:dk1_right_ros2_control
+    name="Dk1RightControl"
+    prefix="$(arg prefix)"
+    selected_robot="$(arg selected_robot)"
+    glove_index="$(arg glove_index)"
+    is_right="$(arg is_right)"
+    publish_rate="$(arg publish_rate)" />
 </robot>

File: senseglove/senseglove_description/urdf/nova/nova_left.urdf.xacro (robot description, xacro)
@@ -1,5 +1,9 @@
 <?xml version="1.0"?>
 <robot xmlns:xacro="http://www.ros.org/wiki/xacro" name="nova">
-  <xacro:arg name="prefix" default="" />
+  <xacro:arg name="prefix"          default="" />
+  <xacro:arg name="selected_robot"  default="nova_left" />
+  <xacro:arg name="glove_index"     default="0" />
+  <xacro:arg name="is_right"        default="false" />
+  <xacro:arg name="publish_rate"    default="60" />
   <!-- Import Nova Description Macro -->
   <xacro:include filename="$(find senseglove_description)/urdf/nova/nova_left.description.xacro" />
@@ -9,4 +13,10 @@
   <link name="world"/>
   <xacro:nova_left parent="world" prefix="$(arg prefix)" />
-  <xacro:nova_left_ros2_control name="NovaLeftControl" prefix="$(arg prefix)" />
+  <xacro:nova_left_ros2_control
+    name="NovaLeftControl"
+    prefix="$(arg prefix)"
+    selected_robot="$(arg selected_robot)"
+    glove_index="$(arg glove_index)"
+    is_right="$(arg is_right)"
+    publish_rate="$(arg publish_rate)" />
 </robot>

File: senseglove/senseglove_description/urdf/nova/nova_right.urdf.xacro (robot description, xacro)
@@ -1,5 +1,9 @@
 <?xml version="1.0"?>
 <robot xmlns:xacro="http://www.ros.org/wiki/xacro" name="nova">
-  <xacro:arg name="prefix" default="" />
+  <xacro:arg name="prefix"          default="" />
+  <xacro:arg name="selected_robot"  default="nova_right" />
+  <xacro:arg name="glove_index"     default="0" />
+  <xacro:arg name="is_right"        default="true" />
+  <xacro:arg name="publish_rate"    default="60" />
   <!-- Import Nova Description Macro -->
   <xacro:include filename="$(find senseglove_description)/urdf/nova/nova_right.description.xacro" />
@@ -9,4 +13,10 @@
   <link name="world"/>
   <xacro:nova_right parent="world" prefix="$(arg prefix)" />
-  <xacro:nova_right_ros2_control name="NovaRightControl" prefix="$(arg prefix)" />
+  <xacro:nova_right_ros2_control
+    name="NovaRightControl"
+    prefix="$(arg prefix)"
+    selected_robot="$(arg selected_robot)"
+    glove_index="$(arg glove_index)"
+    is_right="$(arg is_right)"
+    publish_rate="$(arg publish_rate)" />
 </robot>

File: senseglove/senseglove_description/urdf/nova2/nova2_left.urdf.xacro (robot description, xacro)
@@ -1,5 +1,9 @@
 <?xml version="1.0"?>
 <robot xmlns:xacro="http://www.ros.org/wiki/xacro" name="nova2">
-  <xacro:arg name="prefix" default="" />
+  <xacro:arg name="prefix"          default="" />
+  <xacro:arg name="selected_robot"  default="nova2_left" />
+  <xacro:arg name="glove_index"     default="0" />
+  <xacro:arg name="is_right"        default="false" />
+  <xacro:arg name="publish_rate"    default="60" />
   <!-- Import Nova2 Description Macro -->
   <xacro:include filename="$(find senseglove_description)/urdf/nova2/nova2_left.description.xacro" />
@@ -9,4 +13,10 @@
   <link name="world"/>
   <xacro:nova2_left parent="world" prefix="$(arg prefix)" />
-  <xacro:nova2_left_ros2_control name="Nova2LeftControl" prefix="$(arg prefix)" />
+  <xacro:nova2_left_ros2_control
+    name="Nova2LeftControl"
+    prefix="$(arg prefix)"
+    selected_robot="$(arg selected_robot)"
+    glove_index="$(arg glove_index)"
+    is_right="$(arg is_right)"
+    publish_rate="$(arg publish_rate)" />
 </robot>

File: senseglove/senseglove_description/urdf/nova2/nova2_right.urdf.xacro (robot description, xacro)
@@ -1,5 +1,9 @@
 <?xml version="1.0"?>
 <robot xmlns:xacro="http://www.ros.org/wiki/xacro" name="nova2">
-  <xacro:arg name="prefix" default="" />
+  <xacro:arg name="prefix"          default="" />
+  <xacro:arg name="selected_robot"  default="nova2_right" />
+  <xacro:arg name="glove_index"     default="0" />
+  <xacro:arg name="is_right"        default="true" />
+  <xacro:arg name="publish_rate"    default="60" />
   <!-- Import Nova2 Description Macro -->
   <xacro:include filename="$(find senseglove_description)/urdf/nova2/nova2_right.description.xacro" />
@@ -9,4 +13,10 @@
   <link name="world"/>
   <xacro:nova2_right parent="world" prefix="$(arg prefix)" />
-  <xacro:nova2_right_ros2_control name="Nova2RightControl" prefix="$(arg prefix)" />
+  <xacro:nova2_right_ros2_control
+    name="Nova2RightControl"
+    prefix="$(arg prefix)"
+    selected_robot="$(arg selected_robot)"
+    glove_index="$(arg glove_index)"
+    is_right="$(arg is_right)"
+    publish_rate="$(arg publish_rate)" />
 </robot>
