Commit message: converted urdf::Model to shared_ptr to resolve memory corruption, serial based glove selection

File: senseglove/senseglove_description/ros2_control/nova2/nova2_left.ros2_control.xacro (robot description, xacro)
@@ -1,5 +1,5 @@
 <?xml version='1.0'?>
 <robot xmlns:xacro="http://www.ros.org/wiki/xacro">
-    <xacro:macro name="nova2_left_ros2_control" params="name prefix selected_robot glove_index is_right publish_rate">
+    <xacro:macro name="nova2_left_ros2_control" params="name prefix selected_robot glove_index is_right glove_serial publish_rate">
         <!-- Include joint interfaces macro -->
         <xacro:include filename="$(find senseglove_description)/urdf/urdf_helper_macros/joint_interfaces_macro.xacro"/>
@@ -11,4 +11,5 @@
                 <param name="glove_index">${glove_index}</param>
                 <param name="is_right">${is_right}</param>
+                <param name="glove_serial">${glove_serial}</param>
                 <param name="publish_rate">${publish_rate}</param>
             </hardware>

File: senseglove/senseglove_description/ros2_control/nova2/nova2_right.ros2_control.xacro (robot description, xacro)
@@ -1,5 +1,5 @@
 <?xml version='1.0'?>
 <robot xmlns:xacro="http://www.ros.org/wiki/xacro">
-    <xacro:macro name="nova2_right_ros2_control" params="name prefix selected_robot glove_index is_right publish_rate">
+    <xacro:macro name="nova2_right_ros2_control" params="name prefix selected_robot glove_index is_right glove_serial publish_rate">
         <!-- Include joint interfaces macro -->
         <xacro:include filename="$(find senseglove_description)/urdf/urdf_helper_macros/joint_interfaces_macro.xacro"/>
@@ -11,4 +11,5 @@
                 <param name="glove_index">${glove_index}</param>
                 <param name="is_right">${is_right}</param>
+                <param name="glove_serial">${glove_serial}</param>
                 <param name="publish_rate">${publish_rate}</param>
             </hardware>

File: senseglove/senseglove_description/urdf/nova2/nova2_left.urdf.xacro (robot description, xacro)
@@ -5,4 +5,5 @@
   <xacro:arg name="glove_index"     default="0" />
   <xacro:arg name="is_right"        default="false" />
+  <xacro:arg name="glove_serial"    default=""/>
   <xacro:arg name="publish_rate"    default="60" />
   <!-- Import Nova2 Description Macro -->
@@ -19,4 +20,5 @@
     glove_index="$(arg glove_index)"
     is_right="$(arg is_right)"
+    glove_serial="$(arg glove_serial)"
     publish_rate="$(arg publish_rate)" />
 </robot>

File: senseglove/senseglove_description/urdf/nova2/nova2_right.urdf.xacro (robot description, xacro)
@@ -5,4 +5,5 @@
   <xacro:arg name="glove_index"     default="0" />
   <xacro:arg name="is_right"        default="true" />
+  <xacro:arg name="glove_serial"    default=""/>
   <xacro:arg name="publish_rate"    default="60" />
   <!-- Import Nova2 Description Macro -->
@@ -19,4 +20,5 @@
     glove_index="$(arg glove_index)"
     is_right="$(arg is_right)"
+    glove_serial="$(arg glove_serial)"
     publish_rate="$(arg publish_rate)" />
 </robot>

Commit message: removed senseglove-setup completely, applied clang-format

File: senseglove/senseglove_description/ros2_control/nova2/nova2_left.ros2_control.xacro (robot description, xacro)
@@ -1,5 +1,5 @@
 <?xml version='1.0'?>
 <robot xmlns:xacro="http://www.ros.org/wiki/xacro">
-    <xacro:macro name="nova2_left_ros2_control" params="name prefix selected_robot glove_index is_right glove_serial publish_rate">
+    <xacro:macro name="nova2_left_ros2_control" params="name prefix selected_robot is_right glove_serial publish_rate">
         <!-- Include joint interfaces macro -->
         <xacro:include filename="$(find senseglove_description)/urdf/urdf_helper_macros/joint_interfaces_macro.xacro"/>
@@ -9,5 +9,4 @@
                 <plugin>senseglove_hardware_interface/SenseGloveHardwareInterface</plugin>
                 <param name="selected_robot">${selected_robot}</param>
-                <param name="glove_index">${glove_index}</param>
                 <param name="is_right">${is_right}</param>
                 <param name="glove_serial">${glove_serial}</param>

File: senseglove/senseglove_description/ros2_control/nova2/nova2_right.ros2_control.xacro (robot description, xacro)
@@ -1,5 +1,5 @@
 <?xml version='1.0'?>
 <robot xmlns:xacro="http://www.ros.org/wiki/xacro">
-    <xacro:macro name="nova2_right_ros2_control" params="name prefix selected_robot glove_index is_right glove_serial publish_rate">
+    <xacro:macro name="nova2_right_ros2_control" params="name prefix selected_robot is_right glove_serial publish_rate">
         <!-- Include joint interfaces macro -->
         <xacro:include filename="$(find senseglove_description)/urdf/urdf_helper_macros/joint_interfaces_macro.xacro"/>
@@ -9,5 +9,4 @@
                 <plugin>senseglove_hardware_interface/SenseGloveHardwareInterface</plugin>
                 <param name="selected_robot">${selected_robot}</param>
-                <param name="glove_index">${glove_index}</param>
                 <param name="is_right">${is_right}</param>
                 <param name="glove_serial">${glove_serial}</param>

File: senseglove/senseglove_description/urdf/nova2/nova2_left.description.xacro (robot description, xacro)
@@ -3,7 +3,7 @@
     <xacro:macro name="nova2_left" params="parent prefix">
         <!-- Constants -->
-        <xacro:property name="PI"           value="3.1415926535897931"/>
+        <xacro:property name="PI" value="3.1415926535897931"/>
         <xacro:property name="hover_height" value="0.5"/>
-        <xacro:property name="color_blue"   value="0.0 0.0 1.0 1.0"/>
+        <xacro:property name="color_blue" value="0.0 0.0 1.0 1.0"/>
         <link name="l_glove_hub">
             <visual name="l_glove_hub_visual">

File: senseglove/senseglove_description/urdf/nova2/nova2_left.urdf.xacro (robot description, xacro)
@@ -1,10 +1,9 @@
 <?xml version="1.0"?>
 <robot xmlns:xacro="http://www.ros.org/wiki/xacro" name="nova2">
-  <xacro:arg name="prefix"          default="" />
-  <xacro:arg name="selected_robot"  default="nova2_left" />
-  <xacro:arg name="glove_index"     default="0" />
-  <xacro:arg name="is_right"        default="false" />
-  <xacro:arg name="glove_serial"    default=""/>
-  <xacro:arg name="publish_rate"    default="60" />
+  <xacro:arg name="prefix" default="" />
+  <xacro:arg name="selected_robot" default="nova2_left" />
+  <xacro:arg name="is_right" default="false" />
+  <xacro:arg name="glove_serial" default=""/>
+  <xacro:arg name="publish_rate" default="60" />
   <!-- Import Nova2 Description Macro -->
   <xacro:include filename="$(find senseglove_description)/urdf/nova2/nova2_left.description.xacro" />
@@ -14,11 +13,4 @@
   <link name="world"/>
   <xacro:nova2_left parent="world" prefix="$(arg prefix)" />
-  <xacro:nova2_left_ros2_control
-    name="Nova2LeftControl"
-    prefix="$(arg prefix)"
-    selected_robot="$(arg selected_robot)"
-    glove_index="$(arg glove_index)"
-    is_right="$(arg is_right)"
-    glove_serial="$(arg glove_serial)"
-    publish_rate="$(arg publish_rate)" />
+  <xacro:nova2_left_ros2_control name="Nova2LeftControl" prefix="$(arg prefix)" selected_robot="$(arg selected_robot)" is_right="$(arg is_right)" glove_serial="$(arg glove_serial)" publish_rate="$(arg publish_rate)" />
 </robot>

File: senseglove/senseglove_description/urdf/nova2/nova2_right.description.xacro (robot description, xacro)
@@ -3,7 +3,7 @@
     <xacro:macro name="nova2_right" params="parent prefix">
         <!-- Constants -->
-        <xacro:property name="PI"           value="3.1415926535897931"/>
+        <xacro:property name="PI" value="3.1415926535897931"/>
         <xacro:property name="hover_height" value="0.5"/>
-        <xacro:property name="color_blue"   value="0.0 0.0 1.0 1.0"/>
+        <xacro:property name="color_blue" value="0.0 0.0 1.0 1.0"/>
         <link name="r_glove_hub">
             <visual name="r_glove_hub_visual">

File: senseglove/senseglove_description/urdf/nova2/nova2_right.urdf.xacro (robot description, xacro)
@@ -1,10 +1,9 @@
 <?xml version="1.0"?>
 <robot xmlns:xacro="http://www.ros.org/wiki/xacro" name="nova2">
-  <xacro:arg name="prefix"          default="" />
-  <xacro:arg name="selected_robot"  default="nova2_right" />
-  <xacro:arg name="glove_index"     default="0" />
-  <xacro:arg name="is_right"        default="true" />
-  <xacro:arg name="glove_serial"    default=""/>
-  <xacro:arg name="publish_rate"    default="60" />
+  <xacro:arg name="prefix" default="" />
+  <xacro:arg name="selected_robot" default="nova2_right" />
+  <xacro:arg name="is_right" default="true" />
+  <xacro:arg name="glove_serial" default=""/>
+  <xacro:arg name="publish_rate" default="60" />
   <!-- Import Nova2 Description Macro -->
   <xacro:include filename="$(find senseglove_description)/urdf/nova2/nova2_right.description.xacro" />
@@ -14,11 +13,4 @@
   <link name="world"/>
   <xacro:nova2_right parent="world" prefix="$(arg prefix)" />
-  <xacro:nova2_right_ros2_control
-    name="Nova2RightControl"
-    prefix="$(arg prefix)"
-    selected_robot="$(arg selected_robot)"
-    glove_index="$(arg glove_index)"
-    is_right="$(arg is_right)"
-    glove_serial="$(arg glove_serial)"
-    publish_rate="$(arg publish_rate)" />
+  <xacro:nova2_right_ros2_control name="Nova2RightControl" prefix="$(arg prefix)" selected_robot="$(arg selected_robot)" is_right="$(arg is_right)" glove_serial="$(arg glove_serial)" publish_rate="$(arg publish_rate)" />
 </robot>
